File: _autosave-SFUSat-Radio.kicad_pcb (KiCad board)
At the start: 4 copper layers, 50.8 x 25.4 mm, 61 parts, among them J1 SMA, P1 CONN_02X05, SW1 JS202011SCQN, SW2 JS202011SCQN, SW3 JS202011SCQN, SW4 JS202011SCQN, U1 2N7002DW, U2 CC1125, U3 BALF-112X-02D3, U4 SKY13372-467LF, U5 SKY65366-21, U6 BMI-S-101, U7 TPS799, U8 TPS799, U9 RT9183, X1 KT2520K40000DAW18TAS

Commit message: began RF chain
Parts:
- added C17: C, Capacitors_SMD:C_0402, F.Cu at (126.5, 113.1)
- added C18: C, Capacitors_SMD:C_0402, F.Cu at (127.7, 110.2)
- added C19: 47pF, Capacitors_SMD:C_0201, F.Cu at (129.5, 108.2)
- added C20: 47pF, Capacitors_SMD:C_0402, F.Cu at (136.0, 106.9)
- added C21: 47pF, Capacitors_SMD:C_0402, F.Cu at (136.0, 108.8)
- added L1: INDUCTOR, Capacitors_SMD:C_0402, F.Cu at (125.9, 110.7)
- added R8: R, Resistors_SMD:R_0402, F.Cu at (125.2, 112.9)
- moved C10 43.9 mm to (187.6, 135.8)
- moved C3 15.3 mm to (114.4, 106.8)
- moved U5 12.2 mm to (140.7, 107.4)
- moved U3 3.70 mm to (127.5, 108.2)
- moved U4 3.53 mm to (132.5, 107.9)
- moved U2 1.78 mm to (122.4, 107.2)
Connections:
- U3 pad E3: (no net) -> /Transceiver/RF_PA
Routing:
- net Net-(U5-Pad10): track 0.00 -> 5.69 mm
- net /Transceiver/RF_PA: track 0.00 -> 4.27 mm
- net Net-(C17-Pad1): track 0.00 -> 2.45 mm
- net /Transceiver/RF_TRX: track 0.00 -> 1.81 mm
- net /Transceiver/RF_LNAP: track 0.00 -> 1.81 mm
- net /Transceiver/RF_LNAN: track 0.00 -> 1.81 mm
- net Net-(C18-Pad1): track 0.00 -> 1.58 mm
- net /Front_End/TX: track 0.00 -> 1.53 mm
- net /Front_End/RX: track 0.00 -> 1.51 mm
- net Net-(C20-Pad2): track 0.00 -> 1.11 mm
- net Net-(C21-Pad2): track 0.00 -> 1.11 mm
- net Net-(C19-Pad1): track 0.00 -> 0.98 mm
- net Net-(C19-Pad2): track 0.00 -> 0.87 mm
Other:
- board size 50.8 x 25.4 mm -> 50.9 x 25.4 mm
- net class Default: clearance 0.2 -> 0.127
- net class RF_MS: clearance 0.2 -> 0.127
- rule trace_clearance: 0.2 -> 0.127
