File: Front_End.sch (KiCad schematic (older format))
At the start: 20 parts, among them P2 CONN_01X03, P3 CONN_01X03, SW3 JS202011SCQN, U5 SKY65366-21

Commit message: added CC1101, fixed mission symbols
Parts:
- C22, C23, C24, C25, C26, C27, C28, C29, C30: footprint (none) -> SFUSat:C_0402
- L2: symbol INDUCTOR -> L
- R10, R13, R14, R9: footprint (none) -> SFUSat:R_0402
- RV1: footprint SFUSat-Radio:TC33_SMD -> SFUSat:TC33_SMD; symbol POT-RESCUE-SFUSat-Radio -> POT
Changed lines of the file:
@@
 $EndComp
 $Comp
-L GND #PWR031
+L GND #PWR19
 U 1 1 58719F72
 P 5500 4650
-F 0 "#PWR031" H 5500 4400 50  0001 C CNN
+F 0 "#PWR19" H 5500 4400 50  0001 C CNN
 F 1 "GND" H 5500 4500 50  0000 C CNN
 F 2 "" H 5500 4650 50  0000 C CNN
@@
 F 0 "C25" H 5775 2450 50  0000 L CNN
 F 1 "220pF" H 5775 2250 50  0000 L CNN
-F 2 "" H 5788 2200 50  0001 C CNN
+F 2 "SFUSat:C_0402" H 5788 2200 50  0001 C CNN
 F 3 "" H 5750 2350 50  0000 C CNN
 	1    5750 2350
@@
 F 0 "C26" H 6075 2450 50  0000 L CNN
 F 1 "1nF" H 6075 2250 50  0000 L CNN
-F 2 "" H 6088 2200 50  0001 C CNN
+F 2 "SFUSat:C_0402" H 6088 2200 50  0001 C CNN
 F 3 "" H 6050 2350 50  0000 C CNN
 	1    6050 2350
@@
 F 0 "C27" H 6375 2450 50  0000 L CNN
 F 1 "1uF" H 6375 2250 50  0000 L CNN
-F 2 "" H 6388 2200 50  0001 C CNN
+F 2 "SFUSat:C_0402" H 6388 2200 50  0001 C CNN
 F 3 "" H 6350 2350 50  0000 C CNN
 	1    6350 2350
@@
 $EndComp
 $Comp
-L GND #PWR032
+L GND #PWR20
 U 1 1 5871BAFA
 P 5750 2550
-F 0 "#PWR032" H 5750 2300 50  0001 C CNN
+F 0 "#PWR20" H 5750 2300 50  0001 C CNN
 F 1 "GND" H 5750 2400 50  0000 C CNN
 F 2 "" H 5750 2550 50  0000 C CNN
@@
 $EndComp
 $Comp
-L GND #PWR033
+L GND #PWR21
 U 1 1 5871BB16
 P 6050 2550
-F 0 "#PWR033" H 6050 2300 50  0001 C CNN
+F 0 "#PWR21" H 6050 2300 50  0001 C CNN
 F 1 "GND" H 6050 2400 50  0000 C CNN
 F 2 "" H 6050 2550 50  0000 C CNN
@@
 $EndComp
 $Comp
-L GND #PWR034
+L GND #PWR22
 U 1 1 5871BB32
 P 6350 2550
-F 0 "#PWR034" H 6350 2300 50  0001 C CNN
+F 0 "#PWR22" H 6350 2300 50  0001 C CNN
 F 1 "GND" H 6350 2400 50  0000 C CNN
 F 2 "" H 6350 2550 50  0000 C CNN
@@
 F 0 "C24" H 5175 2450 50  0000 L CNN
 F 1 "220pF" H 5175 2250 50  0000 L CNN
-F 2 "" H 5188 2200 50  0001 C CNN
+F 2 "SFUSat:C_0402" H 5188 2200 50  0001 C CNN
 F 3 "" H 5150 2350 50  0000 C CNN
 	1    5150 2350
@@
 F 0 "C23" H 4875 2450 50  0000 L CNN
 F 1 "10nF" H 4875 2250 50  0000 L CNN
-F 2 "" H 4888 2200 50  0001 C CNN
+F 2 "SFUSat:C_0402" H 4888 2200 50  0001 C CNN
 F 3 "" H 4850 2350 50  0000 C CNN
 	1    4850 2350
@@
 $EndComp
 $Comp
-L GND #PWR035
+L GND #PWR18
 U 1 1 5871BD81
 P 5150 2550
-F 0 "#PWR035" H 5150 2300 50  0001 C CNN
+F 0 "#PWR18" H 5150 2300 50  0001 C CNN
 F 1 "GND" H 5150 2400 50  0000 C CNN
 F 2 "" H 5150 2550 50  0000 C CNN
@@
 $EndComp
 $Comp
-L GND #PWR036
+L GND #PWR17
 U 1 1 5871BDA1
 P 4850 2550
-F 0 "#PWR036" H 4850 2300 50  0001 C CNN
+F 0 "#PWR17" H 4850 2300 50  0001 C CNN
 F 1 "GND" H 4850 2400 50  0000 C CNN
 F 2 "" H 4850 2550 50  0000 C CNN
@@
 F 0 "C29" V 7300 3200 50  0000 C CNN
 F 1 "3pF" V 7600 3200 50  0000 C CNN
-F 2 "" H 7488 3050 50  0001 C CNN
+F 2 "SFUSat:C_0402" H 7488 3050 50  0001 C CNN
 F 3 "" H 7450 3200 50  0000 C CNN
 	1    7450 3200
@@
 F 0 "C28" H 7075 3450 50  0000 L CNN
 F 1 "8.2pF" H 7075 3250 50  0000 L CNN
-F 2 "" H 7088 3200 50  0001 C CNN
+F 2 "SFUSat:C_0402" H 7088 3200 50  0001 C CNN
 F 3 "" H 7050 3350 50  0000 C CNN
 	1    7050 3350
@@
 F 0 "C30" H 7875 3450 50  0000 L CNN
 F 1 "8.2pF" H 7875 3250 50  0000 L CNN
-F 2 "" H 7888 3200 50  0001 C CNN
+F 2 "SFUSat:C_0402" H 7888 3200 50  0001 C CNN
 F 3 "" H 7850 3350 50  0000 C CNN
 	1    7850 3350
@@
 $EndComp
 $Comp
-L INDUCTOR L2
+L L L2
 U 1 1 5871C1AA
 P 7450 2825
-F 0 "L2" V 7400 2825 50  0000 C CNN
+F 0 "L2" V 7399 2825 50  0000 C CNN
 F 1 "12nH" V 7550 2825 50  0000 C CNN
 F 2 "Capacitors_SMD:C_0402" H 7450 2825 50  0001 C CNN
@@
 	7050 2825 7050 3200
 $Comp
-L GND #PWR037
+L GND #PWR24
 U 1 1 5871C376
 P 7050 3600
-F 0 "#PWR037" H 7050 3350 50  0001 C CNN
+F 0 "#PWR24" H 7050 3350 50  0001 C CNN
 F 1 "GND" H 7050 3450 50  0000 C CNN
 F 2 "" H 7050 3600 50  0000 C CNN
@@
 $EndComp
 $Comp
-L GND #PWR038
+L GND #PWR25
 U 1 1 5871C39E
 P 7850 3600
-F 0 "#PWR038" H 7850 3350 50  0001 C CNN
+F 0 "#PWR25" H 7850 3350 50  0001 C CNN
 F 1 "GND" H 7850 3450 50  0000 C CNN
 F 2 "" H 7850 3600 50  0000 C CNN
@@
 F 0 "R9" V 4580 4150 50  0000 C CNN
 F 1 "0" V 4500 4150 50  0000 C CNN
-F 2 "" V 4430 4150 50  0001 C CNN
+F 2 "SFUSat:R_0402" V 4430 4150 50  0001 C CNN
 F 3 "" H 4500 4150 50  0000 C CNN
 	1    4500 4150
@@
 $EndComp
 $Comp
-L GND #PWR039
+L GND #PWR15
 U 1 1 5871CA19
 P 4500 4400
-F 0 "#PWR039" H 4500 4150 50  0001 C CNN
+F 0 "#PWR15" H 4500 4150 50  0001 C CNN
 F 1 "GND" H 4500 4250 50  0000 C CNN
 F 2 "" H 4500 4400 50  0000 C CNN
@@
 F 0 "C22" H 4175 3950 50  0000 L CNN
 F 1 "4.7nF" H 4175 3750 50  0000 L CNN
-F 2 "" H 4188 3700 50  0001 C CNN
+F 2 "SFUSat:C_0402" H 4188 3700 50  0001 C CNN
 F 3 "" H 4150 3850 50  0000 C CNN
 	1    4150 3850
@@
 $EndComp
 $Comp
-L GND #PWR040
+L GND #PWR14
 U 1 1 5871CD23
 P 4150 4050
-F 0 "#PWR040" H 4150 3800 50  0001 C CNN
+F 0 "#PWR14" H 4150 3800 50  0001 C CNN
 F 1 "GND" H 4150 3900 50  0000 C CNN
 F 2 "" H 4150 4050 50  0000 C CNN
@@
 F 0 "R10" V 4730 6450 50  0000 C CNN
 F 1 "634R" V 4650 6450 50  0000 C CNN
-F 2 "" V 4580 6450 50  0001 C CNN
+F 2 "SFUSat:R_0402" V 4580 6450 50  0001 C CNN
 F 3 "" H 4650 6450 50  0000 C CNN
 	1    4650 6450
@@
 $EndComp
 $Comp
-L GND #PWR041
+L GND #PWR16
 U 1 1 587C3C45
 P 4650 6600
-F 0 "#PWR041" H 4650 6350 50  0001 C CNN
+F 0 "#PWR16" H 4650 6350 50  0001 C CNN
 F 1 "GND" H 4650 6450 50  0000 C CNN
 F 2 "" H 4650 6600 50  0000 C CNN
@@
 3V3
 $Comp
-L POT-RESCUE-SFUSat-Radio RV1
+L POT RV1
 U 1 1 587CA745
 P 4650 5850
 F 0 "RV1" H 4650 5750 50  0000 C CNN
 F 1 "POT" H 4650 5850 50  0000 C CNN
-F 2 "SFUSat-Radio:TC33_SMD" H 4650 5850 50  0001 C CNN
+F 2 "SFUSat:TC33_SMD" H 4650 5850 50  0001 C CNN
 F 3 "" H 4650 5850 50  0000 C CNN
 	1    4650 5850
@@
 3V3
 $Comp
-L GND #PWR042
+L GND #PWR23
 U 1 1 58829BDE
 P 6400 6100
-F 0 "#PWR042" H 6400 5850 50  0001 C CNN
+F 0 "#PWR23" H 6400 5850 50  0001 C CNN
 F 1 "GND" H 6400 5950 50  0000 C CNN
 F 2 "" H 6400 6100 50  0000 C CNN
@@
 F 0 "R13" V 3380 5925 50  0000 C CNN
 F 1 "1k" V 3300 5925 50  0000 C CNN
-F 2 "" V 3230 5925 50  0001 C CNN
+F 2 "SFUSat:R_0402" V 3230 5925 50  0001 C CNN
 F 3 "" H 3300 5925 50  0000 C CNN
 	1    3300 5925
@@
 F 0 "R14" V 6830 6050 50  0000 C CNN
 F 1 "1k" V 6750 6050 50  0000 C CNN
-F 2 "" V 6680 6050 50  0001 C CNN
+F 2 "SFUSat:R_0402" V 6680 6050 50  0001 C CNN
 F 3 "" H 6750 6050 50  0000 C CNN
 	1    6750 6050

Commit message: fixed rescue library
Parts:
- P2, P3: footprint (none) -> SFUSat:Socket_Strip_Straight_1x03
- SW3: footprint (none) -> SFUSat:JS2020_TH
- U5: footprint (none) -> SFUSat:MCM-28
- W3: footprint (none) -> SFUSat:EXPOSED
Changed lines of the file:
@@
 EESchema Schematic File Version 2
-LIBS:SFUSat-Radio-rescue
 LIBS:power
 LIBS:device
@@
 F 0 "U5" H 5550 3725 60  0000 C TNN
 F 1 "SKY65366-21" H 5550 3775 60  0000 C BNN
-F 2 "" H 5550 3650 60  0001 C CNN
+F 2 "SFUSat:MCM-28" H 5550 3650 60  0001 C CNN
 F 3 "" H 5550 3650 60  0000 C CNN
 	1    5550 3750
@@
 $EndComp
 $Comp
-L GND #PWR19
+L GND #PWR018
 U 1 1 58719F72
 P 5500 4650
-F 0 "#PWR19" H 5500 4400 50  0001 C CNN
+F 0 "#PWR018" H 5500 4400 50  0001 C CNN
 F 1 "GND" H 5500 4500 50  0000 C CNN
 F 2 "" H 5500 4650 50  0000 C CNN
@@
 $EndComp
 $Comp
-L GND #PWR20
+L GND #PWR019
 U 1 1 5871BAFA
 P 5750 2550
-F 0 "#PWR20" H 5750 2300 50  0001 C CNN
+F 0 "#PWR019" H 5750 2300 50  0001 C CNN
 F 1 "GND" H 5750 2400 50  0000 C CNN
 F 2 "" H 5750 2550 50  0000 C CNN
@@
 $EndComp
 $Comp
-L GND #PWR21
+L GND #PWR020
 U 1 1 5871BB16
 P 6050 2550
-F 0 "#PWR21" H 6050 2300 50  0001 C CNN
+F 0 "#PWR020" H 6050 2300 50  0001 C CNN
 F 1 "GND" H 6050 2400 50  0000 C CNN
 F 2 "" H 6050 2550 50  0000 C CNN
@@
 $EndComp
 $Comp
-L GND #PWR22
+L GND #PWR021
 U 1 1 5871BB32
 P 6350 2550
-F 0 "#PWR22" H 6350 2300 50  0001 C CNN
+F 0 "#PWR021" H 6350 2300 50  0001 C CNN
 F 1 "GND" H 6350 2400 50  0000 C CNN
 F 2 "" H 6350 2550 50  0000 C CNN
@@
 $EndComp
 $Comp
-L GND #PWR18
+L GND #PWR022
 U 1 1 5871BD81
 P 5150 2550
-F 0 "#PWR18" H 5150 2300 50  0001 C CNN
+F 0 "#PWR022" H 5150 2300 50  0001 C CNN
 F 1 "GND" H 5150 2400 50  0000 C CNN
 F 2 "" H 5150 2550 50  0000 C CNN
@@
 $EndComp
 $Comp
-L GND #PWR17
+L GND #PWR023
 U 1 1 5871BDA1
 P 4850 2550
-F 0 "#PWR17" H 4850 2300 50  0001 C CNN
+F 0 "#PWR023" H 4850 2300 50  0001 C CNN
 F 1 "GND" H 4850 2400 50  0000 C CNN
 F 2 "" H 4850 2550 50  0000 C CNN
@@
 	7050 2825 7050 3200
 $Comp
-L GND #PWR24
+L GND #PWR024
 U 1 1 5871C376
 P 7050 3600
-F 0 "#PWR24" H 7050 3350 50  0001 C CNN
+F 0 "#PWR024" H 7050 3350 50  0001 C CNN
 F 1 "GND" H 7050 3450 50  0000 C CNN
 F 2 "" H 7050 3600 50  0000 C CNN
@@
 $EndComp
 $Comp
-L GND #PWR25
+L GND #PWR025
 U 1 1 5871C39E
 P 7850 3600
-F 0 "#PWR25" H 7850 3350 50  0001 C CNN
+F 0 "#PWR025" H 7850 3350 50  0001 C CNN
 F 1 "GND" H 7850 3450 50  0000 C CNN
 F 2 "" H 7850 3600 50  0000 C CNN
@@
 $EndComp
 $Comp
-L GND #PWR15
+L GND #PWR026
 U 1 1 5871CA19
 P 4500 4400
-F 0 "#PWR15" H 4500 4150 50  0001 C CNN
+F 0 "#PWR026" H 4500 4150 50  0001 C CNN
 F 1 "GND" H 4500 4250 50  0000 C CNN
 F 2 "" H 4500 4400 50  0000 C CNN
@@
 $EndComp
 $Comp
-L GND #PWR14
+L GND #PWR027
 U 1 1 5871CD23
 P 4150 4050
-F 0 "#PWR14" H 4150 3800 50  0001 C CNN
+F 0 "#PWR027" H 4150 3800 50  0001 C CNN
 F 1 "GND" H 4150 3900 50  0000 C CNN
 F 2 "" H 4150 4050 50  0000 C CNN
@@
 $EndComp
 $Comp
-L GND #PWR16
+L GND #PWR028
 U 1 1 587C3C45
 P 4650 6600
-F 0 "#PWR16" H 4650 6350 50  0001 C CNN
+F 0 "#PWR028" H 4650 6350 50  0001 C CNN
 F 1 "GND" H 4650 6450 50  0000 C CNN
 F 2 "" H 4650 6600 50  0000 C CNN
@@
 F 0 "SW3" H 6100 5750 60  0000 C CNN
 F 1 "JS202011SCQN" H 5900 6300 60  0000 C CNN
-F 2 "" H 5900 6150 60  0001 C CNN
+F 2 "SFUSat:JS2020_TH" H 5900 6150 60  0001 C CNN
 F 3 "" H 5900 6150 60  0000 C CNN
 	1    5900 6150
@@
 3V3
 $Comp
-L GND #PWR23
+L GND #PWR029
 U 1 1 58829BDE
 P 6400 6100
-F 0 "#PWR23" H 6400 5850 50  0001 C CNN
+F 0 "#PWR029" H 6400 5850 50  0001 C CNN
 F 1 "GND" H 6400 5950 50  0000 C CNN
 F 2 "" H 6400 6100 50  0000 C CNN
@@
 F 0 "P3" H 3900 6500 50  0000 C CNN
 F 1 "CONN_01X03" V 4000 6300 50  0000 C CNN
-F 2 "" H 3900 6300 50  0001 C CNN
+F 2 "SFUSat:Socket_Strip_Straight_1x03" H 3900 6300 50  0001 C CNN
 F 3 "" H 3900 6300 50  0000 C CNN
 	1    3900 6300
@@
 F 0 "P2" H 3100 6500 50  0000 C CNN
 F 1 "CONN_01X03" V 3200 6300 50  0000 C CNN
-F 2 "" H 3100 6300 50  0001 C CNN
+F 2 "SFUSat:Socket_Strip_Straight_1x03" H 3100 6300 50  0001 C CNN
 F 3 "" H 3100 6300 50  0000 C CNN
 	1    3100 6300
@@
 F 0 "W3" H 4300 6320 50  0000 C CNN
 F 1 "TEST_1P" H 4300 6250 50  0000 C CNN
-F 2 "" H 4500 6050 50  0001 C CNN
+F 2 "SFUSat:EXPOSED" H 4500 6050 50  0001 C CNN
 F 3 "" H 4500 6050 50  0000 C CNN
 	1    4300 6050

Commit message: Added CC1101-Q1 and supporting components
Also added the pad that routes to the SMA for RF path testing
Parts:
- L2: footprint Capacitors_SMD:C_0402 -> SFUSat:L_0402
Changed lines of the file:
@@
 $EndComp
 $Comp
-L GND #PWR018
+L GND #PWR025
 U 1 1 58719F72
 P 5500 4650
-F 0 "#PWR018" H 5500 4400 50  0001 C CNN
+F 0 "#PWR025" H 5500 4400 50  0001 C CNN
 F 1 "GND" H 5500 4500 50  0000 C CNN
 F 2 "" H 5500 4650 50  0000 C CNN
@@
 $EndComp
 $Comp
-L GND #PWR019
+L GND #PWR026
 U 1 1 5871BAFA
 P 5750 2550
-F 0 "#PWR019" H 5750 2300 50  0001 C CNN
+F 0 "#PWR026" H 5750 2300 50  0001 C CNN
 F 1 "GND" H 5750 2400 50  0000 C CNN
 F 2 "" H 5750 2550 50  0000 C CNN
@@
 $EndComp
 $Comp
-L GND #PWR020
+L GND #PWR027
 U 1 1 5871BB16
 P 6050 2550
-F 0 "#PWR020" H 6050 2300 50  0001 C CNN
+F 0 "#PWR027" H 6050 2300 50  0001 C CNN
 F 1 "GND" H 6050 2400 50  0000 C CNN
 F 2 "" H 6050 2550 50  0000 C CNN
@@
 $EndComp
 $Comp
-L GND #PWR021
+L GND #PWR028
 U 1 1 5871BB32
 P 6350 2550
-F 0 "#PWR021" H 6350 2300 50  0001 C CNN
+F 0 "#PWR028" H 6350 2300 50  0001 C CNN
 F 1 "GND" H 6350 2400 50  0000 C CNN
 F 2 "" H 6350 2550 50  0000 C CNN
@@
 $EndComp
 $Comp
-L GND #PWR022
+L GND #PWR029
 U 1 1 5871BD81
 P 5150 2550
-F 0 "#PWR022" H 5150 2300 50  0001 C CNN
+F 0 "#PWR029" H 5150 2300 50  0001 C CNN
 F 1 "GND" H 5150 2400 50  0000 C CNN
 F 2 "" H 5150 2550 50  0000 C CNN
@@
 $EndComp
 $Comp
-L GND #PWR023
+L GND #PWR030
 U 1 1 5871BDA1
 P 4850 2550
-F 0 "#PWR023" H 4850 2300 50  0001 C CNN
+F 0 "#PWR030" H 4850 2300 50  0001 C CNN
 F 1 "GND" H 4850 2400 50  0000 C CNN
 F 2 "" H 4850 2550 50  0000 C CNN
@@
 L L L2
 U 1 1 5871C1AA
-P 7450 2825
-F 0 "L2" V 7399 2825 50  0000 C CNN
-F 1 "12nH" V 7550 2825 50  0000 C CNN
-F 2 "Capacitors_SMD:C_0402" H 7450 2825 50  0001 C CNN
-F 3 "" H 7450 2825 50  0000 C CNN
-	1    7450 2825
+P 7450 2850
+F 0 "L2" V 7399 2850 50  0000 C BNN
+F 1 "12nH" V 7500 2850 50  0000 C TNN
+F 2 "SFUSat:L_0402" H 7450 2850 50  0001 C CNN
+F 3 "" H 7450 2850 50  0000 C CNN
+	1    7450 2850
 	0    1    1    0
 $EndComp
@@
 	7600 3200 8200 3200
 Connection ~ 7850 3200
-Wire Wire Line
-	7850 2825 7850 3200
-Wire Wire Line
-	7150 2825 7050 2825
-Wire Wire Line
-	7050 2825 7050 3200
-$Comp
-L GND #PWR024
+$Comp
+L GND #PWR031
 U 1 1 5871C376
 P 7050 3600
-F 0 "#PWR024" H 7050 3350 50  0001 C CNN
+F 0 "#PWR031" H 7050 3350 50  0001 C CNN
 F 1 "GND" H 7050 3450 50  0000 C CNN
 F 2 "" H 7050 3600 50  0000 C CNN
@@
 $EndComp
 $Comp
-L GND #PWR025
+L GND #PWR032
 U 1 1 5871C39E
 P 7850 3600
-F 0 "#PWR025" H 7850 3350 50  0001 C CNN
+F 0 "#PWR032" H 7850 3350 50  0001 C CNN
 F 1 "GND" H 7850 3450 50  0000 C CNN
 F 2 "" H 7850 3600 50  0000 C CNN
@@
 $EndComp
 $Comp
-L GND #PWR026
+L GND #PWR033
 U 1 1 5871CA19
 P 4500 4400
-F 0 "#PWR026" H 4500 4150 50  0001 C CNN
+F 0 "#PWR033" H 4500 4150 50  0001 C CNN
 F 1 "GND" H 4500 4250 50  0000 C CNN
 F 2 "" H 4500 4400 50  0000 C CNN
@@
 $EndComp
 $Comp
-L GND #PWR027
+L GND #PWR034
 U 1 1 5871CD23
 P 4150 4050
-F 0 "#PWR027" H 4150 3800 50  0001 C CNN
+F 0 "#PWR034" H 4150 3800 50  0001 C CNN
 F 1 "GND" H 4150 3900 50  0000 C CNN
 F 2 "" H 4150 4050 50  0000 C CNN
@@
 Wire Notes Line
 	3800 2675 3800 3075
-Wire Wire Line
-	7750 2825 7850 2825
 $Comp
 L R R10
@@
 $EndComp
 $Comp
-L GND #PWR028
+L GND #PWR035
 U 1 1 587C3C45
 P 4650 6600
-F 0 "#PWR028" H 4650 6350 50  0001 C CNN
+F 0 "#PWR035" H 4650 6350 50  0001 C CNN
 F 1 "GND" H 4650 6450 50  0000 C CNN
 F 2 "" H 4650 6600 50  0000 C CNN
@@
 3V3
 $Comp
-L GND #PWR029
+L GND #PWR036
 U 1 1 58829BDE
 P 6400 6100
-F 0 "#PWR029" H 6400 5850 50  0001 C CNN
+F 0 "#PWR036" H 6400 5850 50  0001 C CNN
 F 1 "GND" H 6400 5950 50  0000 C CNN
 F 2 "" H 6400 6100 50  0000 C CNN
@@
 Wire Wire Line
 	6750 5850 6850 5850
+Wire Wire Line
+	7600 2850 7850 2850
+Wire Wire Line
+	7850 2850 7850 3200
+Wire Wire Line
+	7300 2850 7050 2850
+Wire Wire Line
+	7050 2850 7050 3200
 $EndSCHEMATC

Commit message: Renumbered reference designators
Parts:
- R7: renamed from R10; value 634R -> 634
- renumbered C22 to C11, C23 to C12, C24 to C13, C25 to C14, C26 to C15, C27 to C16, C28 to C17, C29 to C18, C30 to C19, L2 to L1, R13 to R5, R9 to R6, R14 to R8, SW3 to SW1, U5 to U8, W3 to W2
Changed lines of the file:
@@
 RX
 $Comp
-L SKY65366-21 U5
+L SKY65366-21 U8
 U 1 1 58719E85
 P 5550 3750
-F 0 "U5" H 5550 3725 60  0000 C TNN
+F 0 "U8" H 5550 3725 60  0000 C TNN
 F 1 "SKY65366-21" H 5550 3775 60  0000 C BNN
 F 2 "SFUSat:MCM-28" H 5550 3650 60  0001 C CNN
@@
 $EndComp
 $Comp
-L GND #PWR025
+L GND #PWR024
 U 1 1 58719F72
 P 5500 4650
-F 0 "#PWR025" H 5500 4400 50  0001 C CNN
+F 0 "#PWR024" H 5500 4400 50  0001 C CNN
 F 1 "GND" H 5500 4500 50  0000 C CNN
 F 2 "" H 5500 4650 50  0000 C CNN
@@
 3V6
 $Comp
-L C C25
+L C C14
 U 1 1 5871B9DF
 P 5750 2350
-F 0 "C25" H 5775 2450 50  0000 L CNN
+F 0 "C14" H 5775 2450 50  0000 L CNN
 F 1 "220pF" H 5775 2250 50  0000 L CNN
 F 2 "SFUSat:C_0402" H 5788 2200 50  0001 C CNN
@@
 $EndComp
 $Comp
-L C C26
+L C C15
 U 1 1 5871BA4C
 P 6050 2350
-F 0 "C26" H 6075 2450 50  0000 L CNN
+F 0 "C15" H 6075 2450 50  0000 L CNN
 F 1 "1nF" H 6075 2250 50  0000 L CNN
 F 2 "SFUSat:C_0402" H 6088 2200 50  0001 C CNN
@@
 $EndComp
 $Comp
-L C C27
+L C C16
 U 1 1 5871BAAB
 P 6350 2350
-F 0 "C27" H 6375 2450 50  0000 L CNN
+F 0 "C16" H 6375 2450 50  0000 L CNN
 F 1 "1uF" H 6375 2250 50  0000 L CNN
 F 2 "SFUSat:C_0402" H 6388 2200 50  0001 C CNN
@@
 $EndComp
 $Comp
-L GND #PWR026
+L GND #PWR025
 U 1 1 5871BAFA
 P 5750 2550
-F 0 "#PWR026" H 5750 2300 50  0001 C CNN
+F 0 "#PWR025" H 5750 2300 50  0001 C CNN
 F 1 "GND" H 5750 2400 50  0000 C CNN
 F 2 "" H 5750 2550 50  0000 C CNN
@@
 $EndComp
 $Comp
-L GND #PWR027
+L GND #PWR026
 U 1 1 5871BB16
 P 6050 2550
-F 0 "#PWR027" H 6050 2300 50  0001 C CNN
+F 0 "#PWR026" H 6050 2300 50  0001 C CNN
 F 1 "GND" H 6050 2400 50  0000 C CNN
 F 2 "" H 6050 2550 50  0000 C CNN
@@
 $EndComp
 $Comp
-L GND #PWR028
+L GND #PWR027
 U 1 1 5871BB32
 P 6350 2550
-F 0 "#PWR028" H 6350 2300 50  0001 C CNN
+F 0 "#PWR027" H 6350 2300 50  0001 C CNN
 F 1 "GND" H 6350 2400 50  0000 C CNN
 F 2 "" H 6350 2550 50  0000 C CNN
@@
 Connection ~ 5700 2900
 $Comp
-L C C24
+L C C13
 U 1 1 5871BCCF
 P 5150 2350
-F 0 "C24" H 5175 2450 50  0000 L CNN
+F 0 "C13" H 5175 2450 50  0000 L CNN
 F 1 "220pF" H 5175 2250 50  0000 L CNN
 F 2 "SFUSat:C_0402" H 5188 2200 50  0001 C CNN
@@
 $EndComp
 $Comp
-L C C23
+L C C12
 U 1 1 5871BD40
 P 4850 2350
-F 0 "C23" H 4875 2450 50  0000 L CNN
+F 0 "C12" H 4875 2450 50  0000 L CNN
 F 1 "10nF" H 4875 2250 50  0000 L CNN
 F 2 "SFUSat:C_0402" H 4888 2200 50  0001 C CNN
@@
 $EndComp
 $Comp
-L GND #PWR029
+L GND #PWR028
 U 1 1 5871BD81
 P 5150 2550
-F 0 "#PWR029" H 5150 2300 50  0001 C CNN
+F 0 "#PWR028" H 5150 2300 50  0001 C CNN
 F 1 "GND" H 5150 2400 50  0000 C CNN
 F 2 "" H 5150 2550 50  0000 C CNN
@@
 $EndComp
 $Comp
-L GND #PWR030
+L GND #PWR029
 U 1 1 5871BDA1
 P 4850 2550
-F 0 "#PWR030" H 4850 2300 50  0001 C CNN
+F 0 "#PWR029" H 4850 2300 50  0001 C CNN
 F 1 "GND" H 4850 2400 50  0000 C CNN
 F 2 "" H 4850 2550 50  0000 C CNN
@@
 	6400 3400 6400 3600
 $Comp
-L C C29
+L C C18
 U 1 1 5871C0B1
 P 7450 3200
-F 0 "C29" V 7300 3200 50  0000 C CNN
+F 0 "C18" V 7300 3200 50  0000 C CNN
 F 1 "3pF" V 7600 3200 50  0000 C CNN
 F 2 "SFUSat:C_0402" H 7488 3050 50  0001 C CNN
@@
 $EndComp
 $Comp
-L C C28
+L C C17
 U 1 1 5871C0F0
 P 7050 3350
-F 0 "C28" H 7075 3450 50  0000 L CNN
+F 0 "C17" H 7075 3450 50  0000 L CNN
 F 1 "8.2pF" H 7075 3250 50  0000 L CNN
 F 2 "SFUSat:C_0402" H 7088 3200 50  0001 C CNN
@@
 $EndComp
 $Comp
-L C C30
+L C C19
 U 1 1 5871C127
 P 7850 3350
-F 0 "C30" H 7875 3450 50  0000 L CNN
+F 0 "C19" H 7875 3450 50  0000 L CNN
 F 1 "8.2pF" H 7875 3250 50  0000 L CNN
 F 2 "SFUSat:C_0402" H 7888 3200 50  0001 C CNN
@@
 $EndComp
 $Comp
-L L L2
+L L L1
 U 1 1 5871C1AA
 P 7450 2850
-F 0 "L2" V 7399 2850 50  0000 C BNN
+F 0 "L1" V 7399 2850 50  0000 C BNN
 F 1 "12nH" V 7500 2850 50  0000 C TNN
 F 2 "SFUSat:L_0402" H 7450 2850 50  0001 C CNN
@@
 Connection ~ 7850 3200
 $Comp
-L GND #PWR031
+L GND #PWR030
 U 1 1 5871C376
 P 7050 3600
-F 0 "#PWR031" H 7050 3350 50  0001 C CNN
+F 0 "#PWR030" H 7050 3350 50  0001 C CNN
 F 1 "GND" H 7050 3450 50  0000 C CNN
 F 2 "" H 7050 3600 50  0000 C CNN
@@
 $EndComp
 $Comp
-L GND #PWR032
+L GND #PWR031
 U 1 1 5871C39E
 P 7850 3600
-F 0 "#PWR032" H 7850 3350 50  0001 C CNN
+F 0 "#PWR031" H 7850 3350 50  0001 C CNN
 F 1 "GND" H 7850 3450 50  0000 C CNN
 F 2 "" H 7850 3600 50  0000 C CNN
@@
 	7050 3500 7050 3600
 $Comp
-L R R9
+L R R6
 U 1 1 5871C966
 P 4500 4150
-F 0 "R9" V 4580 4150 50  0000 C CNN
+F 0 "R6" V 4580 4150 50  0000 C CNN
 F 1 "0" V 4500 4150 50  0000 C CNN
 F 2 "SFUSat:R_0402" V 4430 4150 50  0001 C CNN
@@
 $EndComp
 $Comp
-L GND #PWR033
+L GND #PWR032
 U 1 1 5871CA19
 P 4500 4400
-F 0 "#PWR033" H 4500 4150 50  0001 C CNN
+F 0 "#PWR032" H 4500 4150 50  0001 C CNN
 F 1 "GND" H 4500 4250 50  0000 C CNN
 F 2 "" H 4500 4400 50  0000 C CNN
@@
 	4500 4300 4500 4400
 $Comp
-L C C22
+L C C11
 U 1 1 5871CCE4
 P 4150 3850
-F 0 "C22" H 4175 3950 50  0000 L CNN
+F 0 "C11" H 4175 3950 50  0000 L CNN
 F 1 "4.7nF" H 4175 3750 50  0000 L CNN
 F 2 "SFUSat:C_0402" H 4188 3700 50  0001 C CNN
@@
 $EndComp
 $Comp
-L GND #PWR034
+L GND #PWR033
 U 1 1 5871CD23
 P 4150 4050
-F 0 "#PWR034" H 4150 3800 50  0001 C CNN
+F 0 "#PWR033" H 4150 3800 50  0001 C CNN
 F 1 "GND" H 4150 3900 50  0000 C CNN
 F 2 "" H 4150 4050 50  0000 C CNN
@@
 	3800 2675 3800 3075
 $Comp
-L R R10
+L R R7
 U 1 1 587C3C10
 P 4650 6450
-F 0 "R10" V 4730 6450 50  0000 C CNN
-F 1 "634R" V 4650 6450 50  0000 C CNN
+F 0 "R7" V 4730 6450 50  0000 C CNN
+F 1 "634" V 4650 6450 50  0000 C CNN
 F 2 "SFUSat:R_0402" V 4580 6450 50  0001 C CNN
 F 3 "" H 4650 6450 50  0000 C CNN
@@
 $EndComp
 $Comp
-L GND #PWR035
+L GND #PWR034
 U 1 1 587C3C45
 P 4650 6600
-F 0 "#PWR035" H 4650 6350 50  0001 C CNN
+F 0 "#PWR034" H 4650 6350 50  0001 C CNN
 F 1 "GND" H 4650 6450 50  0000 C CNN
 F 2 "" H 4650 6600 50  0000 C CNN
@@
 TR and BYP should not be \npulled high if EN is pulled low
 $Comp
-L JS202011SCQN SW3
+L JS202011SCQN SW1
 U 1 1 58828A5A
 P 5900 6150
-F 0 "SW3" H 6100 5750 60  0000 C CNN
+F 0 "SW1" H 6100 5750 60  0000 C CNN
 F 1 "JS202011SCQN" H 5900 6300 60  0000 C CNN
 F 2 "SFUSat:JS2020_TH" H 5900 6150 60  0001 C CNN
@@
 3V3
 $Comp
-L GND #PWR036
+L GND #PWR035
 U 1 1 58829BDE
 P 6400 6100
-F 0 "#PWR036" H 6400 5850 50  0001 C CNN
+F 0 "#PWR035" H 6400 5850 50  0001 C CNN
 F 1 "GND" H 6400 5950 50  0000 C CNN
 F 2 "" H 6400 6100 50  0000 C CNN
@@
 	3300 6300 3450 6300
 $Comp
-L TEST_1P W3
+L TEST_1P W2
 U 1 1 58821DE8
 P 4300 6050
-F 0 "W3" H 4300 6320 50  0000 C CNN
+F 0 "W2" H 4300 6320 50  0000 C CNN
 F 1 "TEST_1P" H 4300 6250 50  0000 C CNN
 F 2 "SFUSat:EXPOSED" H 4500 6050 50  0001 C CNN
@@
 Connection ~ 4300 6200
 $Comp
-L R R13
+L R R5
 U 1 1 58948F89
 P 3300 5925
-F 0 "R13" V 3380 5925 50  0000 C CNN
+F 0 "R5" V 3380 5925 50  0000 C CNN
 F 1 "1k" V 3300 5925 50  0000 C CNN
 F 2 "SFUSat:R_0402" V 3230 5925 50  0001 C CNN
@@
 $EndComp
 $Comp
-L R R14
+L R R8
 U 1 1 5894915C
 P 6750 6050
-F 0 "R14" V 6830 6050 50  0000 C CNN
+F 0 "R8" V 6830 6050 50  0000 C CNN
 F 1 "1k" V 6750 6050 50  0000 C CNN
 F 2 "SFUSat:R_0402" V 6680 6050 50  0001 C CNN
