File: Front_End.sch (KiCad schematic (older format))
At the start: 20 parts, among them P2 CONN_01X03, P3 CONN_01X03, SW1 JS202011SCQN, U8 SKY65366-21

Commit message: pulled SKY en high, replaced BYP with jump
Parts:
- removed P2: CONN_01X03, SFUSat:Socket_Strip_Straight_1x03, symbol CONN_01X03
- removed R5: 1k, SFUSat:R_0402, symbol R
- removed SW1: JS202011SCQN, SFUSat:JS2020_TH, symbol JS202011SCQN
- added P?: CONN_01X03, SFUSat:Socket_Strip_Straight_1x03, symbol CONN_01X03
- added R?: 1k, symbol R
Connections:
- net labels removed: EN, EXT_EN
- wire segments 43 -> 44
Other:
- moved on the sheet: RV1
Changed lines of the file:
@@
 	5500 4500 5500 4650
 Connection ~ 5500 4500
-Text HLabel 4650 2200 0    60   Input ~ 0
+Text HLabel 4350 2200 0    60   Input ~ 0
 3V3
 Text HLabel 6600 2200 2    60   Input ~ 0
@@
 	4850 2500 4850 2550
 Wire Wire Line
-	4650 2200 5400 2200
+	4350 2200 5400 2200
 Wire Wire Line
 	5300 2900 5400 2900
@@
 Wire Wire Line
 	3800 3450 4700 3450
-Wire Wire Line
-	4700 3350 3800 3350
-Text HLabel 3300 6400 2    60   Input ~ 0
-EXT_EN
 Text Notes 3400 2775 0    60   ~ 0
 TRX_SIG
@@
 Text Label 4350 6300 2    60   ~ 0
 VPC
-Text HLabel 4800 5850 2    60   Input ~ 0
+Text HLabel 4650 5700 1    60   Input ~ 0
 3V3
 $Comp
 L POT RV1
 U 1 1 587CA745
-P 4650 5850
-F 0 "RV1" H 4650 5750 50  0000 C CNN
-F 1 "POT" H 4650 5850 50  0000 C CNN
-F 2 "SFUSat:TC33_SMD" H 4650 5850 50  0001 C CNN
-F 3 "" H 4650 5850 50  0000 C CNN
-	1    4650 5850
-	0    1    1    0
+P 4650 5950
+F 0 "RV1" H 4650 5850 50  0000 C CNN
+F 1 "POT" H 4650 5950 50  0000 C CNN
+F 2 "SFUSat:TC33_SMD" H 4650 5950 50  0001 C CNN
+F 3 "" H 4650 5950 50  0000 C CNN
+	1    4650 5950
+	1    0    0    -1
 $EndComp
 Wire Wire Line
 	4650 6200 4100 6200
-Text HLabel 3600 5625 2    60   Input ~ 0
-3V3
-Text Label 3800 3350 0    60   ~ 0
-EN
-Text Label 3450 6300 2    60   ~ 0
-EN
 Text Notes 2100 3600 0    60   ~ 0
 TR and BYP should not be \npulled high if EN is pulled low
-$Comp
-L JS202011SCQN SW1
-U 1 1 58828A5A
-P 5900 6150
-F 0 "SW1" H 6100 5750 60  0000 C CNN
-F 1 "JS202011SCQN" H 5900 6300 60  0000 C CNN
-F 2 "SFUSat:JS2020_TH" H 5900 6150 60  0001 C CNN
-F 3 "" H 5900 6150 60  0000 C CNN
-	1    5900 6150
-	1    0    0    -1
-$EndComp
-Wire Wire Line
-	5400 6150 5200 6150
-Text Label 5200 6150 0    60   ~ 0
-BYP
 Text Label 3800 3450 0    60   ~ 0
 BYP
@@
 L GND #PWR035
 U 1 1 58829BDE
-P 6400 6100
-F 0 "#PWR035" H 6400 5850 50  0001 C CNN
-F 1 "GND" H 6400 5950 50  0000 C CNN
-F 2 "" H 6400 6100 50  0000 C CNN
-F 3 "" H 6400 6100 50  0000 C CNN
-	1    6400 6100
+P 6400 6400
+F 0 "#PWR035" H 6400 6150 50  0001 C CNN
+F 1 "GND" H 6400 6250 50  0000 C CNN
+F 2 "" H 6400 6400 50  0000 C CNN
+F 3 "" H 6400 6400 50  0000 C CNN
+	1    6400 6400
 	0    -1   -1   0
 $EndComp
@@
 	-1   0    0    1
 $EndComp
-$Comp
-L CONN_01X03 P2
-U 1 1 5881FDBC
-P 3100 6300
-F 0 "P2" H 3100 6500 50  0000 C CNN
-F 1 "CONN_01X03" V 3200 6300 50  0000 C CNN
-F 2 "SFUSat:Socket_Strip_Straight_1x03" H 3100 6300 50  0001 C CNN
-F 3 "" H 3100 6300 50  0000 C CNN
-	1    3100 6300
-	-1   0    0    1
-$EndComp
 Wire Wire Line
 	4100 6300 4350 6300
-Wire Wire Line
-	3300 6300 3450 6300
 $Comp
 L TEST_1P W2
@@
 Connection ~ 4300 6200
 $Comp
-L R R5
-U 1 1 58948F89
-P 3300 5925
-F 0 "R5" V 3380 5925 50  0000 C CNN
-F 1 "1k" V 3300 5925 50  0000 C CNN
-F 2 "SFUSat:R_0402" V 3230 5925 50  0001 C CNN
-F 3 "" H 3300 5925 50  0000 C CNN
-	1    3300 5925
-	1    0    0    -1
-$EndComp
-$Comp
 L R R8
 U 1 1 5894915C
@@
 $EndComp
 Wire Wire Line
-	3300 6075 3300 6200
-Wire Wire Line
-	3300 5775 3300 5625
-Wire Wire Line
-	3300 5625 3600 5625
-Wire Wire Line
-	6750 6200 6400 6200
+	2900 5625 3200 5625
+Wire Wire Line
+	6300 6200 6750 6200
 Wire Wire Line
 	6750 5900 6750 5850
@@
 Wire Wire Line
 	7050 2850 7050 3200
+Wire Wire Line
+	4550 3350 4700 3350
+Wire Wire Line
+	4550 3100 4550 3350
+Wire Wire Line
+	4550 2800 4550 2200
+Connection ~ 4550 2200
+$Comp
+L CONN_01X03 P?
+U 1 1 592E3D25
+P 6100 6300
+F 0 "P?" H 6100 6500 50  0000 C CNN
+F 1 "CONN_01X03" V 6200 6300 50  0000 C CNN
+F 2 "SFUSat:Socket_Strip_Straight_1x03" H 6100 6300 50  0001 C CNN
+F 3 "" H 6100 6300 50  0000 C CNN
+	1    6100 6300
+	-1   0    0    1
+$EndComp
+Wire Wire Line
+	6400 6400 6300 6400
+Wire Wire Line
+	6300 6300 6800 6300
+Text Label 6800 6300 0    60   ~ 0
+BYP
+Wire Wire Line
+	4650 5700 4650 5800
+$Comp
+L R R?
+U 1 1 592E46FC
+P 4550 2950
+F 0 "R?" V 4630 2950 50  0000 C CNN
+F 1 "1k" V 4550 2950 50  0000 C CNN
+F 2 "" V 4480 2950 50  0001 C CNN
+F 3 "" H 4550 2950 50  0001 C CNN
+	1    4550 2950
+	1    0    0    -1
+$EndComp
 $EndSCHEMATC

Commit message: Updated schematic and layout
Added extra decoupling caps based on TI feedback and forward annotated changes to the PCB
Parts:
- R6: renamed from R?; footprint (none) -> SFUSat:R_0402
- W2: footprint SFUSat:EXPOSED -> SFUSat:Measurement_Point_Round-SMD-Pad_Big
- gave numbers to parts that had none: 1
- renumbered C11 to C16, C12 to C17, C13 to C18, C14 to C19, C15 to C20, C16 to C21, C17 to C22, C18 to C23, C19 to C24, P3 to P2, R6 to R5
Changed lines of the file:
@@
 EESchema Schematic File Version 2
+LIBS:SFUSat-Radio-rescue
 LIBS:power
 LIBS:device
@@
 $EndComp
 $Comp
-L GND #PWR024
+L GND #PWR029
 U 1 1 58719F72
 P 5500 4650
-F 0 "#PWR024" H 5500 4400 50  0001 C CNN
+F 0 "#PWR029" H 5500 4400 50  0001 C CNN
 F 1 "GND" H 5500 4500 50  0000 C CNN
 F 2 "" H 5500 4650 50  0000 C CNN
@@
 3V6
 $Comp
-L C C14
+L C C19
 U 1 1 5871B9DF
 P 5750 2350
-F 0 "C14" H 5775 2450 50  0000 L CNN
+F 0 "C19" H 5775 2450 50  0000 L CNN
 F 1 "220pF" H 5775 2250 50  0000 L CNN
 F 2 "SFUSat:C_0402" H 5788 2200 50  0001 C CNN
@@
 $EndComp
 $Comp
-L C C15
+L C C20
 U 1 1 5871BA4C
 P 6050 2350
-F 0 "C15" H 6075 2450 50  0000 L CNN
+F 0 "C20" H 6075 2450 50  0000 L CNN
 F 1 "1nF" H 6075 2250 50  0000 L CNN
 F 2 "SFUSat:C_0402" H 6088 2200 50  0001 C CNN
@@
 $EndComp
 $Comp
-L C C16
+L C C21
 U 1 1 5871BAAB
 P 6350 2350
-F 0 "C16" H 6375 2450 50  0000 L CNN
+F 0 "C21" H 6375 2450 50  0000 L CNN
 F 1 "1uF" H 6375 2250 50  0000 L CNN
 F 2 "SFUSat:C_0402" H 6388 2200 50  0001 C CNN
@@
 $EndComp
 $Comp
-L GND #PWR025
+L GND #PWR030
 U 1 1 5871BAFA
 P 5750 2550
-F 0 "#PWR025" H 5750 2300 50  0001 C CNN
+F 0 "#PWR030" H 5750 2300 50  0001 C CNN
 F 1 "GND" H 5750 2400 50  0000 C CNN
 F 2 "" H 5750 2550 50  0000 C CNN
@@
 $EndComp
 $Comp
-L GND #PWR026
+L GND #PWR031
 U 1 1 5871BB16
 P 6050 2550
-F 0 "#PWR026" H 6050 2300 50  0001 C CNN
+F 0 "#PWR031" H 6050 2300 50  0001 C CNN
 F 1 "GND" H 6050 2400 50  0000 C CNN
 F 2 "" H 6050 2550 50  0000 C CNN
@@
 $EndComp
 $Comp
-L GND #PWR027
+L GND #PWR032
 U 1 1 5871BB32
 P 6350 2550
-F 0 "#PWR027" H 6350 2300 50  0001 C CNN
+F 0 "#PWR032" H 6350 2300 50  0001 C CNN
 F 1 "GND" H 6350 2400 50  0000 C CNN
 F 2 "" H 6350 2550 50  0000 C CNN
@@
 Connection ~ 5700 2900
 $Comp
-L C C13
+L C C18
 U 1 1 5871BCCF
 P 5150 2350
-F 0 "C13" H 5175 2450 50  0000 L CNN
+F 0 "C18" H 5175 2450 50  0000 L CNN
 F 1 "220pF" H 5175 2250 50  0000 L CNN
 F 2 "SFUSat:C_0402" H 5188 2200 50  0001 C CNN
@@
 $EndComp
 $Comp
-L C C12
+L C C17
 U 1 1 5871BD40
 P 4850 2350
-F 0 "C12" H 4875 2450 50  0000 L CNN
+F 0 "C17" H 4875 2450 50  0000 L CNN
 F 1 "10nF" H 4875 2250 50  0000 L CNN
 F 2 "SFUSat:C_0402" H 4888 2200 50  0001 C CNN
@@
 $EndComp
 $Comp
-L GND #PWR028
+L GND #PWR033
 U 1 1 5871BD81
 P 5150 2550
-F 0 "#PWR028" H 5150 2300 50  0001 C CNN
+F 0 "#PWR033" H 5150 2300 50  0001 C CNN
 F 1 "GND" H 5150 2400 50  0000 C CNN
 F 2 "" H 5150 2550 50  0000 C CNN
@@
 $EndComp
 $Comp
-L GND #PWR029
+L GND #PWR034
 U 1 1 5871BDA1
 P 4850 2550
-F 0 "#PWR029" H 4850 2300 50  0001 C CNN
+F 0 "#PWR034" H 4850 2300 50  0001 C CNN
 F 1 "GND" H 4850 2400 50  0000 C CNN
 F 2 "" H 4850 2550 50  0000 C CNN
@@
 	6400 3400 6400 3600
 $Comp
-L C C18
+L C C23
 U 1 1 5871C0B1
 P 7450 3200
-F 0 "C18" V 7300 3200 50  0000 C CNN
+F 0 "C23" V 7300 3200 50  0000 C CNN
 F 1 "3pF" V 7600 3200 50  0000 C CNN
 F 2 "SFUSat:C_0402" H 7488 3050 50  0001 C CNN
@@
 $EndComp
 $Comp
-L C C17
+L C C22
 U 1 1 5871C0F0
 P 7050 3350
-F 0 "C17" H 7075 3450 50  0000 L CNN
+F 0 "C22" H 7075 3450 50  0000 L CNN
 F 1 "8.2pF" H 7075 3250 50  0000 L CNN
 F 2 "SFUSat:C_0402" H 7088 3200 50  0001 C CNN
@@
 $EndComp
 $Comp
-L C C19
+L C C24
 U 1 1 5871C127
 P 7850 3350
-F 0 "C19" H 7875 3450 50  0000 L CNN
+F 0 "C24" H 7875 3450 50  0000 L CNN
 F 1 "8.2pF" H 7875 3250 50  0000 L CNN
 F 2 "SFUSat:C_0402" H 7888 3200 50  0001 C CNN
@@
 Connection ~ 7850 3200
 $Comp
-L GND #PWR030
+L GND #PWR035
 U 1 1 5871C376
 P 7050 3600
-F 0 "#PWR030" H 7050 3350 50  0001 C CNN
+F 0 "#PWR035" H 7050 3350 50  0001 C CNN
 F 1 "GND" H 7050 3450 50  0000 C CNN
 F 2 "" H 7050 3600 50  0000 C CNN
@@
 $EndComp
 $Comp
-L GND #PWR031
+L GND #PWR036
 U 1 1 5871C39E
 P 7850 3600
-F 0 "#PWR031" H 7850 3350 50  0001 C CNN
+F 0 "#PWR036" H 7850 3350 50  0001 C CNN
 F 1 "GND" H 7850 3450 50  0000 C CNN
 F 2 "" H 7850 3600 50  0000 C CNN
@@
 	7050 3500 7050 3600
 $Comp
-L R R6
+L R R5
 U 1 1 5871C966
 P 4500 4150
-F 0 "R6" V 4580 4150 50  0000 C CNN
+F 0 "R5" V 4580 4150 50  0000 C CNN
 F 1 "0" V 4500 4150 50  0000 C CNN
 F 2 "SFUSat:R_0402" V 4430 4150 50  0001 C CNN
@@
 $EndComp
 $Comp
-L GND #PWR032
+L GND #PWR037
 U 1 1 5871CA19
 P 4500 4400
-F 0 "#PWR032" H 4500 4150 50  0001 C CNN
+F 0 "#PWR037" H 4500 4150 50  0001 C CNN
 F 1 "GND" H 4500 4250 50  0000 C CNN
 F 2 "" H 4500 4400 50  0000 C CNN
@@
 	4500 4300 4500 4400
 $Comp
-L C C11
+L C C16
 U 1 1 5871CCE4
 P 4150 3850
-F 0 "C11" H 4175 3950 50  0000 L CNN
+F 0 "C16" H 4175 3950 50  0000 L CNN
 F 1 "4.7nF" H 4175 3750 50  0000 L CNN
 F 2 "SFUSat:C_0402" H 4188 3700 50  0001 C CNN
@@
 $EndComp
 $Comp
-L GND #PWR033
+L GND #PWR038
 U 1 1 5871CD23
 P 4150 4050
-F 0 "#PWR033" H 4150 3800 50  0001 C CNN
+F 0 "#PWR038" H 4150 3800 50  0001 C CNN
 F 1 "GND" H 4150 3900 50  0000 C CNN
 F 2 "" H 4150 4050 50  0000 C CNN
@@
 $EndComp
 $Comp
-L GND #PWR034
+L GND #PWR039
 U 1 1 587C3C45
 P 4650 6600
-F 0 "#PWR034" H 4650 6350 50  0001 C CNN
+F 0 "#PWR039" H 4650 6350 50  0001 C CNN
 F 1 "GND" H 4650 6450 50  0000 C CNN
 F 2 "" H 4650 6600 50  0000 C CNN
@@
 3V3
 $Comp
-L GND #PWR035
+L GND #PWR040
 U 1 1 58829BDE
 P 6400 6400
-F 0 "#PWR035" H 6400 6150 50  0001 C CNN
+F 0 "#PWR040" H 6400 6150 50  0001 C CNN
 F 1 "GND" H 6400 6250 50  0000 C CNN
 F 2 "" H 6400 6400 50  0000 C CNN
@@
 LNA and PA can be bypassed if\n BYP in pulled HIGH. Good as a \nkill switch to high power output.\n
 $Comp
-L CONN_01X03 P3
+L CONN_01X03 P2
 U 1 1 5881FCF5
 P 3900 6300
-F 0 "P3" H 3900 6500 50  0000 C CNN
+F 0 "P2" H 3900 6500 50  0000 C CNN
 F 1 "CONN_01X03" V 4000 6300 50  0000 C CNN
 F 2 "SFUSat:Socket_Strip_Straight_1x03" H 3900 6300 50  0001 C CNN
@@
 F 0 "W2" H 4300 6320 50  0000 C CNN
 F 1 "TEST_1P" H 4300 6250 50  0000 C CNN
-F 2 "SFUSat:EXPOSED" H 4500 6050 50  0001 C CNN
+F 2 "SFUSat:Measurement_Point_Round-SMD-Pad_Big" H 4500 6050 50  0001 C CNN
 F 3 "" H 4500 6050 50  0000 C CNN
 	1    4300 6050
@@
 Connection ~ 4550 2200
 $Comp
-L CONN_01X03 P?
+L CONN_01X03 P3
 U 1 1 592E3D25
 P 6100 6300
-F 0 "P?" H 6100 6500 50  0000 C CNN
+F 0 "P3" H 6100 6500 50  0000 C CNN
 F 1 "CONN_01X03" V 6200 6300 50  0000 C CNN
 F 2 "SFUSat:Socket_Strip_Straight_1x03" H 6100 6300 50  0001 C CNN
@@
 	4650 5700 4650 5800
 $Comp
-L R R?
+L R R6
 U 1 1 592E46FC
 P 4550 2950
-F 0 "R?" V 4630 2950 50  0000 C CNN
+F 0 "R6" V 4630 2950 50  0000 C CNN
 F 1 "1k" V 4550 2950 50  0000 C CNN
-F 2 "" V 4480 2950 50  0001 C CNN
+F 2 "SFUSat:R_0402" V 4480 2950 50  0001 C CNN
 F 3 "" H 4550 2950 50  0001 C CNN
 	1    4550 2950
