File: LB_XCVR.sch (KiCad schematic (older format))
At the start: 25 parts, among them J7 SMA, J8 SMA, J9 SMA, U2 CC1101-Q1, U3 0433BM15A0001, U4 SINGLE_0402, U5 SKY13372-467LF, U6 SINGLE_0402, U7 SINGLE_0402, X1 NX3225GA

Commit message: included all new sfusat libraries
Parts:
- X1: Frequency (none) -> 26MHz
Changed lines of the file:
@@
 LIBS:valves
 LIBS:SFUSat
+LIBS:SFUSat-Radio-cache
 EELAYER 25 0
 EELAYER END
 $Descr A4 11693 8268
 encoding utf-8
-Sheet 2 6
+Sheet 6 6
 Title ""
 Date ""
@@
 F 2 "SFUSat:NX3225GA" H 1600 3550 60  0001 C CNN
 F 3 "" H 1600 3550 60  0001 C CNN
+F 4 "26MHz" V 1600 3550 60  0001 C CNN "Frequency"
 	1    1600 3550
 	0    1    1    0

Commit message: Replaced SMA with u.fl for debug ports
Parts:
- J7, J8, J9: footprint SFUSat:SMA-Vert-TH -> SFUSat:UFL-R-SMT-1-Coaxial-Connector; Digikey (none) -> H9161-ND
Changed lines of the file:
@@
 LIBS:valves
 LIBS:SFUSat
+LIBS:SFUSat-cap
+LIBS:SFUSat-ind
+LIBS:SFUSat-res
 LIBS:SFUSat-Radio-cache
 EELAYER 25 0
@@
 F 0 "J7" H 7400 2750 60  0000 C CNN
 F 1 "SMA" H 7450 3100 60  0000 C CNN
-F 2 "SFUSat:SMA-Vert-TH" H 7650 3000 60  0001 C CNN
+F 2 "SFUSat:UFL-R-SMT-1-Coaxial-Connector" H 7650 3000 60  0001 C CNN
 F 3 "" H 7650 3000 60  0000 C CNN
+F 4 "H9161-ND" H 7450 2950 60  0001 C CNN "Digikey"
 	1    7450 2950
 	0    -1   -1   0
@@
 F 0 "J9" H 9975 2500 60  0000 C CNN
 F 1 "SMA" H 10025 2850 60  0000 C CNN
-F 2 "SFUSat:SMA-Vert-TH" H 10225 2750 60  0001 C CNN
+F 2 "SFUSat:UFL-R-SMT-1-Coaxial-Connector" H 10225 2750 60  0001 C CNN
 F 3 "" H 10225 2750 60  0000 C CNN
+F 4 "H9161-ND" H 10025 2700 60  0001 C CNN "Digikey"
 	1    10025 2700
 	0    -1   -1   0
@@
 F 0 "J8" H 9875 4700 60  0000 C CNN
 F 1 "SMA" H 9925 5050 60  0000 C CNN
-F 2 "SFUSat:SMA-Vert-TH" H 10125 4950 60  0001 C CNN
+F 2 "SFUSat:UFL-R-SMT-1-Coaxial-Connector" H 10125 4950 60  0001 C CNN
 F 3 "" H 10125 4950 60  0000 C CNN
+F 4 "H9161-ND" H 9925 4900 60  0001 C CNN "Digikey"
 	1    9925 4900
 	0    1    1    0

Commit message: consolidated PA to one sch for both bands
Parts:
- added J?: SMA, SFUSat:UFL-R-SMT-1-Coaxial-Connector, symbol SMA
Connections:
- wire segments 55 -> 56
Changed lines of the file:
@@
 $Descr A4 11693 8268
 encoding utf-8
-Sheet 6 6
+Sheet 6 7
 Title ""
 Date ""
@@
 TX
 $Comp
-L GND #PWR013
+L GND #PWR063
 U 1 1 58748992
 P 8725 4525
-F 0 "#PWR013" H 8725 4275 50  0001 C CNN
+F 0 "#PWR063" H 8725 4275 50  0001 C CNN
 F 1 "GND" H 8725 4375 50  0000 C CNN
 F 2 "" H 8725 4525 50  0000 C CNN
@@
 $EndComp
 $Comp
-L GND #PWR014
+L GND #PWR064
 U 1 1 5883AD14
 P 9000 3225
-F 0 "#PWR014" H 9000 2975 50  0001 C CNN
+F 0 "#PWR064" H 9000 2975 50  0001 C CNN
 F 1 "GND" H 9000 3075 50  0000 C CNN
 F 2 "" H 9000 3225 50  0000 C CNN
@@
 $EndComp
 $Comp
-L GND #PWR015
+L GND #PWR065
 U 1 1 592A76F5
 P 3525 5025
-F 0 "#PWR015" H 3525 4775 50  0001 C CNN
+F 0 "#PWR065" H 3525 4775 50  0001 C CNN
 F 1 "GND" H 3525 4875 50  0000 C CNN
 F 2 "" H 3525 5025 50  0000 C CNN
@@
 $EndComp
 $Comp
-L GND #PWR016
+L GND #PWR066
 U 1 1 592A8C09
 P 4125 5450
-F 0 "#PWR016" H 4125 5200 50  0001 C CNN
+F 0 "#PWR066" H 4125 5200 50  0001 C CNN
 F 1 "GND" H 4125 5300 50  0000 C CNN
 F 2 "" H 4125 5450 50  0000 C CNN
@@
 $EndComp
 $Comp
-L GND #PWR017
+L GND #PWR067
 U 1 1 592ACEFE
 P 5325 4575
-F 0 "#PWR017" H 5325 4325 50  0001 C CNN
+F 0 "#PWR067" H 5325 4325 50  0001 C CNN
 F 1 "GND" H 5325 4425 50  0000 C CNN
 F 2 "" H 5325 4575 50  0000 C CNN
@@
 $EndComp
 $Comp
-L GND #PWR018
+L GND #PWR068
 U 1 1 592AD242
 P 6300 4475
-F 0 "#PWR018" H 6300 4225 50  0001 C CNN
+F 0 "#PWR068" H 6300 4225 50  0001 C CNN
 F 1 "GND" H 6300 4325 50  0000 C CNN
 F 2 "" H 6300 4475 50  0000 C CNN
@@
 $EndComp
 $Comp
-L GND #PWR019
+L GND #PWR069
 U 1 1 592AE8E9
 P 2900 2275
-F 0 "#PWR019" H 2900 2025 50  0001 C CNN
+F 0 "#PWR069" H 2900 2025 50  0001 C CNN
 F 1 "GND" H 2900 2125 50  0000 C CNN
 F 2 "" H 2900 2275 50  0000 C CNN
@@
 $EndComp
 $Comp
-L GND #PWR020
+L GND #PWR070
 U 1 1 592A789E
 P 1000 3250
-F 0 "#PWR020" H 1000 3000 50  0001 C CNN
+F 0 "#PWR070" H 1000 3000 50  0001 C CNN
 F 1 "GND" H 1000 3100 50  0000 C CNN
 F 2 "" H 1000 3250 50  0000 C CNN
@@
 $EndComp
 $Comp
-L GND #PWR021
+L GND #PWR071
 U 1 1 592A7939
 P 1000 3850
-F 0 "#PWR021" H 1000 3600 50  0001 C CNN
+F 0 "#PWR071" H 1000 3600 50  0001 C CNN
 F 1 "GND" H 1000 3700 50  0000 C CNN
 F 2 "" H 1000 3850 50  0000 C CNN
@@
 $EndComp
 $Comp
-L GND #PWR022
+L GND #PWR072
 U 1 1 592AD916
 P 7550 3250
-F 0 "#PWR022" H 7550 3000 50  0001 C CNN
+F 0 "#PWR072" H 7550 3000 50  0001 C CNN
 F 1 "GND" H 7550 3100 50  0000 C CNN
 F 2 "" H 7550 3250 50  0000 C CNN
@@
 $EndComp
 $Comp
-L GND #PWR023
+L GND #PWR073
 U 1 1 592AE228
 P 10125 3000
-F 0 "#PWR023" H 10125 2750 50  0001 C CNN
+F 0 "#PWR073" H 10125 2750 50  0001 C CNN
 F 1 "GND" H 10125 2850 50  0000 C CNN
 F 2 "" H 10125 3000 50  0000 C CNN
@@
 $EndComp
 $Comp
-L GND #PWR024
+L GND #PWR074
 U 1 1 592AEC08
 P 9825 4600
-F 0 "#PWR024" H 9825 4350 50  0001 C CNN
+F 0 "#PWR074" H 9825 4350 50  0001 C CNN
 F 1 "GND" H 9825 4450 50  0000 C CNN
 F 2 "" H 9825 4600 50  0000 C CNN
@@
 $EndComp
 $Comp
-L GND #PWR025
+L GND #PWR075
 U 1 1 592F1736
 P 2900 1400
-F 0 "#PWR025" H 2900 1150 50  0001 C CNN
+F 0 "#PWR075" H 2900 1150 50  0001 C CNN
 F 1 "GND" H 2900 1250 50  0000 C CNN
 F 2 "" H 2900 1400 50  0000 C CNN
@@
 $EndComp
 $Comp
-L GND #PWR026
+L GND #PWR076
 U 1 1 592F173C
 P 2900 1825
-F 0 "#PWR026" H 2900 1575 50  0001 C CNN
+F 0 "#PWR076" H 2900 1575 50  0001 C CNN
 F 1 "GND" H 2900 1675 50  0000 C CNN
 F 2 "" H 2900 1825 50  0000 C CNN
@@
 $EndComp
 $Comp
-L GND #PWR027
+L GND #PWR077
 U 1 1 592F1E87
 P 4850 2700
-F 0 "#PWR027" H 4850 2450 50  0001 C CNN
+F 0 "#PWR077" H 4850 2450 50  0001 C CNN
 F 1 "GND" H 4850 2550 50  0000 C CNN
 F 2 "" H 4850 2700 50  0000 C CNN
@@
 $EndComp
 $Comp
-L GND #PWR028
+L GND #PWR078
 U 1 1 592F1E8D
 P 4850 2275
-F 0 "#PWR028" H 4850 2025 50  0001 C CNN
+F 0 "#PWR078" H 4850 2025 50  0001 C CNN
 F 1 "GND" H 4850 2125 50  0000 C CNN
 F 2 "" H 4850 2275 50  0000 C CNN
@@
 $EndComp
 $Comp
-L GND #PWR029
+L GND #PWR079
 U 1 1 593C6ADB
 P 6900 1725
-F 0 "#PWR029" H 6900 1475 50  0001 C CNN
+F 0 "#PWR079" H 6900 1475 50  0001 C CNN
 F 1 "GND" H 6900 1575 50  0000 C CNN
 F 2 "" H 6900 1725 50  0001 C CNN
@@
 Wire Wire Line
 	6750 3800 7250 3800
+$Comp
+L SMA J?
+U 1 1 5A9FAB32
+P 7000 4450
+F 0 "J?" H 6950 4250 60  0000 C CNN
+F 1 "SMA" H 7000 4600 60  0000 C CNN
+F 2 "SFUSat:UFL-R-SMT-1-Coaxial-Connector" H 7200 4500 60  0001 C CNN
+F 3 "" H 7200 4500 60  0000 C CNN
+F 4 "H9161-ND" H 7000 4450 60  0001 C CNN "Digikey"
+	1    7000 4450
+	0    1    1    0
+$EndComp
+$Comp
+L GND #PWR080
+U 1 1 5A9FABED
+P 7050 4150
+F 0 "#PWR080" H 7050 3900 50  0001 C CNN
+F 1 "GND" H 7050 4000 50  0000 C CNN
+F 2 "" H 7050 4150 50  0000 C CNN
+F 3 "" H 7050 4150 50  0000 C CNN
+	1    7050 4150
+	-1   0    0    1
+$EndComp
+Wire Wire Line
+	6900 4150 6900 3800
+Connection ~ 6900 3800
 $EndSCHEMATC
