File: LNA.sch (KiCad schematic (older format))
At the start: 16 parts

Commit message: consolidated PA to one sch for both bands
Connections:
- net labels added: 5V0
- net labels removed: LNA_5V0
Changed lines of the file:
@@
 $Descr A4 11693 8268
 encoding utf-8
-Sheet 3 6
+Sheet 3 7
 Title ""
 Date ""
@@
 $EndComp
 $Comp
-L GND #PWR?
+L GND #PWR039
 U 1 1 5A585C68
 P 5175 4875
-F 0 "#PWR?" H 5175 4625 50  0001 C CNN
+F 0 "#PWR039" H 5175 4625 50  0001 C CNN
 F 1 "GND" H 5175 4725 50  0000 C CNN
 F 2 "" H 5175 4875 50  0000 C CNN
@@
 $EndComp
 $Comp
-L GND #PWR?
+L GND #PWR040
 U 1 1 5A585C82
 P 6700 3450
-F 0 "#PWR?" H 6700 3200 50  0001 C CNN
+F 0 "#PWR040" H 6700 3200 50  0001 C CNN
 F 1 "GND" H 6700 3300 50  0000 C CNN
 F 2 "" H 6700 3450 50  0000 C CNN
@@
 $EndComp
 $Comp
-L GND #PWR?
+L GND #PWR041
 U 1 1 5A585C92
 P 6325 3450
-F 0 "#PWR?" H 6325 3200 50  0001 C CNN
+F 0 "#PWR041" H 6325 3200 50  0001 C CNN
 F 1 "GND" H 6325 3300 50  0000 C CNN
 F 2 "" H 6325 3450 50  0000 C CNN
@@
 $EndComp
 $Comp
-L GND #PWR?
+L GND #PWR042
 U 1 1 5A585CA2
 P 4675 3450
-F 0 "#PWR?" H 4675 3200 50  0001 C CNN
+F 0 "#PWR042" H 4675 3200 50  0001 C CNN
 F 1 "GND" H 4675 3300 50  0000 C CNN
 F 2 "" H 4675 3450 50  0000 C CNN
@@
 $EndComp
 $Comp
-L GND #PWR?
+L GND #PWR043
 U 1 1 5A585CB2
 P 4300 3450
-F 0 "#PWR?" H 4300 3200 50  0001 C CNN
+F 0 "#PWR043" H 4300 3200 50  0001 C CNN
 F 1 "GND" H 4300 3300 50  0000 C CNN
 F 2 "" H 4300 3450 50  0000 C CNN
@@
 $EndComp
 Text HLabel 5300 2425 2    60   Input ~ 0
-LNA_5V0
+5V0
 $Comp
 L C C?
@@
 $EndComp
 $Comp
-L GND #PWR?
+L GND #PWR044
 U 1 1 5A585CF1
 P 4350 5100
-F 0 "#PWR?" H 4350 4850 50  0001 C CNN
+F 0 "#PWR044" H 4350 4850 50  0001 C CNN
 F 1 "GND" H 4350 4950 50  0000 C CNN
 F 2 "" H 4350 5100 50  0000 C CNN
@@
 $EndComp
 $Comp
-L GND #PWR?
+L GND #PWR045
 U 1 1 5A585D01
 P 3975 5100
-F 0 "#PWR?" H 3975 4850 50  0001 C CNN
+F 0 "#PWR045" H 3975 4850 50  0001 C CNN
 F 1 "GND" H 3975 4950 50  0000 C CNN
 F 2 "" H 3975 5100 50  0000 C CNN

Commit message: layed out upper band and lower band schematic. Need to add a 2W rated SPDT switch to connect the RX and TX stages together before the diplexer
Parts:
- added J?: SMA, SFUSat:UFL-R-SMT-1-Coaxial-Connector, symbol SMA
- added U?: SINGLE_0402, SFUSat:SINGLE_0402, symbol SINGLE_0402
Connections:
- wire segments 35 -> 46
Other:
- moved on the sheet: C?
Changed lines of the file:
@@
 L C C?
 U 1 1 5A585C61
-P 7075 4200
-F 0 "C?" V 6950 4200 50  0000 C BNN
-F 1 "100pF" V 7200 4200 50  0000 C TNN
-F 2 "SFUSat:C_0402" H 7113 4050 50  0001 C CNN
-F 3 "" H 7075 4200 50  0000 C CNN
-F 4 "GRM1555C1H101JA01D" V 7075 4200 60  0001 C CNN "Part Number"
-F 5 "490-5922-1-ND" V 7075 4200 60  0001 C CNN "Digi-Key"
-F 6 "81-GRM1555C1H101JA1D" V 7075 4200 60  0001 C CNN "Mouser"
-	1    7075 4200
+P 7525 4200
+F 0 "C?" V 7400 4200 50  0000 C BNN
+F 1 "100pF" V 7650 4200 50  0000 C TNN
+F 2 "SFUSat:C_0402" H 7563 4050 50  0001 C CNN
+F 3 "" H 7525 4200 50  0000 C CNN
+F 4 "GRM1555C1H101JA01D" V 7525 4200 60  0001 C CNN "Part Number"
+F 5 "490-5922-1-ND" V 7525 4200 60  0001 C CNN "Digi-Key"
+F 6 "81-GRM1555C1H101JA1D" V 7525 4200 60  0001 C CNN "Mouser"
+	1    7525 4200
 	0    1    1    0
 $EndComp
@@
 $EndComp
 Wire Wire Line
-	5175 2800 5175 3025
+	5175 2800 5175 2900
+Wire Wire Line
+	5175 2900 5175 3025
 Wire Wire Line
 	5175 2425 5175 2500
@@
 	4400 3875 4525 3875
 Wire Wire Line
-	3850 3875 4100 3875
+	3850 3875 3975 3875
+Wire Wire Line
+	3975 3875 4100 3875
 Connection ~ 3975 4550
 Wire Wire Line
 	3975 4050 3975 3875
 Wire Wire Line
-	3975 4350 3975 4675
+	3975 4350 3975 4550
+Wire Wire Line
+	3975 4550 3975 4675
 Connection ~ 6325 2900
 Connection ~ 5950 2900
@@
 Connection ~ 5175 2900
 Wire Wire Line
-	4300 2900 6700 2900
+	4300 2900 4675 2900
+Wire Wire Line
+	4675 2900 5175 2900
+Wire Wire Line
+	5175 2900 5950 2900
+Wire Wire Line
+	5950 2900 6325 2900
+Wire Wire Line
+	6325 2900 6700 2900
 Wire Wire Line
 	3550 3875 3425 3875
@@
 	4525 4550 4525 4200
 Wire Wire Line
-	3975 4550 4525 4550
+	3975 4550 4350 4550
+Wire Wire Line
+	4350 4550 4525 4550
 Wire Wire Line
 	4350 4675 4350 4550
@@
 	4525 3875 4525 4000
 Wire Wire Line
-	7225 4200 7350 4200
+	7675 4200 7925 4200
 Wire Wire Line
 	5950 2900 5950 3025
@@
 Connection ~ 5950 4200
 Wire Wire Line
-	5950 3325 5950 4200
+	5950 3325 5950 4100
+Wire Wire Line
+	5950 4100 5950 4200
 Wire Wire Line
 	5175 3450 5175 3325
@@
 	5825 4100 5950 4100
 Wire Wire Line
-	5825 4200 6925 4200
+	5825 4200 5950 4200
+Wire Wire Line
+	5950 4200 6800 4200
+Wire Wire Line
+	6800 4200 7375 4200
 Wire Wire Line
 	6800 4425 6800 4200
@@
 Text HLabel 3425 3875 0    60   Input ~ 0
 IN
-Text HLabel 7350 4200 2    60   Input ~ 0
+Text HLabel 7925 4200 2    60   Input ~ 0
 OUT
+$Comp
+L SMA J?
+U 1 1 5AB879E9
+P 7575 3350
+F 0 "J?" H 7525 3150 60  0000 C CNN
+F 1 "SMA" H 7575 3500 60  0000 C CNN
+F 2 "SFUSat:UFL-R-SMT-1-Coaxial-Connector" H 7775 3400 60  0001 C CNN
+F 3 "" H 7775 3400 60  0000 C CNN
+F 4 "H9161-ND" H 7575 3350 60  0001 C CNN "Digikey"
+	1    7575 3350
+	0    -1   -1   0
+$EndComp
+$Comp
+L SINGLE_0402 U?
+U 1 1 5AB879F0
+P 7525 3900
+F 0 "U?" V 7525 3825 60  0000 R CNN
+F 1 "SINGLE_0402" H 7525 3800 60  0001 C TNN
+F 2 "SFUSat:SINGLE_0402" H 7525 3900 60  0001 C CNN
+F 3 "" H 7525 3900 60  0001 C CNN
+	1    7525 3900
+	0    1    1    0
+$EndComp
+$Comp
+L GND #PWR?
+U 1 1 5AB879F7
+P 7675 3650
+F 0 "#PWR?" H 7675 3400 50  0001 C CNN
+F 1 "GND" H 7675 3500 50  0000 C CNN
+F 2 "" H 7675 3650 50  0000 C CNN
+F 3 "" H 7675 3650 50  0000 C CNN
+	1    7675 3650
+	1    0    0    -1
+$EndComp
 $EndSCHEMATC
