File: LNA.sch (KiCad schematic (older format))
At the start: 18 parts

Commit message: Fixed rescue-lib components and CONN_02X05
Connections:
- wire segments 46 -> 35
Changed lines of the file:
@@
 $Descr A4 11693 8268
 encoding utf-8
-Sheet 3 15
+Sheet 3 14
 Title ""
 Date ""
@@
 $EndComp
 Wire Wire Line
-	5175 2800 5175 2900
-Wire Wire Line
-	5175 2900 5175 3025
+	5175 2800 5175 3025
 Wire Wire Line
 	5175 2425 5175 2500
@@
 	4400 3875 4525 3875
 Wire Wire Line
-	3850 3875 3975 3875
-Wire Wire Line
-	3975 3875 4100 3875
+	3850 3875 4100 3875
 Connection ~ 3975 4550
 Wire Wire Line
 	3975 4050 3975 3875
 Wire Wire Line
-	3975 4350 3975 4550
-Wire Wire Line
-	3975 4550 3975 4675
+	3975 4350 3975 4675
 Connection ~ 6325 2900
 Connection ~ 5950 2900
@@
 Connection ~ 5175 2900
 Wire Wire Line
-	4300 2900 4675 2900
-Wire Wire Line
-	4675 2900 5175 2900
-Wire Wire Line
-	5175 2900 5950 2900
-Wire Wire Line
-	5950 2900 6325 2900
-Wire Wire Line
-	6325 2900 6700 2900
+	4300 2900 6700 2900
 Wire Wire Line
 	3550 3875 3425 3875
@@
 	4525 4550 4525 4200
 Wire Wire Line
-	3975 4550 4350 4550
-Wire Wire Line
-	4350 4550 4525 4550
+	3975 4550 4525 4550
 Wire Wire Line
 	4350 4675 4350 4550
@@
 Connection ~ 5950 4200
 Wire Wire Line
-	5950 3325 5950 4100
-Wire Wire Line
-	5950 4100 5950 4200
+	5950 3325 5950 4200
 Wire Wire Line
 	5175 3450 5175 3325
@@
 	5825 4100 5950 4100
 Wire Wire Line
-	5825 4200 5950 4200
-Wire Wire Line
-	5950 4200 6800 4200
-Wire Wire Line
-	6800 4200 7375 4200
+	5825 4200 7375 4200
 Wire Wire Line
 	6800 4425 6800 4200

Commit message: Annotated the schematics
Parts:
- gave numbers to parts that had none: 18
Changed lines of the file:
@@
 $EndDescr
 $Comp
-L R R?
+L R R7
 U 1 1 5A585C57
 P 6525 4425
-F 0 "R?" V 6450 4425 50  0000 C BNN
+F 0 "R7" V 6450 4425 50  0000 C BNN
 F 1 "100" V 6525 4425 50  0000 C CNN
 F 2 "SFUSat:R_0402" V 6455 4425 50  0001 C CNN
@@
 $EndComp
 $Comp
-L C C?
+L C C11
 U 1 1 5A585C61
 P 7525 4200
-F 0 "C?" V 7400 4200 50  0000 C BNN
+F 0 "C11" V 7400 4200 50  0000 C BNN
 F 1 "100pF" V 7650 4200 50  0000 C TNN
 F 2 "SFUSat:C_0402" H 7563 4050 50  0001 C CNN
@@
 $EndComp
 $Comp
-L GND #PWR039
+L GND #PWR47
 U 1 1 5A585C68
 P 5175 4875
-F 0 "#PWR039" H 5175 4625 50  0001 C CNN
+F 0 "#PWR47" H 5175 4625 50  0001 C CNN
 F 1 "GND" H 5175 4725 50  0000 C CNN
 F 2 "" H 5175 4875 50  0000 C CNN
@@
 $EndComp
 $Comp
-L L L?
+L L L3
 U 1 1 5A585C71
 P 5950 3175
-F 0 "L?" H 5925 3175 50  0000 R CNN
+F 0 "L3" H 5925 3175 50  0000 R CNN
 F 1 "24nH" H 6000 3175 50  0000 L CNN
 F 2 "SFUSat:L_0402" H 5950 3175 50  0001 C CNN
@@
 $EndComp
 $Comp
-L C C?
+L C C10
 U 1 1 5A585C7B
 P 6700 3175
-F 0 "C?" H 6725 3275 50  0000 L CNN
+F 0 "C10" H 6725 3275 50  0000 L CNN
 F 1 "0.1uF" H 6725 3075 50  0000 L CNN
 F 2 "SFUSat:C_0402" H 6738 3025 50  0001 C CNN
@@
 $EndComp
 $Comp
-L GND #PWR040
+L GND #PWR49
 U 1 1 5A585C82
 P 6700 3450
-F 0 "#PWR040" H 6700 3200 50  0001 C CNN
+F 0 "#PWR49" H 6700 3200 50  0001 C CNN
 F 1 "GND" H 6700 3300 50  0000 C CNN
 F 2 "" H 6700 3450 50  0000 C CNN
@@
 $EndComp
 $Comp
-L C C?
+L C C9
 U 1 1 5A585C8B
 P 6325 3175
-F 0 "C?" H 6350 3275 50  0000 L CNN
+F 0 "C9" H 6350 3275 50  0000 L CNN
 F 1 "390pF" H 6350 3075 50  0000 L CNN
 F 2 "SFUSat:C_0402" H 6363 3025 50  0001 C CNN
@@
 $EndComp
 $Comp
-L GND #PWR041
+L GND #PWR48
 U 1 1 5A585C92
 P 6325 3450
-F 0 "#PWR041" H 6325 3200 50  0001 C CNN
+F 0 "#PWR48" H 6325 3200 50  0001 C CNN
 F 1 "GND" H 6325 3300 50  0000 C CNN
 F 2 "" H 6325 3450 50  0000 C CNN
@@
 $EndComp
 $Comp
-L C C?
+L C C7
 U 1 1 5A585C9B
 P 4675 3175
-F 0 "C?" H 4700 3275 50  0000 L CNN
+F 0 "C7" H 4700 3275 50  0000 L CNN
 F 1 "56pF" H 4700 3075 50  0000 L CNN
 F 2 "SFUSat:C_0402" H 4713 3025 50  0001 C CNN
@@
 $EndComp
 $Comp
-L GND #PWR042
+L GND #PWR46
 U 1 1 5A585CA2
 P 4675 3450
-F 0 "#PWR042" H 4675 3200 50  0001 C CNN
+F 0 "#PWR46" H 4675 3200 50  0001 C CNN
 F 1 "GND" H 4675 3300 50  0000 C CNN
 F 2 "" H 4675 3450 50  0000 C CNN
@@
 $EndComp
 $Comp
-L C C?
+L C C5
 U 1 1 5A585CAB
 P 4300 3175
-F 0 "C?" H 4325 3275 50  0000 L CNN
+F 0 "C5" H 4325 3275 50  0000 L CNN
 F 1 "0.01uF" H 4325 3075 50  0000 L CNN
 F 2 "SFUSat:C_0402" H 4338 3025 50  0001 C CNN
@@
 $EndComp
 $Comp
-L GND #PWR043
+L GND #PWR44
 U 1 1 5A585CB2
 P 4300 3450
-F 0 "#PWR043" H 4300 3200 50  0001 C CNN
+F 0 "#PWR44" H 4300 3200 50  0001 C CNN
 F 1 "GND" H 4300 3300 50  0000 C CNN
 F 2 "" H 4300 3450 50  0000 C CNN
@@
 $EndComp
 $Comp
-L R R?
+L R R6
 U 1 1 5A585CBB
 P 5175 3175
-F 0 "R?" H 5100 3175 50  0000 R CNN
+F 0 "R6" H 5100 3175 50  0000 R CNN
 F 1 "1210" V 5175 3175 50  0000 C CNN
 F 2 "SFUSat:R_0402" V 5105 3175 50  0001 C CNN
@@
 5V0
 $Comp
-L C C?
+L C C3
 U 1 1 5A585CD6
 P 3700 3875
-F 0 "C?" V 3575 3875 50  0000 C BNN
+F 0 "C3" V 3575 3875 50  0000 C BNN
 F 1 "100pF" V 3825 3875 50  0000 C TNN
 F 2 "SFUSat:C_0402" H 3738 3725 50  0001 C CNN
@@
 $EndComp
 $Comp
-L MML09211H U?
+L MML09211H U5
 U 1 1 5A585CE0
 P 5175 4100
-F 0 "U?" H 5575 4600 60  0000 R BNN
+F 0 "U5" H 5575 4600 60  0000 R BNN
 F 1 "MML09211H" H 5725 3600 60  0000 R TNN
 F 2 "SFUSat:8-VFDFN" H 5075 4000 60  0001 C CNN
@@
 $EndComp
 $Comp
-L C C?
+L C C6
 U 1 1 5A585CEA
 P 4350 4825
-F 0 "C?" H 4375 4925 50  0000 L CNN
+F 0 "C6" H 4375 4925 50  0000 L CNN
 F 1 "0.01uF" H 4375 4725 50  0000 L CNN
 F 2 "SFUSat:C_0402" H 4388 4675 50  0001 C CNN
@@
 $EndComp
 $Comp
-L GND #PWR044
+L GND #PWR45
 U 1 1 5A585CF1
 P 4350 5100
-F 0 "#PWR044" H 4350 4850 50  0001 C CNN
+F 0 "#PWR45" H 4350 4850 50  0001 C CNN
 F 1 "GND" H 4350 4950 50  0000 C CNN
 F 2 "" H 4350 5100 50  0000 C CNN
@@
 $EndComp
 $Comp
-L C C?
+L C C4
 U 1 1 5A585CFA
 P 3975 4825
-F 0 "C?" H 4000 4925 50  0000 L CNN
+F 0 "C4" H 4000 4925 50  0000 L CNN
 F 1 "390pF" H 4000 4725 50  0000 L CNN
 F 2 "SFUSat:C_0402" H 4013 4675 50  0001 C CNN
@@
 $EndComp
 $Comp
-L GND #PWR045
+L GND #PWR43
 U 1 1 5A585D01
 P 3975 5100
-F 0 "#PWR045" H 3975 4850 50  0001 C CNN
+F 0 "#PWR43" H 3975 4850 50  0001 C CNN
 F 1 "GND" H 3975 4950 50  0000 C CNN
 F 2 "" H 3975 5100 50  0000 C CNN
@@
 $EndComp
 $Comp
-L L L?
+L L L2
 U 1 1 5A585D1A
 P 4250 3875
-F 0 "L?" V 4200 3875 50  0000 C CNN
+F 0 "L2" V 4200 3875 50  0000 C CNN
 F 1 "4.3nH" V 4325 3875 50  0000 C CNN
 F 2 "SFUSat:L_0402" H 4250 3875 50  0001 C CNN
@@
 NoConn ~ 4525 4100
 $Comp
-L R R?
+L R R5
 U 1 1 5A585D25
 P 5175 2650
-F 0 "R?" V 5255 2650 50  0000 C CNN
+F 0 "R5" V 5255 2650 50  0000 C CNN
 F 1 "0R05" V 5175 2650 50  0000 C CNN
 F 2 "SFUSat:C_0603" V 5105 2650 50  0001 C CNN
@@
 Ferrite bead, 220 Ohm @ 100MHz
 $Comp
-L L L?
+L L L1
 U 1 1 5A585D4B
 P 3975 4200
-F 0 "L?" H 4025 4275 50  0000 L BNN
+F 0 "L1" H 4025 4275 50  0000 L BNN
 F 1 "22nH" H 4025 4125 50  0000 L TNN
 F 2 "SFUSat:L_0402" H 3975 4200 50  0001 C CNN
@@
 $EndComp
 $Comp
-L C C?
+L C C8
 U 1 1 5A585D55
 P 6100 4425
-F 0 "C?" V 5975 4425 50  0000 C BNN
+F 0 "C8" V 5975 4425 50  0000 C BNN
 F 1 "56pF" V 6225 4425 50  0000 C TNN
 F 2 "SFUSat:C_0402" H 6138 4275 50  0001 C CNN
@@
 OUT
 $Comp
-L SMA J?
+L SMA J16
 U 1 1 5AB879E9
 P 7575 3350
-F 0 "J?" H 7525 3150 60  0000 C CNN
+F 0 "J16" H 7525 3150 60  0000 C CNN
 F 1 "SMA" H 7575 3500 60  0000 C CNN
 F 2 "SFUSat:UFL-R-SMT-1-Coaxial-Connector" H 7775 3400 60  0001 C CNN
@@
 $EndComp
 $Comp
-L SINGLE_0402 U?
+L SINGLE_0402 U6
 U 1 1 5AB879F0
 P 7525 3900
-F 0 "U?" V 7525 3825 60  0000 R CNN
+F 0 "U6" V 7525 3825 60  0000 R CNN
 F 1 "SINGLE_0402" H 7525 3800 60  0001 C TNN
 F 2 "SFUSat:SINGLE_0402" H 7525 3900 60  0001 C CNN
@@
 $EndComp
 $Comp
-L GND #PWR?
+L GND #PWR50
 U 1 1 5AB879F7
 P 7675 3650
-F 0 "#PWR?" H 7675 3400 50  0001 C CNN
+F 0 "#PWR50" H 7675 3400 50  0001 C CNN
 F 1 "GND" H 7675 3500 50  0000 C CNN
 F 2 "" H 7675 3650 50  0000 C CNN
