File: LNA.sch (KiCad schematic (older format))
At the start: 18 parts, among them J16 SMA, U5 MML09211H, U6 SINGLE_0402

Commit message: Closes #58
Parts:
- C10: value 0.1uF -> 100nF
- C5, C6: value 0.01uF -> 10nF
Changed lines of the file:
@@
 $Descr A4 11693 8268
 encoding utf-8
-Sheet 3 15
+Sheet 2 15
 Title ""
 Date ""
@@
 P 6700 3175
 F 0 "C10" H 6725 3275 50  0000 L CNN
-F 1 "0.1uF" H 6725 3075 50  0000 L CNN
+F 1 "100nF" H 6725 3075 50  0000 L CNN
 F 2 "SFUSat:C_0402" H 6738 3025 50  0001 C CNN
 F 3 "" H 6700 3175 50  0000 C CNN
@@
 P 4300 3175
 F 0 "C5" H 4325 3275 50  0000 L CNN
-F 1 "0.01uF" H 4325 3075 50  0000 L CNN
+F 1 "10nF" H 4325 3075 50  0000 L CNN
 F 2 "SFUSat:C_0402" H 4338 3025 50  0001 C CNN
 F 3 "" H 4300 3175 50  0000 C CNN
@@
 P 4350 4825
 F 0 "C6" H 4375 4925 50  0000 L CNN
-F 1 "0.01uF" H 4375 4725 50  0000 L CNN
+F 1 "10nF" H 4375 4725 50  0000 L CNN
 F 2 "SFUSat:C_0402" H 4388 4675 50  0001 C CNN
 F 3 "" H 4350 4825 50  0000 C CNN

Commit message: Changed R5 value to 220R
Parts:
- R5: value 0R05 -> 220R
Changed lines of the file:
@@
 P 5175 2650
 F 0 "R5" V 5255 2650 50  0000 C CNN
-F 1 "0R05" V 5175 2650 50  0000 C CNN
+F 1 "220R" V 5175 2650 50  0000 C CNN
 F 2 "SFUSat:C_0603" V 5105 2650 50  0001 C CNN
 F 3 "" H 5175 2650 50  0001 C CNN
