File: PA.sch (KiCad schematic (older format))
At the start: 75 parts

Commit message: consolidated PA to one sch for both bands
Parts:
- removed C?: DNP, SFUSat:C_0402, symbol C
- removed C? (x2): 10pF, SFUSat:C_0402, symbol C
- removed C?: 27pF, SFUSat:C_0402, symbol C
- removed C?: 1.2pF, SFUSat:C_0402, symbol C
- removed C? (x2): 10uF, SFUSat:C_1210, symbol C
- removed C? (x5): 0.1uF, SFUSat:C_0402, symbol C
- removed C? (x2): 1uF, SFUSat:C_0402, symbol C
- removed C? (x2): 100pF, SFUSat:C_0402, symbol C
- removed C?: 22pF, SFUSat:C_0402, symbol C
- removed C?: 2.2uF, SFUSat:C_0402, symbol C
- removed D? (x4): PESD5Zx, SFUSat:PESD57zx, symbol PESD5Zx
- removed J? (x2): CONN_01X03, SFUSat:Socket_Strip_Straight_1x03, symbol CONN_01X03
- removed J? (x3): TEST_1P, SFUSat:Measurement_Point_Round-SMD-Pad_Big, symbol TEST_1P
- removed J?: CONN_01X02, SFUSat:2x01In_Header_v2, symbol CONN_01X02
- removed L? (x4): 0R0, SFUSat:L_0603, symbol L
- removed L?: 8.2nH, SFUSat:L_0402, symbol L
- removed L?: 12.55nH, SFUSat:L_0402, symbol L
- removed R? (x2): 1k, SFUSat:R_0402, symbol R
- removed R?: 287R, SFUSat:R_0402, symbol R
- removed R?: 1K, SFUSat:R_0402, symbol R
- removed U?: RT9183, SFUSat:TO-263-5Lead, symbol RT9183
- removed U?: TLV702, SFUSat:SOT_23_5, symbol TLV702
- removed U?: LTC2644, SFUSat:12-TSSOP, symbol LTC2644
- removed U?: SN74LVC1G17, SFUSat:SOT_23_5, symbol SN74LVC1G17
Connections:
- net labels added: GAIN
- net labels removed: G_DAC, G_MAN, MCU_PWM
- wire segments 192 -> 92
- no-connect marks 1 -> 0
Other:
- note removed: "430MHz"
- note removed: "PWM DAC"
- moved on the sheet: C?, J?, R?, RV?

Commit message: layed out upper band and lower band schematic. Need to add a 2W rated SPDT switch to connect the RX and TX stages together before the diplexer
Parts:
- gave numbers to parts that had none: 1
Changed lines of the file:
@@
 PA
 $Comp
-L RF6886 U?
+L RF6886 U201
 U 1 1 5A587750
 P 3600 3100
-F 0 "U?" H 3050 3750 60  0000 C CNN
+AR Path="/5A585E42/5A587750" Ref="U201"  Part="1"
+AR Path="/5A9CE314/5A587750" Ref="U201"  Part="1"
+F 0 "U201" H 3050 3750 60  0000 C CNN
 F 1 "RF6886" H 3600 3100 60  0000 C CNN
 F 2 "SFUSat:QFN-24" H 3600 2750 60  0001 C CNN
@@
 U 1 1 5A58777F
 P 1975 2850
+AR Path="/5A585E42/5A58777F" Ref="C?"  Part="1"
+AR Path="/5A9CE314/5A58777F" Ref="C?"  Part="1"
 F 0 "C?" H 2000 2950 50  0000 L CNN
 F 1 "2.2uF" H 2000 2750 50  0000 L CNN
@@
 U 1 1 5A587792
 P 3700 2100
+AR Path="/5A585E42/5A587792" Ref="#PWR046"  Part="1"
+AR Path="/5A9CE314/5A587792" Ref="#PWR046"  Part="1"
 F 0 "#PWR046" H 3700 1850 50  0001 C CNN
 F 1 "GND" H 3700 1950 50  0000 C CNN
@@
 U 1 1 5A587798
 P 3600 3875
+AR Path="/5A585E42/5A587798" Ref="#PWR047"  Part="1"
+AR Path="/5A9CE314/5A587798" Ref="#PWR047"  Part="1"
 F 0 "#PWR047" H 3600 3625 50  0001 C CNN
 F 1 "GND" H 3600 3725 50  0000 C CNN
@@
 U 1 1 5A5877A4
 P 1975 3050
+AR Path="/5A585E42/5A5877A4" Ref="#PWR048"  Part="1"
+AR Path="/5A9CE314/5A5877A4" Ref="#PWR048"  Part="1"
 F 0 "#PWR048" H 1975 2800 50  0001 C CNN
 F 1 "GND" H 1975 2900 50  0000 C CNN
@@
 U 1 1 5A5877AD
 P 1750 2650
+AR Path="/5A585E42/5A5877AD" Ref="R?"  Part="1"
+AR Path="/5A9CE314/5A5877AD" Ref="R?"  Part="1"
 F 0 "R?" V 1830 2650 50  0000 C CNN
 F 1 "220R" V 1750 2650 50  0000 C CNN
@@
 U 1 1 5A5877B7
 P 1225 2850
+AR Path="/5A585E42/5A5877B7" Ref="C?"  Part="1"
+AR Path="/5A9CE314/5A5877B7" Ref="C?"  Part="1"
 F 0 "C?" H 1250 2950 50  0000 L CNN
 F 1 "10uF" H 1250 2750 50  0000 L CNN
@@
 U 1 1 5A5877BE
 P 4500 1375
+AR Path="/5A585E42/5A5877BE" Ref="#PWR049"  Part="1"
+AR Path="/5A9CE314/5A5877BE" Ref="#PWR049"  Part="1"
 F 0 "#PWR049" H 4500 1125 50  0001 C CNN
 F 1 "GND" H 4500 1225 50  0000 C CNN
@@
 U 1 1 5A5877C4
 P 1325 3100
+AR Path="/5A585E42/5A5877C4" Ref="#PWR050"  Part="1"
+AR Path="/5A9CE314/5A5877C4" Ref="#PWR050"  Part="1"
 F 0 "#PWR050" H 1325 2850 50  0001 C CNN
 F 1 "GND" H 1325 2950 50  0000 C CNN
@@
 U 1 1 5A5877CD
 P 2400 2750
+AR Path="/5A585E42/5A5877CD" Ref="C?"  Part="1"
+AR Path="/5A9CE314/5A5877CD" Ref="C?"  Part="1"
 F 0 "C?" H 2425 2850 50  0000 L CNN
 F 1 "220pF" H 2425 2650 50  0000 L CNN
@@
 U 1 1 5A5877D4
 P 2400 2950
+AR Path="/5A585E42/5A5877D4" Ref="#PWR051"  Part="1"
+AR Path="/5A9CE314/5A5877D4" Ref="#PWR051"  Part="1"
 F 0 "#PWR051" H 2400 2700 50  0001 C CNN
 F 1 "GND" H 2400 2800 50  0000 C CNN
@@
 U 1 1 5A5877DD
 P 2950 1350
+AR Path="/5A585E42/5A5877DD" Ref="C?"  Part="1"
+AR Path="/5A9CE314/5A5877DD" Ref="C?"  Part="1"
 F 0 "C?" H 2975 1450 50  0000 L CNN
 F 1 "1uF" H 2975 1250 50  0000 L CNN
@@
 U 1 1 5A5877E4
 P 2950 2200
+AR Path="/5A585E42/5A5877E4" Ref="#PWR052"  Part="1"
+AR Path="/5A9CE314/5A5877E4" Ref="#PWR052"  Part="1"
 F 0 "#PWR052" H 2950 1950 50  0001 C CNN
 F 1 "GND" H 2950 2050 50  0000 C CNN
@@
 U 1 1 5A5877EA
 P 2950 1550
+AR Path="/5A585E42/5A5877EA" Ref="#PWR053"  Part="1"
+AR Path="/5A9CE314/5A5877EA" Ref="#PWR053"  Part="1"
 F 0 "#PWR053" H 2950 1300 50  0001 C CNN
 F 1 "GND" H 2950 1400 50  0000 C CNN
@@
 U 1 1 5A5877F3
 P 2600 1150
+AR Path="/5A585E42/5A5877F3" Ref="R?"  Part="1"
+AR Path="/5A9CE314/5A5877F3" Ref="R?"  Part="1"
 F 0 "R?" V 2680 1150 50  0000 C CNN
 F 1 "390R" V 2600 1150 50  0000 C CNN
@@
 U 1 1 5A587804
 P 3375 5775
+AR Path="/5A585E42/5A587804" Ref="U?"  Part="1"
+AR Path="/5A9CE314/5A587804" Ref="U?"  Part="1"
 F 0 "U?" H 3375 5925 50  0000 L CNN
 F 1 "LMV358" H 3375 5625 50  0000 L CNN
@@
 U 1 1 5A58780E
 P 2325 5875
+AR Path="/5A585E42/5A58780E" Ref="U?"  Part="1"
+AR Path="/5A9CE314/5A58780E" Ref="U?"  Part="1"
 F 0 "U?" H 2325 6025 50  0000 L CNN
 F 1 "LMV358" H 2325 5725 50  0000 L CNN
@@
 U 1 1 5A587818
 P 2850 5775
+AR Path="/5A585E42/5A587818" Ref="R?"  Part="1"
+AR Path="/5A9CE314/5A587818" Ref="R?"  Part="1"
 F 0 "R?" V 2930 5775 50  0000 C CNN
 F 1 "1K" V 2850 5775 50  0000 C CNN
@@
 U 1 1 5A587822
 P 3525 5275
+AR Path="/5A585E42/5A587822" Ref="R?"  Part="1"
+AR Path="/5A9CE314/5A587822" Ref="R?"  Part="1"
 F 0 "R?" V 3605 5275 50  0000 C CNN
 F 1 "10K" V 3525 5275 50  0000 C CNN
@@
 U 1 1 5A58782C
 P 3800 6100
+AR Path="/5A585E42/5A58782C" Ref="R?"  Part="1"
+AR Path="/5A9CE314/5A58782C" Ref="R?"  Part="1"
 F 0 "R?" V 3880 6100 50  0000 C CNN
 F 1 "10K" V 3800 6100 50  0000 C CNN
@@
 U 1 1 5A587836
 P 4075 5675
+AR Path="/5A585E42/5A587836" Ref="R?"  Part="1"
+AR Path="/5A9CE314/5A587836" Ref="R?"  Part="1"
 F 0 "R?" V 4155 5675 50  0000 C CNN
 F 1 "10K" V 4075 5675 50  0000 C CNN
@@
 U 1 1 5A587840
 P 4075 5875
+AR Path="/5A585E42/5A587840" Ref="R?"  Part="1"
+AR Path="/5A9CE314/5A587840" Ref="R?"  Part="1"
 F 0 "R?" V 4155 5875 50  0000 C CNN
 F 1 "10K" V 4075 5875 50  0000 C CNN
@@
 U 1 1 5A58784A
 P 2175 5275
+AR Path="/5A585E42/5A58784A" Ref="C?"  Part="1"
+AR Path="/5A9CE314/5A58784A" Ref="C?"  Part="1"
 F 0 "C?" H 2200 5375 50  0000 L CNN
 F 1 "0.1uF" H 2200 5175 50  0000 L CNN
@@
 U 1 1 5A587853
 P 2850 5350
+AR Path="/5A585E42/5A587853" Ref="#PWR054"  Part="1"
+AR Path="/5A9CE314/5A587853" Ref="#PWR054"  Part="1"
 F 0 "#PWR054" H 2850 5100 50  0001 C CNN
 F 1 "GND" H 2850 5200 50  0000 C CNN
@@
 U 1 1 5A587859
 P 3800 6300
+AR Path="/5A585E42/5A587859" Ref="#PWR055"  Part="1"
+AR Path="/5A9CE314/5A587859" Ref="#PWR055"  Part="1"
 F 0 "#PWR055" H 3800 6050 50  0001 C CNN
 F 1 "GND" H 3800 6150 50  0000 C CNN
@@
 U 1 1 5A58786F
 P 9175 3525
+AR Path="/5A585E42/5A58786F" Ref="RV?"  Part="1"
+AR Path="/5A9CE314/5A58786F" Ref="RV?"  Part="1"
 F 0 "RV?" V 9000 3525 50  0000 C CNN
 F 1 "POT" V 9075 3525 50  0000 C CNN
@@
 U 1 1 5A587879
 P 9175 3875
+AR Path="/5A585E42/5A587879" Ref="R?"  Part="1"
+AR Path="/5A9CE314/5A587879" Ref="R?"  Part="1"
 F 0 "R?" V 9255 3875 50  0000 C CNN
 F 1 "1K" V 9175 3875 50  0000 C CNN
@@
 U 1 1 5A587883
 P 9075 4350
+AR Path="/5A585E42/5A587883" Ref="#PWR056"  Part="1"
+AR Path="/5A9CE314/5A587883" Ref="#PWR056"  Part="1"
 F 0 "#PWR056" H 9075 4100 50  0001 C CNN
 F 1 "GND" H 9075 4200 50  0000 C CNN
@@
 U 1 1 5A5878F3
 P 2975 5600
+AR Path="/5A585E42/5A5878F3" Ref="J?"  Part="1"
+AR Path="/5A9CE314/5A5878F3" Ref="J?"  Part="1"
 F 0 "J?" H 2975 5870 50  0000 C CNN
 F 1 "TEST_1P" H 2975 5800 50  0000 C CNN
@@
 U 1 1 5A5878FA
 P 4250 5600
+AR Path="/5A585E42/5A5878FA" Ref="J?"  Part="1"
+AR Path="/5A9CE314/5A5878FA" Ref="J?"  Part="1"
 F 0 "J?" H 4250 5870 50  0000 C CNN
 F 1 "TEST_1P" H 4250 5800 50  0000 C CNN
@@
 U 1 1 5A587901
 P 4250 5950
+AR Path="/5A585E42/5A587901" Ref="J?"  Part="1"
+AR Path="/5A9CE314/5A587901" Ref="J?"  Part="1"
 F 0 "J?" H 4250 6220 50  0000 C CNN
 F 1 "TEST_1P" H 4250 6150 50  0000 C CNN
@@
 U 1 1 5A587908
 P 1875 5275
+AR Path="/5A585E42/5A587908" Ref="J?"  Part="1"
+AR Path="/5A9CE314/5A587908" Ref="J?"  Part="1"
 F 0 "J?" H 1875 5545 50  0000 C CNN
 F 1 "TEST_1P" H 1875 5475 50  0000 C CNN
@@
 U 1 1 5A58790F
 P 9300 3700
+AR Path="/5A585E42/5A58790F" Ref="J?"  Part="1"
+AR Path="/5A9CE314/5A58790F" Ref="J?"  Part="1"
 F 0 "J?" H 9300 3970 50  0000 C CNN
 F 1 "TEST_1P" H 9300 3900 50  0000 C CNN
@@
 U 1 1 5A587919
 P 8950 4000
+AR Path="/5A585E42/5A587919" Ref="D?"  Part="1"
+AR Path="/5A9CE314/5A587919" Ref="D?"  Part="1"
 F 0 "D?" H 9050 3800 60  0000 C CNN
 F 1 "PESD5Zx" H 8700 4100 60  0000 C CNN
@@
 U 1 1 5A587B17
 P 1975 2125
+AR Path="/5A585E42/5A587B17" Ref="C?"  Part="1"
+AR Path="/5A9CE314/5A587B17" Ref="C?"  Part="1"
 F 0 "C?" H 2000 2225 50  0000 L CNN
 F 1 "10uF" H 2000 2025 50  0000 L CNN
@@
 U 1 1 5A587B1E
 P 1975 2325
+AR Path="/5A585E42/5A587B1E" Ref="#PWR057"  Part="1"
+AR Path="/5A9CE314/5A587B1E" Ref="#PWR057"  Part="1"
 F 0 "#PWR057" H 1975 2075 50  0001 C CNN
 F 1 "GND" H 1975 2175 50  0000 C CNN
@@
 U 1 1 5A587B76
 P 4050 1125
+AR Path="/5A585E42/5A587B76" Ref="C?"  Part="1"
+AR Path="/5A9CE314/5A587B76" Ref="C?"  Part="1"
 F 0 "C?" H 4075 1225 50  0000 L CNN
 F 1 "2.2uF" H 4075 1025 50  0000 L CNN
@@
 U 1 1 5A587B8A
 P 2950 2000
+AR Path="/5A585E42/5A587B8A" Ref="C?"  Part="1"
+AR Path="/5A9CE314/5A587B8A" Ref="C?"  Part="1"
 F 0 "C?" H 2975 2100 50  0000 L CNN
 F 1 "1uF" H 2975 1900 50  0000 L CNN
@@
 U 1 1 5A587B94
 P 3700 1900
+AR Path="/5A585E42/5A587B94" Ref="C?"  Part="1"
+AR Path="/5A9CE314/5A587B94" Ref="C?"  Part="1"
 F 0 "C?" H 3725 2000 50  0000 L CNN
 F 1 "1uF" H 3725 1800 50  0000 L CNN
@@
 U 1 1 5A587BB2
 P 4350 925
+AR Path="/5A585E42/5A587BB2" Ref="R?"  Part="1"
+AR Path="/5A9CE314/5A587BB2" Ref="R?"  Part="1"
 F 0 "R?" V 4430 925 50  0000 C CNN
 F 1 "220R" V 4350 925 50  0000 C CNN
@@
 U 1 1 5A587BBC
 P 4900 1125
+AR Path="/5A585E42/5A587BBC" Ref="C?"  Part="1"
+AR Path="/5A9CE314/5A587BBC" Ref="C?"  Part="1"
 F 0 "C?" H 4925 1225 50  0000 L CNN
 F 1 "10uF" H 4925 1025 50  0000 L CNN
@@
 U 1 1 5A587BD2
 P 3075 5000
+AR Path="/5A585E42/5A587BD2" Ref="J?"  Part="1"
+AR Path="/5A9CE314/5A587BD2" Ref="J?"  Part="1"
 F 0 "J?" H 3075 5200 50  0000 C CNN
 F 1 "CONN_01X03" V 3175 5000 50  0000 C CNN
@@
 U 1 1 5A587BDC
 P 2600 1800
+AR Path="/5A585E42/5A587BDC" Ref="R?"  Part="1"
+AR Path="/5A9CE314/5A587BDC" Ref="R?"  Part="1"
 F 0 "R?" V 2680 1800 50  0000 C CNN
 F 1 "390R" V 2600 1800 50  0000 C CNN
@@
 U 1 1 5A587BE6
 P 1475 2850
+AR Path="/5A585E42/5A587BE6" Ref="C?"  Part="1"
+AR Path="/5A9CE314/5A587BE6" Ref="C?"  Part="1"
 F 0 "C?" H 1500 2950 50  0000 L CNN
 F 1 "1uF" H 1500 2750 50  0000 L CNN
@@
 U 1 1 5A587BF0
 P 4600 1125
+AR Path="/5A585E42/5A587BF0" Ref="C?"  Part="1"
+AR Path="/5A9CE314/5A587BF0" Ref="C?"  Part="1"
 F 0 "C?" H 4625 1225 50  0000 L CNN
 F 1 "1uF" H 4625 1025 50  0000 L CNN
@@
 U 1 1 5AA2BE5C
 P 8975 3525
+AR Path="/5A585E42/5AA2BE5C" Ref="#PWR058"  Part="1"
+AR Path="/5A9CE314/5AA2BE5C" Ref="#PWR058"  Part="1"
 F 0 "#PWR058" H 8975 3275 50  0001 C CNN
 F 1 "GND" H 8975 3375 50  0000 C CNN

Commit message: added 2 temp sensors for the 2 PAs
Changed lines of the file:
@@
 $Descr A4 11693 8268
 encoding utf-8
-Sheet 6 9
+Sheet 7 15
 Title ""
 Date ""
@@
 Wire Wire Line
 	3600 3875 3600 3800
+$Sheet
+S 5925 2700 750  525
+U 5AC22D6C
+F0 "Temperature_Sensor" 118
+F1 "TEMP_SENSE.sch" 118
+$EndSheet
 $EndSCHEMATC

Commit message: Added SP3T and 2:4 decoder
Parts:
- U201: symbol RF6886 -> RF6886-RESCUE-SFUSat-Radio
Changed lines of the file:
@@
 EESchema Schematic File Version 2
+LIBS:SFUSat-Radio-rescue
 LIBS:power
 LIBS:device
@@
 PA
 $Comp
-L RF6886 U201
+L RF6886-RESCUE-SFUSat-Radio U201
 U 1 1 5A587750
 P 3600 3100
