File: PA.sch (KiCad schematic (older format))
At the start: 32 parts, among them J401 TEST_1P, J402 TEST_1P, J403 CONN_01X03, J404 TEST_1P, J405 TEST_1P, J406 TEST_1P, U401 LMV358, U402 RF6886

Commit message: layed out power system
Changed lines of the file:
@@
 $Descr A4 11693 8268
 encoding utf-8
-Sheet 4 15
+Sheet 3 15
 Title ""
 Date ""
@@
 AR Path="/5A585E42/5A587750" Ref="U402"  Part="1"
 AR Path="/5A9CE314/5A587750" Ref="U502"  Part="1"
-F 0 "U502" H 3050 3750 60  0000 C CNN
+F 0 "U402" H 3050 3750 60  0000 C CNN
 F 1 "RF6886" H 3600 3100 60  0000 C CNN
 F 2 "SFUSat:QFN-24" H 3600 2750 60  0001 C CNN
@@
 AR Path="/5A585E42/5A58777F" Ref="C404"  Part="1"
 AR Path="/5A9CE314/5A58777F" Ref="C504"  Part="1"
-F 0 "C504" H 2000 2950 50  0000 L CNN
+F 0 "C404" H 2000 2950 50  0000 L CNN
 F 1 "2.2uF" H 2000 2750 50  0000 L CNN
 F 2 "SFUSat:C_0402" H 2013 2700 50  0001 C CNN
@@
 AR Path="/5A585E42/5A5877AD" Ref="R401"  Part="1"
 AR Path="/5A9CE314/5A5877AD" Ref="R501"  Part="1"
-F 0 "R501" V 1830 2650 50  0000 C CNN
+F 0 "R401" V 1830 2650 50  0000 C CNN
 F 1 "220R" V 1750 2650 50  0000 C CNN
 F 2 "SFUSat:R_0402" V 1680 2650 50  0001 C CNN
@@
 AR Path="/5A585E42/5A5877CD" Ref="C406"  Part="1"
 AR Path="/5A9CE314/5A5877CD" Ref="C506"  Part="1"
-F 0 "C506" H 2425 2850 50  0000 L CNN
+F 0 "C406" H 2425 2850 50  0000 L CNN
 F 1 "220pF" H 2425 2650 50  0000 L CNN
 F 2 "SFUSat:C_0402" H 2438 2600 50  0001 C CNN
@@
 AR Path="/5A585E42/5A5877DD" Ref="C407"  Part="1"
 AR Path="/5A9CE314/5A5877DD" Ref="C507"  Part="1"
-F 0 "C507" H 2975 1450 50  0000 L CNN
+F 0 "C407" H 2975 1450 50  0000 L CNN
 F 1 "1uF" H 2975 1250 50  0000 L CNN
 F 2 "SFUSat:C_0402" H 2988 1200 50  0001 C CNN
@@
 AR Path="/5A585E42/5A5877F3" Ref="R402"  Part="1"
 AR Path="/5A9CE314/5A5877F3" Ref="R502"  Part="1"
-F 0 "R502" V 2680 1150 50  0000 C CNN
+F 0 "R402" V 2680 1150 50  0000 C CNN
 F 1 "390R" V 2600 1150 50  0000 C CNN
 F 2 "SFUSat:R_0402" V 2530 1150 50  0001 C CNN
@@
 AR Path="/5A585E42/5A587804" Ref="U401"  Part="2"
 AR Path="/5A9CE314/5A587804" Ref="U501"  Part="2"
-F 0 "U501" H 3375 5925 50  0000 L CNN
+F 0 "U401" H 3375 5925 50  0000 L CNN
 F 1 "LMV358" H 3375 5625 50  0000 L CNN
 F 2 "SFUSat:TSSOP-8_4.4x3mm_Pitch0.65mm" H 3275 5825 50  0001 C CNN
@@
 AR Path="/5A585E42/5A58780E" Ref="U401"  Part="1"
 AR Path="/5A9CE314/5A58780E" Ref="U501"  Part="1"
-F 0 "U501" H 2325 6025 50  0000 L CNN
+F 0 "U401" H 2325 6025 50  0000 L CNN
 F 1 "LMV358" H 2325 5725 50  0000 L CNN
 F 2 "SFUSat:TSSOP-8_4.4x3mm_Pitch0.65mm" H 2225 5925 50  0001 C CNN
@@
 AR Path="/5A585E42/5A587818" Ref="R404"  Part="1"
 AR Path="/5A9CE314/5A587818" Ref="R504"  Part="1"
-F 0 "R504" V 2930 5775 50  0000 C CNN
+F 0 "R404" V 2930 5775 50  0000 C CNN
 F 1 "1K" V 2850 5775 50  0000 C CNN
 F 2 "SFUSat:R_0402" V 2780 5775 50  0001 C CNN
@@
 AR Path="/5A585E42/5A587822" Ref="R405"  Part="1"
 AR Path="/5A9CE314/5A587822" Ref="R505"  Part="1"
-F 0 "R505" V 3605 5275 50  0000 C CNN
+F 0 "R405" V 3605 5275 50  0000 C CNN
 F 1 "10K" V 3525 5275 50  0000 C CNN
 F 2 "SFUSat:R_0402" V 3455 5275 50  0001 C CNN
@@
 AR Path="/5A585E42/5A58782C" Ref="R406"  Part="1"
 AR Path="/5A9CE314/5A58782C" Ref="R506"  Part="1"
-F 0 "R506" V 3880 6100 50  0000 C CNN
+F 0 "R406" V 3880 6100 50  0000 C CNN
 F 1 "10K" V 3800 6100 50  0000 C CNN
 F 2 "SFUSat:R_0402" V 3730 6100 50  0001 C CNN
@@
 AR Path="/5A585E42/5A587836" Ref="R407"  Part="1"
 AR Path="/5A9CE314/5A587836" Ref="R507"  Part="1"
-F 0 "R507" V 4155 5675 50  0000 C CNN
+F 0 "R407" V 4155 5675 50  0000 C CNN
 F 1 "10K" V 4075 5675 50  0000 C CNN
 F 2 "SFUSat:R_0402" V 4005 5675 50  0001 C CNN
@@
 AR Path="/5A585E42/5A587840" Ref="R408"  Part="1"
 AR Path="/5A9CE314/5A587840" Ref="R508"  Part="1"
-F 0 "R508" V 4155 5875 50  0000 C CNN
+F 0 "R408" V 4155 5875 50  0000 C CNN
 F 1 "10K" V 4075 5875 50  0000 C CNN
 F 2 "SFUSat:R_0402" V 4005 5875 50  0001 C CNN
@@
 AR Path="/5A585E42/5A58784A" Ref="C405"  Part="1"
 AR Path="/5A9CE314/5A58784A" Ref="C505"  Part="1"
-F 0 "C505" H 2200 5375 50  0000 L CNN
+F 0 "C405" H 2200 5375 50  0000 L CNN
 F 1 "0.1uF" H 2200 5175 50  0000 L CNN
 F 2 "SFUSat:C_0402" H 2213 5125 50  0001 C CNN
@@
 AR Path="/5A585E42/5A58786F" Ref="RV401"  Part="1"
 AR Path="/5A9CE314/5A58786F" Ref="RV501"  Part="1"
-F 0 "RV501" V 9000 3525 50  0000 C CNN
+F 0 "RV401" V 9000 3525 50  0000 C CNN
 F 1 "POT" V 9075 3525 50  0000 C CNN
 F 2 "SFUSat:TC33_SMD" H 9175 3525 50  0001 C CNN
@@
 AR Path="/5A585E42/5A587879" Ref="R410"  Part="1"
 AR Path="/5A9CE314/5A587879" Ref="R510"  Part="1"
-F 0 "R510" V 9255 3875 50  0000 C CNN
+F 0 "R410" V 9255 3875 50  0000 C CNN
 F 1 "1K" V 9175 3875 50  0000 C CNN
 F 2 "SFUSat:R_0402" V 9105 3875 50  0001 C CNN
@@
 AR Path="/5A585E42/5A5878F3" Ref="J402"  Part="1"
 AR Path="/5A9CE314/5A5878F3" Ref="J502"  Part="1"
-F 0 "J502" H 2975 5870 50  0000 C CNN
+F 0 "J402" H 2975 5870 50  0000 C CNN
 F 1 "TEST_1P" H 2975 5800 50  0000 C CNN
 F 2 "SFUSat:Measurement_Point_Round-SMD-Pad_Big" H 3175 5600 50  0001 C CNN
@@
 AR Path="/5A585E42/5A5878FA" Ref="J404"  Part="1"
 AR Path="/5A9CE314/5A5878FA" Ref="J504"  Part="1"
-F 0 "J504" H 4250 5870 50  0000 C CNN
+F 0 "J404" H 4250 5870 50  0000 C CNN
 F 1 "TEST_1P" H 4250 5800 50  0000 C CNN
 F 2 "SFUSat:Measurement_Point_Round-SMD-Pad_Big" H 4450 5600 50  0001 C CNN
@@
 AR Path="/5A585E42/5A587901" Ref="J405"  Part="1"
 AR Path="/5A9CE314/5A587901" Ref="J505"  Part="1"
-F 0 "J505" H 4250 6220 50  0000 C CNN
+F 0 "J405" H 4250 6220 50  0000 C CNN
 F 1 "TEST_1P" H 4250 6150 50  0000 C CNN
 F 2 "SFUSat:Measurement_Point_Round-SMD-Pad_Big" H 4450 5950 50  0001 C CNN
@@
 AR Path="/5A585E42/5A587908" Ref="J401"  Part="1"
 AR Path="/5A9CE314/5A587908" Ref="J501"  Part="1"
-F 0 "J501" H 1875 5545 50  0000 C CNN
+F 0 "J401" H 1875 5545 50  0000 C CNN
 F 1 "TEST_1P" H 1875 5475 50  0000 C CNN
 F 2 "SFUSat:Measurement_Point_Round-SMD-Pad_Big" H 2075 5275 50  0001 C CNN
@@
 AR Path="/5A585E42/5A58790F" Ref="J406"  Part="1"
 AR Path="/5A9CE314/5A58790F" Ref="J506"  Part="1"
-F 0 "J506" H 9300 3970 50  0000 C CNN
+F 0 "J406" H 9300 3970 50  0000 C CNN
 F 1 "TEST_1P" H 9300 3900 50  0000 C CNN
 F 2 "SFUSat:Measurement_Point_Round-SMD-Pad_Big" H 9500 3700 50  0001 C CNN
@@
 AR Path="/5A585E42/5A587919" Ref="D401"  Part="1"
 AR Path="/5A9CE314/5A587919" Ref="D501"  Part="1"
-F 0 "D501" H 9050 3800 60  0000 C CNN
+F 0 "D401" H 9050 3800 60  0000 C CNN
 F 1 "PESD5Zx" H 8700 4100 60  0000 C CNN
 F 2 "SFUSat:PESD57zx" H 8950 4000 60  0001 C CNN
@@
 AR Path="/5A585E42/5A587B76" Ref="C410"  Part="1"
 AR Path="/5A9CE314/5A587B76" Ref="C510"  Part="1"
-F 0 "C510" H 4075 1225 50  0000 L CNN
+F 0 "C410" H 4075 1225 50  0000 L CNN
 F 1 "2.2uF" H 4075 1025 50  0000 L CNN
 F 2 "SFUSat:C_0402" H 4088 975 50  0001 C CNN
@@
 AR Path="/5A585E42/5A587B8A" Ref="C408"  Part="1"
 AR Path="/5A9CE314/5A587B8A" Ref="C508"  Part="1"
-F 0 "C508" H 2975 2100 50  0000 L CNN
+F 0 "C408" H 2975 2100 50  0000 L CNN
 F 1 "1uF" H 2975 1900 50  0000 L CNN
 F 2 "SFUSat:C_0402" H 2988 1850 50  0001 C CNN
@@
 AR Path="/5A585E42/5A587B94" Ref="C409"  Part="1"
 AR Path="/5A9CE314/5A587B94" Ref="C509"  Part="1"
-F 0 "C509" H 3725 2000 50  0000 L CNN
+F 0 "C409" H 3725 2000 50  0000 L CNN
 F 1 "1uF" H 3725 1800 50  0000 L CNN
 F 2 "SFUSat:C_0402" H 3738 1750 50  0001 C CNN
@@
 AR Path="/5A585E42/5A587BB2" Ref="R409"  Part="1"
 AR Path="/5A9CE314/5A587BB2" Ref="R509"  Part="1"
-F 0 "R509" V 4430 925 50  0000 C CNN
+F 0 "R409" V 4430 925 50  0000 C CNN
 F 1 "220R" V 4350 925 50  0000 C CNN
 F 2 "SFUSat:R_0402" V 4280 925 50  0001 C CNN
@@
 AR Path="/5A585E42/5A587BD2" Ref="J403"  Part="1"
 AR Path="/5A9CE314/5A587BD2" Ref="J503"  Part="1"
-F 0 "J503" H 3075 5200 50  0000 C CNN
+F 0 "J403" H 3075 5200 50  0000 C CNN
 F 1 "CONN_01X03" V 3175 5000 50  0000 C CNN
 F 2 "SFUSat:Socket_Strip_Straight_1x03" H 3075 5000 50  0001 C CNN
@@
 AR Path="/5A585E42/5A587BDC" Ref="R403"  Part="1"
 AR Path="/5A9CE314/5A587BDC" Ref="R503"  Part="1"
-F 0 "R503" V 2680 1800 50  0000 C CNN
+F 0 "R403" V 2680 1800 50  0000 C CNN
 F 1 "390R" V 2600 1800 50  0000 C CNN
 F 2 "SFUSat:R_0402" V 2530 1800 50  0001 C CNN
@@
 AR Path="/5A585E42/5A587BE6" Ref="C402"  Part="1"
 AR Path="/5A9CE314/5A587BE6" Ref="C502"  Part="1"
-F 0 "C502" H 1500 2950 50  0000 L CNN
+F 0 "C402" H 1500 2950 50  0000 L CNN
 F 1 "1uF" H 1500 2750 50  0000 L CNN
 F 2 "SFUSat:C_0402" H 1513 2700 50  0001 C CNN
@@
 AR Path="/5A585E42/5A587BF0" Ref="C411"  Part="1"
 AR Path="/5A9CE314/5A587BF0" Ref="C511"  Part="1"
-F 0 "C511" H 4625 1225 50  0000 L CNN
+F 0 "C411" H 4625 1225 50  0000 L CNN
 F 1 "DNP" H 4625 1025 50  0000 L CNN
 F 2 "SFUSat:C_0402" H 4638 975 50  0001 C CNN
@@
 AR Path="/5A585E42/5ABEC321" Ref="C401"  Part="1"
 AR Path="/5A9CE314/5ABEC321" Ref="C501"  Part="1"
-F 0 "C501" H 1225 2925 50  0000 L BNN
+F 0 "C401" H 1225 2925 50  0000 L BNN
 F 1 "10uF" H 1225 2775 50  0000 L TNN
 F 2 "SFUSat-cap:C_TANT_1411" H 1225 2850 50  0001 C CNN
@@
 AR Path="/5A585E42/5ABED10A" Ref="C412"  Part="1"
 AR Path="/5A9CE314/5ABED10A" Ref="C512"  Part="1"
-F 0 "C512" H 4900 1200 50  0000 L BNN
+F 0 "C412" H 4900 1200 50  0000 L BNN
 F 1 "10uF" H 4900 1050 50  0000 L TNN
 F 2 "SFUSat-cap:C_TANT_1411" H 4900 1125 50  0001 C CNN
@@
 AR Path="/5A585E42/5ABEC9B2" Ref="C403"  Part="1"
 AR Path="/5A9CE314/5ABEC9B2" Ref="C503"  Part="1"
-F 0 "C503" H 1975 2175 50  0000 L BNN
+F 0 "C403" H 1975 2175 50  0000 L BNN
 F 1 "10uF" H 1975 2075 50  0000 L TNN
 F 2 "SFUSat-cap:C_TANT_2312" H 1975 2125 50  0001 C CNN

Commit message: removed PA feedback jumper
Parts:
- removed J403: CONN_01X03, SFUSat:Socket_Strip_Straight_1x03, symbol CONN_01X03
Connections:
- wire segments 92 -> 88
Changed lines of the file:
@@
 AR Path="/5A585E42/5A587750" Ref="U402"  Part="1"
 AR Path="/5A9CE314/5A587750" Ref="U502"  Part="1"
-F 0 "U402" H 3050 3750 60  0000 C CNN
+F 0 "U502" H 3050 3750 60  0000 C CNN
 F 1 "RF6886" H 3600 3100 60  0000 C CNN
 F 2 "SFUSat:QFN-24" H 3600 2750 60  0001 C CNN
@@
 AR Path="/5A585E42/5A58777F" Ref="C404"  Part="1"
 AR Path="/5A9CE314/5A58777F" Ref="C504"  Part="1"
-F 0 "C404" H 2000 2950 50  0000 L CNN
+F 0 "C504" H 2000 2950 50  0000 L CNN
 F 1 "2.2uF" H 2000 2750 50  0000 L CNN
 F 2 "SFUSat:C_0402" H 2013 2700 50  0001 C CNN
@@
 AR Path="/5A585E42/5A5877AD" Ref="R401"  Part="1"
 AR Path="/5A9CE314/5A5877AD" Ref="R501"  Part="1"
-F 0 "R401" V 1830 2650 50  0000 C CNN
+F 0 "R501" V 1830 2650 50  0000 C CNN
 F 1 "220R" V 1750 2650 50  0000 C CNN
 F 2 "SFUSat:R_0402" V 1680 2650 50  0001 C CNN
@@
 AR Path="/5A585E42/5A5877CD" Ref="C406"  Part="1"
 AR Path="/5A9CE314/5A5877CD" Ref="C506"  Part="1"
-F 0 "C406" H 2425 2850 50  0000 L CNN
+F 0 "C506" H 2425 2850 50  0000 L CNN
 F 1 "220pF" H 2425 2650 50  0000 L CNN
 F 2 "SFUSat:C_0402" H 2438 2600 50  0001 C CNN
@@
 AR Path="/5A585E42/5A5877DD" Ref="C407"  Part="1"
 AR Path="/5A9CE314/5A5877DD" Ref="C507"  Part="1"
-F 0 "C407" H 2975 1450 50  0000 L CNN
+F 0 "C507" H 2975 1450 50  0000 L CNN
 F 1 "1uF" H 2975 1250 50  0000 L CNN
 F 2 "SFUSat:C_0402" H 2988 1200 50  0001 C CNN
@@
 AR Path="/5A585E42/5A5877F3" Ref="R402"  Part="1"
 AR Path="/5A9CE314/5A5877F3" Ref="R502"  Part="1"
-F 0 "R402" V 2680 1150 50  0000 C CNN
+F 0 "R502" V 2680 1150 50  0000 C CNN
 F 1 "390R" V 2600 1150 50  0000 C CNN
 F 2 "SFUSat:R_0402" V 2530 1150 50  0001 C CNN
@@
 AR Path="/5A585E42/5A587804" Ref="U401"  Part="2"
 AR Path="/5A9CE314/5A587804" Ref="U501"  Part="2"
-F 0 "U401" H 3375 5925 50  0000 L CNN
+F 0 "U501" H 3375 5925 50  0000 L CNN
 F 1 "LMV358" H 3375 5625 50  0000 L CNN
 F 2 "SFUSat:TSSOP-8_4.4x3mm_Pitch0.65mm" H 3275 5825 50  0001 C CNN
@@
 AR Path="/5A585E42/5A58780E" Ref="U401"  Part="1"
 AR Path="/5A9CE314/5A58780E" Ref="U501"  Part="1"
-F 0 "U401" H 2325 6025 50  0000 L CNN
+F 0 "U501" H 2325 6025 50  0000 L CNN
 F 1 "LMV358" H 2325 5725 50  0000 L CNN
 F 2 "SFUSat:TSSOP-8_4.4x3mm_Pitch0.65mm" H 2225 5925 50  0001 C CNN
@@
 AR Path="/5A585E42/5A587818" Ref="R404"  Part="1"
 AR Path="/5A9CE314/5A587818" Ref="R504"  Part="1"
-F 0 "R404" V 2930 5775 50  0000 C CNN
+F 0 "R504" V 2930 5775 50  0000 C CNN
 F 1 "1K" V 2850 5775 50  0000 C CNN
 F 2 "SFUSat:R_0402" V 2780 5775 50  0001 C CNN
@@
 AR Path="/5A585E42/5A587822" Ref="R405"  Part="1"
 AR Path="/5A9CE314/5A587822" Ref="R505"  Part="1"
-F 0 "R405" V 3605 5275 50  0000 C CNN
+F 0 "R505" V 3605 5275 50  0000 C CNN
 F 1 "10K" V 3525 5275 50  0000 C CNN
 F 2 "SFUSat:R_0402" V 3455 5275 50  0001 C CNN
@@
 AR Path="/5A585E42/5A58782C" Ref="R406"  Part="1"
 AR Path="/5A9CE314/5A58782C" Ref="R506"  Part="1"
-F 0 "R406" V 3880 6100 50  0000 C CNN
+F 0 "R506" V 3880 6100 50  0000 C CNN
 F 1 "10K" V 3800 6100 50  0000 C CNN
 F 2 "SFUSat:R_0402" V 3730 6100 50  0001 C CNN
@@
 AR Path="/5A585E42/5A587836" Ref="R407"  Part="1"
 AR Path="/5A9CE314/5A587836" Ref="R507"  Part="1"
-F 0 "R407" V 4155 5675 50  0000 C CNN
+F 0 "R507" V 4155 5675 50  0000 C CNN
 F 1 "10K" V 4075 5675 50  0000 C CNN
 F 2 "SFUSat:R_0402" V 4005 5675 50  0001 C CNN
@@
 AR Path="/5A585E42/5A587840" Ref="R408"  Part="1"
 AR Path="/5A9CE314/5A587840" Ref="R508"  Part="1"
-F 0 "R408" V 4155 5875 50  0000 C CNN
+F 0 "R508" V 4155 5875 50  0000 C CNN
 F 1 "10K" V 4075 5875 50  0000 C CNN
 F 2 "SFUSat:R_0402" V 4005 5875 50  0001 C CNN
@@
 AR Path="/5A585E42/5A58784A" Ref="C405"  Part="1"
 AR Path="/5A9CE314/5A58784A" Ref="C505"  Part="1"
-F 0 "C405" H 2200 5375 50  0000 L CNN
+F 0 "C505" H 2200 5375 50  0000 L CNN
 F 1 "0.1uF" H 2200 5175 50  0000 L CNN
 F 2 "SFUSat:C_0402" H 2213 5125 50  0001 C CNN
@@
 AR Path="/5A585E42/5A58786F" Ref="RV401"  Part="1"
 AR Path="/5A9CE314/5A58786F" Ref="RV501"  Part="1"
-F 0 "RV401" V 9000 3525 50  0000 C CNN
+F 0 "RV501" V 9000 3525 50  0000 C CNN
 F 1 "POT" V 9075 3525 50  0000 C CNN
 F 2 "SFUSat:TC33_SMD" H 9175 3525 50  0001 C CNN
@@
 AR Path="/5A585E42/5A587879" Ref="R410"  Part="1"
 AR Path="/5A9CE314/5A587879" Ref="R510"  Part="1"
-F 0 "R410" V 9255 3875 50  0000 C CNN
+F 0 "R510" V 9255 3875 50  0000 C CNN
 F 1 "1K" V 9175 3875 50  0000 C CNN
 F 2 "SFUSat:R_0402" V 9105 3875 50  0001 C CNN
@@
 AR Path="/5A585E42/5A5878F3" Ref="J402"  Part="1"
 AR Path="/5A9CE314/5A5878F3" Ref="J502"  Part="1"
-F 0 "J402" H 2975 5870 50  0000 C CNN
+F 0 "J502" H 2975 5870 50  0000 C CNN
 F 1 "TEST_1P" H 2975 5800 50  0000 C CNN
 F 2 "SFUSat:Measurement_Point_Round-SMD-Pad_Big" H 3175 5600 50  0001 C CNN
@@
 AR Path="/5A585E42/5A5878FA" Ref="J404"  Part="1"
 AR Path="/5A9CE314/5A5878FA" Ref="J504"  Part="1"
-F 0 "J404" H 4250 5870 50  0000 C CNN
+F 0 "J504" H 4250 5870 50  0000 C CNN
 F 1 "TEST_1P" H 4250 5800 50  0000 C CNN
 F 2 "SFUSat:Measurement_Point_Round-SMD-Pad_Big" H 4450 5600 50  0001 C CNN
@@
 AR Path="/5A585E42/5A587901" Ref="J405"  Part="1"
 AR Path="/5A9CE314/5A587901" Ref="J505"  Part="1"
-F 0 "J405" H 4250 6220 50  0000 C CNN
+F 0 "J505" H 4250 6220 50  0000 C CNN
 F 1 "TEST_1P" H 4250 6150 50  0000 C CNN
 F 2 "SFUSat:Measurement_Point_Round-SMD-Pad_Big" H 4450 5950 50  0001 C CNN
@@
 AR Path="/5A585E42/5A587908" Ref="J401"  Part="1"
 AR Path="/5A9CE314/5A587908" Ref="J501"  Part="1"
-F 0 "J401" H 1875 5545 50  0000 C CNN
+F 0 "J501" H 1875 5545 50  0000 C CNN
 F 1 "TEST_1P" H 1875 5475 50  0000 C CNN
 F 2 "SFUSat:Measurement_Point_Round-SMD-Pad_Big" H 2075 5275 50  0001 C CNN
@@
 AR Path="/5A585E42/5A58790F" Ref="J406"  Part="1"
 AR Path="/5A9CE314/5A58790F" Ref="J506"  Part="1"
-F 0 "J406" H 9300 3970 50  0000 C CNN
+F 0 "J506" H 9300 3970 50  0000 C CNN
 F 1 "TEST_1P" H 9300 3900 50  0000 C CNN
 F 2 "SFUSat:Measurement_Point_Round-SMD-Pad_Big" H 9500 3700 50  0001 C CNN
@@
 AR Path="/5A585E42/5A587919" Ref="D401"  Part="1"
 AR Path="/5A9CE314/5A587919" Ref="D501"  Part="1"
-F 0 "D401" H 9050 3800 60  0000 C CNN
+F 0 "D501" H 9050 3800 60  0000 C CNN
 F 1 "PESD5Zx" H 8700 4100 60  0000 C CNN
 F 2 "SFUSat:PESD57zx" H 8950 4000 60  0001 C CNN
@@
 	2975 5600 3025 5600
 Wire Wire Line
-	3175 5275 3175 5200
-Wire Wire Line
-	3075 5275 3075 5200
-Wire Wire Line
-	3025 5275 3075 5275
-Connection ~ 2975 5425
-Wire Wire Line
-	2975 5200 2975 5425
+	3025 5275 3375 5275
 Wire Wire Line
 	3675 5275 3800 5275
-Wire Wire Line
-	3175 5275 3375 5275
 Wire Wire Line
 	2200 2650 1900 2650
@@
 AR Path="/5A585E42/5A587B76" Ref="C410"  Part="1"
 AR Path="/5A9CE314/5A587B76" Ref="C510"  Part="1"
-F 0 "C410" H 4075 1225 50  0000 L CNN
+F 0 "C510" H 4075 1225 50  0000 L CNN
 F 1 "2.2uF" H 4075 1025 50  0000 L CNN
 F 2 "SFUSat:C_0402" H 4088 975 50  0001 C CNN
@@
 AR Path="/5A585E42/5A587B8A" Ref="C408"  Part="1"
 AR Path="/5A9CE314/5A587B8A" Ref="C508"  Part="1"
-F 0 "C408" H 2975 2100 50  0000 L CNN
+F 0 "C508" H 2975 2100 50  0000 L CNN
 F 1 "1uF" H 2975 1900 50  0000 L CNN
 F 2 "SFUSat:C_0402" H 2988 1850 50  0001 C CNN
@@
 AR Path="/5A585E42/5A587B94" Ref="C409"  Part="1"
 AR Path="/5A9CE314/5A587B94" Ref="C509"  Part="1"
-F 0 "C409" H 3725 2000 50  0000 L CNN
+F 0 "C509" H 3725 2000 50  0000 L CNN
 F 1 "1uF" H 3725 1800 50  0000 L CNN
 F 2 "SFUSat:C_0402" H 3738 1750 50  0001 C CNN
@@
 AR Path="/5A585E42/5A587BB2" Ref="R409"  Part="1"
 AR Path="/5A9CE314/5A587BB2" Ref="R509"  Part="1"
-F 0 "R409" V 4430 925 50  0000 C CNN
+F 0 "R509" V 4430 925 50  0000 C CNN
 F 1 "220R" V 4350 925 50  0000 C CNN
 F 2 "SFUSat:R_0402" V 4280 925 50  0001 C CNN
@@
 $EndComp
 $Comp
-L CONN_01X03 J403
-U 1 1 5A587BD2
-P 3075 5000
-AR Path="/5A585E42/5A587BD2" Ref="J403"  Part="1"
-AR Path="/5A9CE314/5A587BD2" Ref="J503"  Part="1"
-F 0 "J403" H 3075 5200 50  0000 C CNN
-F 1 "CONN_01X03" V 3175 5000 50  0000 C CNN
-F 2 "SFUSat:Socket_Strip_Straight_1x03" H 3075 5000 50  0001 C CNN
-F 3 "" H 3075 5000 50  0001 C CNN
-F 4 "PRPC003SAAN-RC" H 3075 5000 60  0001 C CNN "Part Number"
-F 5 "S1011EC-03-ND" H 3075 5000 60  0001 C CNN "Digi-Key"
-F 6 "N/A" H 3075 5000 60  0001 C CNN "Mouser"
-	1    3075 5000
-	0    -1   -1   0
-$EndComp
-$Comp
 L R R403
 U 1 1 5A587BDC
@@
 AR Path="/5A585E42/5A587BDC" Ref="R403"  Part="1"
 AR Path="/5A9CE314/5A587BDC" Ref="R503"  Part="1"
-F 0 "R403" V 2680 1800 50  0000 C CNN
+F 0 "R503" V 2680 1800 50  0000 C CNN
 F 1 "390R" V 2600 1800 50  0000 C CNN
 F 2 "SFUSat:R_0402" V 2530 1800 50  0001 C CNN
@@
 AR Path="/5A585E42/5A587BE6" Ref="C402"  Part="1"
 AR Path="/5A9CE314/5A587BE6" Ref="C502"  Part="1"
-F 0 "C402" H 1500 2950 50  0000 L CNN
+F 0 "C502" H 1500 2950 50  0000 L CNN
 F 1 "1uF" H 1500 2750 50  0000 L CNN
 F 2 "SFUSat:C_0402" H 1513 2700 50  0001 C CNN
@@
 AR Path="/5A585E42/5A587BF0" Ref="C411"  Part="1"
 AR Path="/5A9CE314/5A587BF0" Ref="C511"  Part="1"
-F 0 "C411" H 4625 1225 50  0000 L CNN
+F 0 "C511" H 4625 1225 50  0000 L CNN
 F 1 "DNP" H 4625 1025 50  0000 L CNN
 F 2 "SFUSat:C_0402" H 4638 975 50  0001 C CNN
@@
 AR Path="/5A585E42/5ABEC321" Ref="C401"  Part="1"
 AR Path="/5A9CE314/5ABEC321" Ref="C501"  Part="1"
-F 0 "C401" H 1225 2925 50  0000 L BNN
+F 0 "C501" H 1225 2925 50  0000 L BNN
 F 1 "10uF" H 1225 2775 50  0000 L TNN
 F 2 "SFUSat-cap:C_TANT_1411" H 1225 2850 50  0001 C CNN
@@
 AR Path="/5A585E42/5ABED10A" Ref="C412"  Part="1"
 AR Path="/5A9CE314/5ABED10A" Ref="C512"  Part="1"
-F 0 "C412" H 4900 1200 50  0000 L BNN
+F 0 "C512" H 4900 1200 50  0000 L BNN
 F 1 "10uF" H 4900 1050 50  0000 L TNN
 F 2 "SFUSat-cap:C_TANT_1411" H 4900 1125 50  0001 C CNN
@@
 AR Path="/5A585E42/5ABEC9B2" Ref="C403"  Part="1"
 AR Path="/5A9CE314/5ABEC9B2" Ref="C503"  Part="1"
-F 0 "C403" H 1975 2175 50  0000 L BNN
+F 0 "C503" H 1975 2175 50  0000 L BNN
 F 1 "10uF" H 1975 2075 50  0000 L TNN
 F 2 "SFUSat-cap:C_TANT_2312" H 1975 2125 50  0001 C CNN

Commit message: Added extra DNP filter caps for PAs
Also confirmed PA UB components and updated Google Sheet
Parts:
- added C523, C524, C525, C526, C527: DNP, SFUSat:C_0402, symbol C
Connections:
- wire segments 88 -> 90

Commit message: Continued PA routing
Parts:
- added C428: DNP, SFUSat:C_0402, symbol C
Connections:
- wire segments 90 -> 91

Commit message: Added PA shield
Parts:
- removed J401, J402, J404, J405, J406: TEST_1P, SFUSat:Measurement_Point_Round-SMD-Pad_Big, symbol TEST_1P
- added J401, J402, J404, J405, J406: TP_100_SMD, SFUSat:TP_SMD_100, symbol TP_100_SMD
- added SH500: BMI-S-205-F, BMI-S-205-F, symbol BMI-S-205-F
Connections:
- wire segments 91 -> 96
Other:
- moved on the sheet: C405, R404, R405, R406, R407, R408

Commit message: Essentially done PA
Parts:
- removed J401, J402, J404, J405, J406: TP_100_SMD, SFUSat:TP_SMD_100, symbol TP_100_SMD
- added J401, J402, J404, J405, J406: TP_TH_150, SFUSat:TP_TH_150, symbol TP_TH_150
