File: PA.sch (KiCad schematic (older format))
At the start: 38 parts, among them J401 TP_TH_150, J402 TP_TH_150, J404 TP_TH_150, J405 TP_TH_150, J406 TP_TH_150, U401 LMV358, U402 RF6886

Commit message: Added inverter and new pots
Parts:
- removed RV401: POT, SFUSat:TC33_SMD, symbol POT
- added RV401: CT6EP103, SFUSat:CT6EP103, symbol CT6EP103
- SH500: footprint BMI-S-205-F -> SFUSat:BMI-S-205-F
Changed lines of the file:
@@
 $Descr A4 11693 8268
 encoding utf-8
-Sheet 4 15
+Sheet 3 15
 Title ""
 Date ""
@@
 $EndComp
 $Comp
-L GND #PWR038
+L GND #PWR47
 U 1 1 5A587792
 P 3700 2100
-AR Path="/5A585E42/5A587792" Ref="#PWR038"  Part="1"
-AR Path="/5A9CE314/5A587792" Ref="#PWR053"  Part="1"
-F 0 "#PWR053" H 3700 1850 50  0001 C CNN
+AR Path="/5A585E42/5A587792" Ref="#PWR47"  Part="1"
+AR Path="/5A9CE314/5A587792" Ref="#PWR62"  Part="1"
+F 0 "#PWR62" H 3700 1850 50  0001 C CNN
 F 1 "GND" H 3700 1950 50  0000 C CNN
 F 2 "" H 3700 2100 50  0001 C CNN
@@
 $EndComp
 $Comp
-L GND #PWR039
+L GND #PWR46
 U 1 1 5A587798
 P 3600 3875
-AR Path="/5A585E42/5A587798" Ref="#PWR039"  Part="1"
-AR Path="/5A9CE314/5A587798" Ref="#PWR054"  Part="1"
-F 0 "#PWR054" H 3600 3625 50  0001 C CNN
+AR Path="/5A585E42/5A587798" Ref="#PWR46"  Part="1"
+AR Path="/5A9CE314/5A587798" Ref="#PWR61"  Part="1"
+F 0 "#PWR61" H 3600 3625 50  0001 C CNN
 F 1 "GND" H 3600 3725 50  0000 C CNN
 F 2 "" H 3600 3875 50  0001 C CNN
@@
 $EndComp
 $Comp
-L GND #PWR040
+L GND #PWR40
 U 1 1 5A5877A4
 P 1975 3050
-AR Path="/5A585E42/5A5877A4" Ref="#PWR040"  Part="1"
-AR Path="/5A9CE314/5A5877A4" Ref="#PWR055"  Part="1"
-F 0 "#PWR055" H 1975 2800 50  0001 C CNN
+AR Path="/5A585E42/5A5877A4" Ref="#PWR40"  Part="1"
+AR Path="/5A9CE314/5A5877A4" Ref="#PWR55"  Part="1"
+F 0 "#PWR55" H 1975 2800 50  0001 C CNN
 F 1 "GND" H 1975 2900 50  0000 C CNN
 F 2 "" H 1975 3050 50  0001 C CNN
@@
 $EndComp
 $Comp
-L GND #PWR041
+L GND #PWR49
 U 1 1 5A5877BE
 P 4500 1375
-AR Path="/5A585E42/5A5877BE" Ref="#PWR041"  Part="1"
-AR Path="/5A9CE314/5A5877BE" Ref="#PWR056"  Part="1"
-F 0 "#PWR056" H 4500 1125 50  0001 C CNN
+AR Path="/5A585E42/5A5877BE" Ref="#PWR49"  Part="1"
+AR Path="/5A9CE314/5A5877BE" Ref="#PWR64"  Part="1"
+F 0 "#PWR64" H 4500 1125 50  0001 C CNN
 F 1 "GND" H 4500 1225 50  0000 C CNN
 F 2 "" H 4500 1375 50  0001 C CNN
@@
 $EndComp
 $Comp
-L GND #PWR042
+L GND #PWR38
 U 1 1 5A5877C4
 P 1325 3100
-AR Path="/5A585E42/5A5877C4" Ref="#PWR042"  Part="1"
-AR Path="/5A9CE314/5A5877C4" Ref="#PWR057"  Part="1"
-F 0 "#PWR057" H 1325 2850 50  0001 C CNN
+AR Path="/5A585E42/5A5877C4" Ref="#PWR38"  Part="1"
+AR Path="/5A9CE314/5A5877C4" Ref="#PWR53"  Part="1"
+F 0 "#PWR53" H 1325 2850 50  0001 C CNN
 F 1 "GND" H 1325 2950 50  0000 C CNN
 F 2 "" H 1325 3100 50  0001 C CNN
@@
 $EndComp
 $Comp
-L GND #PWR043
+L GND #PWR41
 U 1 1 5A5877D4
 P 2400 2950
-AR Path="/5A585E42/5A5877D4" Ref="#PWR043"  Part="1"
-AR Path="/5A9CE314/5A5877D4" Ref="#PWR058"  Part="1"
-F 0 "#PWR058" H 2400 2700 50  0001 C CNN
+AR Path="/5A585E42/5A5877D4" Ref="#PWR41"  Part="1"
+AR Path="/5A9CE314/5A5877D4" Ref="#PWR56"  Part="1"
+F 0 "#PWR56" H 2400 2700 50  0001 C CNN
 F 1 "GND" H 2400 2800 50  0000 C CNN
 F 2 "" H 2400 2950 50  0001 C CNN
@@
 $EndComp
 $Comp
-L GND #PWR044
+L GND #PWR45
 U 1 1 5A5877E4
 P 2950 2200
-AR Path="/5A585E42/5A5877E4" Ref="#PWR044"  Part="1"
-AR Path="/5A9CE314/5A5877E4" Ref="#PWR059"  Part="1"
-F 0 "#PWR059" H 2950 1950 50  0001 C CNN
+AR Path="/5A585E42/5A5877E4" Ref="#PWR45"  Part="1"
+AR Path="/5A9CE314/5A5877E4" Ref="#PWR60"  Part="1"
+F 0 "#PWR60" H 2950 1950 50  0001 C CNN
 F 1 "GND" H 2950 2050 50  0000 C CNN
 F 2 "" H 2950 2200 50  0001 C CNN
@@
 $EndComp
 $Comp
-L GND #PWR045
+L GND #PWR44
 U 1 1 5A5877EA
 P 2950 1550
-AR Path="/5A585E42/5A5877EA" Ref="#PWR045"  Part="1"
-AR Path="/5A9CE314/5A5877EA" Ref="#PWR060"  Part="1"
-F 0 "#PWR060" H 2950 1300 50  0001 C CNN
+AR Path="/5A585E42/5A5877EA" Ref="#PWR44"  Part="1"
+AR Path="/5A9CE314/5A5877EA" Ref="#PWR59"  Part="1"
+F 0 "#PWR59" H 2950 1300 50  0001 C CNN
 F 1 "GND" H 2950 1400 50  0000 C CNN
 F 2 "" H 2950 1550 50  0001 C CNN
@@
 $EndComp
 $Comp
-L GND #PWR046
+L GND #PWR43
 U 1 1 5A587853
 P 2825 5325
-AR Path="/5A585E42/5A587853" Ref="#PWR046"  Part="1"
-AR Path="/5A9CE314/5A587853" Ref="#PWR061"  Part="1"
-F 0 "#PWR061" H 2825 5075 50  0001 C CNN
+AR Path="/5A585E42/5A587853" Ref="#PWR43"  Part="1"
+AR Path="/5A9CE314/5A587853" Ref="#PWR58"  Part="1"
+F 0 "#PWR58" H 2825 5075 50  0001 C CNN
 F 1 "GND" H 2825 5175 50  0000 C CNN
 F 2 "" H 2825 5325 50  0001 C CNN
@@
 $EndComp
 $Comp
-L GND #PWR047
+L GND #PWR48
 U 1 1 5A587859
 P 3775 6275
-AR Path="/5A585E42/5A587859" Ref="#PWR047"  Part="1"
-AR Path="/5A9CE314/5A587859" Ref="#PWR062"  Part="1"
-F 0 "#PWR062" H 3775 6025 50  0001 C CNN
+AR Path="/5A585E42/5A587859" Ref="#PWR48"  Part="1"
+AR Path="/5A9CE314/5A587859" Ref="#PWR63"  Part="1"
+F 0 "#PWR63" H 3775 6025 50  0001 C CNN
 F 1 "GND" H 3775 6125 50  0000 C CNN
 F 2 "" H 3775 6275 50  0001 C CNN
@@
 Text HLabel 2975 6200 3    60   Input ~ 0
 3V1
-$Comp
-L POT RV401
-U 1 1 5A58786F
-P 9175 3525
-AR Path="/5A585E42/5A58786F" Ref="RV401"  Part="1"
-AR Path="/5A9CE314/5A58786F" Ref="RV501"  Part="1"
-F 0 "RV501" V 9000 3525 50  0000 C CNN
-F 1 "POT" V 9075 3525 50  0000 C CNN
-F 2 "SFUSat:TC33_SMD" H 9175 3525 50  0001 C CNN
-F 3 "" H 9175 3525 50  0001 C CNN
-F 4 "TC33X-2-103E" V 9175 3525 60  0001 C CNN "Part Number"
-F 5 "TC33X-103ECT-ND" V 9175 3525 60  0001 C CNN "Digi-Key"
-F 6 "652-TC33X-2-103E" V 9175 3525 60  0001 C CNN "Mouser"
-	1    9175 3525
-	0    1    1    0
-$EndComp
 $Comp
 L R R410
@@
 $EndComp
 $Comp
-L GND #PWR048
+L GND #PWR52
 U 1 1 5A587883
 P 9075 4350
-AR Path="/5A585E42/5A587883" Ref="#PWR048"  Part="1"
-AR Path="/5A9CE314/5A587883" Ref="#PWR063"  Part="1"
-F 0 "#PWR063" H 9075 4100 50  0001 C CNN
+AR Path="/5A585E42/5A587883" Ref="#PWR52"  Part="1"
+AR Path="/5A9CE314/5A587883" Ref="#PWR67"  Part="1"
+F 0 "#PWR67" H 9075 4100 50  0001 C CNN
 F 1 "GND" H 9075 4200 50  0000 C CNN
 F 2 "" H 9075 4350 50  0001 C CNN
@@
 0.28V to 3.1V
 $Comp
-L GND #PWR049
+L GND #PWR39
 U 1 1 5A587B1E
 P 1975 2325
-AR Path="/5A585E42/5A587B1E" Ref="#PWR049"  Part="1"
-AR Path="/5A9CE314/5A587B1E" Ref="#PWR064"  Part="1"
-F 0 "#PWR064" H 1975 2075 50  0001 C CNN
+AR Path="/5A585E42/5A587B1E" Ref="#PWR39"  Part="1"
+AR Path="/5A9CE314/5A587B1E" Ref="#PWR54"  Part="1"
+F 0 "#PWR54" H 1975 2075 50  0001 C CNN
 F 1 "GND" H 1975 2175 50  0000 C CNN
 F 2 "" H 1975 2325 50  0001 C CNN
@@
 GAIN
 $Comp
-L GND #PWR050
+L GND #PWR51
 U 1 1 5AA2BE5C
 P 8975 3525
-AR Path="/5A585E42/5AA2BE5C" Ref="#PWR050"  Part="1"
-AR Path="/5A9CE314/5AA2BE5C" Ref="#PWR065"  Part="1"
-F 0 "#PWR065" H 8975 3275 50  0001 C CNN
+AR Path="/5A585E42/5AA2BE5C" Ref="#PWR51"  Part="1"
+AR Path="/5A9CE314/5AA2BE5C" Ref="#PWR66"  Part="1"
+F 0 "#PWR66" H 8975 3275 50  0001 C CNN
 F 1 "GND" H 8975 3375 50  0000 C CNN
 F 2 "" H 8975 3525 50  0001 C CNN
@@
 	2525 2275 2525 2325
 $Comp
-L GND #PWR066
+L GND #PWR57
 U 1 1 5AC765FE
 P 2525 2325
-AR Path="/5A9CE314/5AC765FE" Ref="#PWR066"  Part="1"
-AR Path="/5A585E42/5AC765FE" Ref="#PWR051"  Part="1"
-F 0 "#PWR066" H 2525 2075 50  0001 C CNN
+AR Path="/5A9CE314/5AC765FE" Ref="#PWR57"  Part="1"
+AR Path="/5A585E42/5AC765FE" Ref="#PWR42"  Part="1"
+F 0 "#PWR57" H 2525 2075 50  0001 C CNN
 F 1 "GND" H 2525 2175 50  0000 C CNN
 F 2 "" H 2525 2325 50  0001 C CNN
@@
 F 0 "SH500" H 6250 3200 50  0000 L BNN
 F 1 "BMI-S-205-F" H 6250 2600 50  0000 L TNN
-F 2 "BMI-S-205-F" H 6000 2900 50  0001 C CNN
+F 2 "SFUSat:BMI-S-205-F" H 6000 2900 50  0001 C CNN
 F 3 "" H 6000 2900 50  0001 C CNN
 F 4 "RF/IF and RFID - RF Shields" H 6000 2900 50  0001 C CNN "Categories"
@@
 	6000 3350 6000 3450
 $Comp
-L GND #PWR067
+L GND #PWR65
 U 1 1 5ACCCEBA
 P 6000 3450
-AR Path="/5A9CE314/5ACCCEBA" Ref="#PWR067"  Part="1"
-AR Path="/5A585E42/5ACCCEBA" Ref="#PWR052"  Part="1"
-F 0 "#PWR067" H 6000 3200 50  0001 C CNN
+AR Path="/5A9CE314/5ACCCEBA" Ref="#PWR65"  Part="1"
+AR Path="/5A585E42/5ACCCEBA" Ref="#PWR50"  Part="1"
+F 0 "#PWR65" H 6000 3200 50  0001 C CNN
 F 1 "GND" H 6000 3300 50  0000 C CNN
 F 2 "" H 6000 3450 50  0001 C CNN
@@
 	0    1    1    0
 $EndComp
+$Comp
+L CT6EP103 RV401
+U 1 1 5AD75A41
+P 9175 3525
+AR Path="/5A585E42/5AD75A41" Ref="RV401"  Part="1"
+AR Path="/5A9CE314/5AD75A41" Ref="RV501"  Part="1"
+F 0 "RV501" H 9175 3465 50  0000 C TNN
+F 1 "CT6EP103" H 9175 3525 50  0001 C CNN
+F 2 "SFUSat:CT6EP103" H 9175 3525 50  0001 C CNN
+F 3 "" H 9175 3525 50  0001 C CNN
+F 4 "Top Adjustment" H 9175 3525 50  0001 C CNN "Adjustment Type"
+F 5 "Potentiometers, Variable Resistors - Trimmer Potentiometers" H 9175 3525 50  0001 C CNN "Categories"
+F 6 "Lead free / RoHS Compliant" H 9175 3525 50  0001 C CNN "Lead Free Status / RoHS Status"
+F 7 "Nidec Copal Electronics" H 9175 3525 50  0001 C CNN "Manufacturer 1"
+F 8 "CT6EP103" H 9175 3525 50  0001 C CNN "Manufacturer Part Number 1"
+F 9 "9 Weeks" H 9175 3525 50  0001 C CNN "Manufacturer Standard Lead Time 1"
+F 10 "Through Hole" H 9175 3525 50  0001 C CNN "Mounting Type"
+F 11 "1" H 9175 3525 50  0001 C CNN "Number of Turns"
+F 12 "Active" H 9175 3525 50  0001 C CNN "Part Status"
+F 13 "0.5W, 1/2W" H 9175 3525 50  0001 C CNN "Power (Watts)"
+F 14 "10 kOhms" H 9175 3525 50  0001 C CNN "Resistance"
+F 15 "Cermet" H 9175 3525 50  0001 C CNN "Resistive Material"
+F 16 "CT6" H 9175 3525 50  0001 C CNN "Series"
+F 17 "Square - 0.276\" x 0.276\" Face x 0.228\" L (7.00mm x 7.00mm x 5.80mm)" H 9175 3525 50  0001 C CNN "Size / Dimension"
+F 18 "Digi-Key" H 9175 3525 50  0001 C CNN "Supplier 1"
+F 19 "CT6EP103-ND" H 9175 3525 50  0001 C CNN "Supplier Part Number 1"
+F 20 "±100ppm/°C" H 9175 3525 50  0001 C CNN "Temperature Coefficient"
+F 21 "PC Pins" H 9175 3525 50  0001 C CNN "Termination Style"
+F 22 "±10%" H 9175 3525 50  0001 C CNN "Tolerance"
+	1    9175 3525
+	-1   0    0    1
+$EndComp
 $EndSCHEMATC
