File: PA.sch (KiCad schematic (older format))
At the start: 38 parts, among them J401 TP_TH_150, J402 TP_TH_150, J404 TP_TH_150, J405 TP_TH_150, J406 TP_TH_150, U401 LMV358, U402 RF6886

Commit message: added optional gain select resistor
Parts:
- added R411: DNP, SFUSat:R_0402, symbol R
Connections:
- wire segments 96 -> 98

Commit message: Continued power floods
Other:
- note added: "0.062V to 3.038V"
- note removed: "0.28V to 3.1V"
Changed lines of the file:
@@
 $Descr A4 11693 8268
 encoding utf-8
-Sheet 3 15
+Sheet 4 15
 Title ""
 Date ""
@@
 Text Notes 2400 7000 0    79   ~ 0
 R*05,R*06/R*07,R*08 * (Vref - Vsense) = Vout
-Text Notes 7900 3250 0    79   ~ 0
-0.28V to 3.1V
+Text Notes 7650 3250 0    79   ~ 0
+0.062V to 3.038V
 $Comp
 L GND #PWR053

Commit message: modified proposed pot schematic
Parts:
- removed D401: PESD5Zx, SFUSat:PESD57zx, symbol PESD5Zx
- added R512: DNP, SFUSat:R_0402, symbol R
- R411: Digi-Key 311-1.0KJRCT-ND -> (none); Mouser 603-RC0402JR-071KL -> (none); Part Number RC0402JR-071KL -> (none)
Connections:
- wire segments 98 -> 169
Other:
- note removed: "0.062V to 3.038V"
- moved on the sheet: R410, R411
