File: SFUSat-Radio.sch (KiCad schematic (older format))
At the start: 55 parts, among them J1 PC104-8BIT, J2 PC104PTH, J3 PC104PTH, J4 PC104PTH, J5 PC104PTH, J6 SMA, U1 2N7002DW, U101 0433BM15A0001, U111 0915BM15A0001E

Commit message: added 2 temp sensors for the 2 PAs
Parts:
- removed D1, D2: GREEN, SFUSat:LED_0603, symbol LED
- removed R1, R2: 287, SFUSat:R_0402, symbol R
- removed U1: 2N7002DW, SFUSat:SOT-363, symbol 2N7002DW
- added R400, R403, R405, R411, R412, R415: 0R, SFUSat-res:R_0402, symbol R_0R0_0%_0.063W_0402
- added R401, R402, R404, R410, R413, R414: DNP, SFUSat-cap:C_0402, symbol R
- added R? (x2): 1K0, symbol R
Connections:
- net labels added: LB_RX0TX1, SCL, SDA, UB_RX0TX1
- net labels removed: GPIO0, RX0TX1, VDD_3.3
- wire segments 124 -> 157
Other:
- note added: "ADDR: 0x49"
- note added: "ADDR: 0x4A"
- note added: "REF 40*"
- note added: "REF 41*"

Commit message: added test points
Parts:
- added J? (x5): TEST_1P, SFUSat:Measurement_Point_Round-SMD-Pad_Big, symbol TEST_1P
Changed lines of the file:
@@
+	0    1    1    0
+$EndComp
+$Comp
+L TEST_1P J?
+U 1 1 5AD70F8B
+P 4875 2250
+F 0 "J?" H 4875 2520 50  0000 C CNN
+F 1 "TEST_1P" H 4875 2450 50  0000 C CNN
+F 2 "SFUSat:Measurement_Point_Round-SMD-Pad_Big" H 5075 2250 50  0001 C CNN
+F 3 "" H 5075 2250 50  0001 C CNN
+	1    4875 2250
+	0    1    1    0
+$EndComp
+$Comp
+L TEST_1P J?
+U 1 1 5AD79A73
+P 4875 2575
+F 0 "J?" H 4875 2845 50  0000 C CNN
+F 1 "TEST_1P" H 4875 2775 50  0000 C CNN
+F 2 "SFUSat:Measurement_Point_Round-SMD-Pad_Big" H 5075 2575 50  0001 C CNN
+F 3 "" H 5075 2575 50  0001 C CNN
+	1    4875 2575
+	0    1    1    0
+$EndComp
+$Comp
+L TEST_1P J?
+U 1 1 5AD79F8B
+P 4875 1925
+F 0 "J?" H 4875 2195 50  0000 C CNN
+F 1 "TEST_1P" H 4875 2125 50  0000 C CNN
+F 2 "SFUSat:Measurement_Point_Round-SMD-Pad_Big" H 5075 1925 50  0001 C CNN
+F 3 "" H 5075 1925 50  0001 C CNN
+	1    4875 1925
+	0    1    1    0
+$EndComp
+$Comp
+L TEST_1P J?
+U 1 1 5AD7A1DC
+P 4875 1600
+F 0 "J?" H 4875 1870 50  0000 C CNN
+F 1 "TEST_1P" H 4875 1800 50  0000 C CNN
+F 2 "SFUSat:Measurement_Point_Round-SMD-Pad_Big" H 5075 1600 50  0001 C CNN
+F 3 "" H 5075 1600 50  0001 C CNN
+	1    4875 1600
+	0    1    1    0
+$EndComp
+Text Label 4875 1600 2    60   ~ 0
+3V6
+Text Label 4875 1925 2    60   ~ 0
+3V3
+Text Label 4875 2250 2    60   ~ 0
+3V1
+Text Label 4875 2575 2    60   ~ 0
+5V0
+$Comp
+L TEST_1P J?
+U 1 1 5AD837C6
+P 4875 2925
+F 0 "J?" H 4875 3195 50  0000 C CNN
+F 1 "TEST_1P" H 4875 3125 50  0000 C CNN
+F 2 "SFUSat:Measurement_Point_Round-SMD-Pad_Big" H 5075 2925 50  0001 C CNN
+F 3 "" H 5075 2925 50  0001 C CNN
+	1    4875 2925
+	0    1    1    0
+$EndComp
+$Comp
+L GND #PWR?
+U 1 1 5AD83A23
+P 4875 2925
+F 0 "#PWR?" H 4875 2675 50  0001 C CNN
+F 1 "GND" H 4875 2775 50  0000 C CNN
+F 2 "" H 4875 2925 50  0001 C CNN
+F 3 "" H 4875 2925 50  0001 C CNN
+	1    4875 2925
 	0    1    1    0
 $EndComp

Commit message: Added SP3T and 2:4 decoder
Parts:
- added U?: SKY13345-368LF, SFUSat:12-UFQFN-PAD, symbol SKY13345-368LF
- added U?: CD4555BPWR, SFUSat:TSSOP-16, symbol CD4555BPWR
- J1: symbol PC104-8BIT -> PC104-8BIT-RESCUE-SFUSat-Radio
Connections:
- net labels added: V1, V2, V3
- wire segments 157 -> 172
- no-connect marks 0 -> 7
Other:
- note added: "Draw the truth table!\nNote that the state of one band affects\nthe other..."
- moved on the sheet: J6
Changed lines of the file:
@@
 EESchema Schematic File Version 2
+LIBS:SFUSat-Radio-rescue
 LIBS:power
 LIBS:device
@@
 L SMA J6
 U 1 1 5883A1B6
-P 16950 8450
-F 0 "J6" H 17000 8250 60  0000 C TNN
-F 1 "SMA" H 17000 8600 60  0000 C BNN
-F 2 "SFUSat:SMA-Vert-TH" H 16950 8450 60  0001 C CNN
-F 3 "" H 16950 8450 60  0000 C CNN
-	1    16950 8450
+P 18300 8450
+F 0 "J6" H 18350 8250 60  0000 C TNN
+F 1 "SMA" H 18350 8600 60  0000 C BNN
+F 2 "SFUSat:SMA-Vert-TH" H 18300 8450 60  0001 C CNN
+F 3 "" H 18300 8450 60  0000 C CNN
+	1    18300 8450
 	1    0    0    -1
 $EndComp
@@
 L GND #PWR04
 U 1 1 5883A521
-P 16600 8550
-F 0 "#PWR04" H 16600 8300 50  0001 C CNN
-F 1 "GND" H 16600 8400 50  0000 C CNN
-F 2 "" H 16600 8550 50  0000 C CNN
-F 3 "" H 16600 8550 50  0000 C CNN
-	1    16600 8550
-	1    0    0    -1
-$EndComp
-$Comp
-L PC104-8BIT J1
+P 17950 8550
+F 0 "#PWR04" H 17950 8300 50  0001 C CNN
+F 1 "GND" H 17950 8400 50  0000 C CNN
+F 2 "" H 17950 8550 50  0000 C CNN
+F 3 "" H 17950 8550 50  0000 C CNN
+	1    17950 8550
+	1    0    0    -1
+$EndComp
+$Comp
+L PC104-8BIT-RESCUE-SFUSat-Radio J1
 U 1 1 59239648
 P 1750 2500
@@
 	3200 2100 3150 2100
 Wire Wire Line
-	16650 8550 16600 8550
+	18000 8550 17950 8550
 Wire Wire Line
 	7550 1050 7550 1100
@@
 $EndSheet
 $Sheet
-S 15875 8225 600  375
+S 18250 5925 600  375
 U 5A589287
 F0 "Diplexer" 60
 F1 "Diplexer.sch" 60
-F2 "LB" I L 15875 8325 60
-F3 "UB" I L 15875 8500 60
-F4 "Mixed" I R 16475 8400 60
+F2 "LB" I L 18250 6025 60
+F3 "UB" I L 18250 6200 60
+F4 "Mixed" I R 18850 6100 60
 $EndSheet
 $Comp
@@
 Text Notes 10500 9050 0    60   ~ 0
 Copy eval board BOM
-Text Notes 17225 8475 0    60   ~ 0
+Text Notes 18575 8475 0    60   ~ 0
 to antenna
 Text Notes 8525 1200 0    60   ~ 0
@@
 	10300 9575 10375 9575
 Wire Wire Line
-	16475 8400 16650 8400
+	18850 6100 19025 6100
 Wire Wire Line
 	7500 9775 9275 9775
@@
 Text Label 8225 6575 2    60   ~ 0
 LB_RX0TX1
-Text Label 14475 6975 2    60   ~ 0
+Text Label 16600 10000 2    60   ~ 0
 LB_RX0TX1
 Text Label 6300 750  2    60   ~ 0
@@
 	0    1    1    0
 $EndComp
+$Comp
+L SKY13345-368LF U?
+U 1 1 5AADCA71
+P 16550 8400
+F 0 "U?" H 16250 8725 50  0000 L BNN
+F 1 "SKY13345-368LF" H 15675 7775 50  0000 L TNN
+F 2 "SFUSat:12-UFQFN-PAD" H 16550 8400 50  0001 C CNN
+F 3 "" H 16550 8400 50  0001 C CNN
+F 4 "RF/IF and RFID - RF Switches" H 16550 8400 50  0001 C CNN "Categories"
+F 5 "SP3T" H 16550 8400 50  0001 C CNN "Circuit"
+F 6 "DC Blocked" H 16550 8400 50  0001 C CNN "Features"
+F 7 "100MHz" H 16550 8400 50  0001 C CNN "Frequency - Lower"
+F 8 "3.5GHz" H 16550 8400 50  0001 C CNN "Frequency - Upper"
+F 9 "57dBm (typ)" H 16550 8400 50  0001 C CNN "IIP3"
+F 10 "50 Ohm" H 16550 8400 50  0001 C CNN "Impedance"
+F 11 "0.55dB @ 2.5GHz" H 16550 8400 50  0001 C CNN "Insertion Loss @ Frequency"
+F 12 "35dB @ 2.5GHz (typ)" H 16550 8400 50  0001 C CNN "Isolation @ Frequency"
+F 13 "Lead free / RoHS Compliant" H 16550 8400 50  0001 C CNN "Lead Free Status / RoHS Status"
+F 14 "Skyworks Solutions Inc." H 16550 8400 50  0001 C CNN "Manufacturer 1"
+F 15 "SKY13345-368LF" H 16550 8400 50  0001 C CNN "Manufacturer Part Number 1"
+F 16 "16 Weeks" H 16550 8400 50  0001 C CNN "Manufacturer Standard Lead Time 1"
+F 17 "-40°C ~ 85°C" H 16550 8400 50  0001 C CNN "Operating Temperature"
+F 18 "-" H 16550 8400 50  0001 C CNN "P1dB"
+F 19 "12-UFQFN Exposed Pad" H 16550 8400 50  0001 C CNN "Package / Case"
+F 20 "Active" H 16550 8400 50  0001 C CNN "Part Status"
+F 21 "802.11b/g Bluetooth" H 16550 8400 50  0001 C CNN "RF Type"
+F 22 "-" H 16550 8400 50  0001 C CNN "Series"
+F 23 "Digi-Key" H 16550 8400 50  0001 C CNN "Supplier 1"
+F 24 "12-QFN (2x2)" H 16550 8400 50  0001 C CNN "Supplier Device Package"
+F 25 "863-1450-1-ND" H 16550 8400 50  0001 C CNN "Supplier Part Number 1"
+F 26 "Reflective" H 16550 8400 50  0001 C CNN "Topology"
+F 27 "2.5 V ~ 5.5 V" H 16550 8400 50  0001 C CNN "Voltage - Supply"
+	1    16550 8400
+	-1   0    0    -1
+$EndComp
+Wire Wire Line
+	17050 8400 18000 8400
+$Comp
+L GND #PWR?
+U 1 1 5AAE914E
+P 16350 9300
+F 0 "#PWR?" H 16350 9050 50  0001 C CNN
+F 1 "GND" H 16350 9150 50  0000 C CNN
+F 2 "" H 16350 9300 50  0000 C CNN
+F 3 "" H 16350 9300 50  0000 C CNN
+	1    16350 9300
+	1    0    0    -1
+$EndComp
+Wire Wire Line
+	16350 9200 16750 9200
+Connection ~ 16650 9200
+Connection ~ 16550 9200
+Connection ~ 16450 9200
+Wire Wire Line
+	16350 9200 16350 9300
+$Comp
+L CD4555BPWR U?
+U 1 1 5AAEF9C5
+P 17100 10400
+F 0 "U?" H 16900 11025 50  0000 L BNN
+F 1 "CD4555BPWR" H 17125 9875 50  0000 L TNN
+F 2 "SFUSat:TSSOP-16" H 17100 10400 50  0001 C CNN
+F 3 "" H 17100 9750 50  0001 C CNN
+F 4 "4555" H 17100 10400 50  0001 C CNN "Base Part Number"
+F 5 "Integrated Circuits (ICs) - Logic - Signal Switches, Multiplexers, Decoders" H 17100 10400 50  0001 C CNN "Categories"
+F 6 "1 x 2:4" H 17100 10400 50  0001 C CNN "Circuit"
+F 7 "6.8mA, 6.8mA" H 17100 10400 50  0001 C CNN "Current - Output High, Low"
+F 8 "2" H 17100 10400 50  0001 C CNN "Independent Circuits"
+F 9 "Lead free / RoHS Compliant" H 17100 10400 50  0001 C CNN "Lead Free Status / RoHS Status"
+F 10 "Texas Instruments" H 17100 10400 50  0001 C CNN "Manufacturer 1"
+F 11 "CD4555BPWR" H 17100 10400 50  0001 C CNN "Manufacturer Part Number 1"
+F 12 "6 Weeks" H 17100 10400 50  0001 C CNN "Manufacturer Standard Lead Time 1"
+F 13 "Surface Mount" H 17100 10400 50  0001 C CNN "Mounting Type"
+F 14 "-55°C ~ 125°C" H 17100 10400 50  0001 C CNN "Operating Temperature"
+F 15 "16-TSSOP (0.173\", 4.40mm Width)" H 17100 10400 50  0001 C CNN "Package / Case"
+F 16 "Active" H 17100 10400 50  0001 C CNN "Part Status"
+F 17 "4000B" H 17100 10400 50  0001 C CNN "Series"
+F 18 "Digi-Key" H 17100 10400 50  0001 C CNN "Supplier 1"
+F 19 "16-TSSOP" H 17100 10400 50  0001 C CNN "Supplier Device Package"
+F 20 "296-31540-1-ND" H 17100 10400 50  0001 C CNN "Supplier Part Number 1"
+F 21 "Decoder/Demultiplexer" H 17100 10400 50  0001 C CNN "Type"
+F 22 "3 V ~ 18 V" H 17100 10400 50  0001 C CNN "Voltage - Supply"
+F 23 "Dual Supply" H 17100 10400 50  0001 C CNN "Voltage Supply Source"
+	1    17100 10400
+	1    0    0    -1
+$EndComp
+$Comp
+L GND #PWR?
+U 1 1 5AAF1FA7
+P 16600 10700
+F 0 "#PWR?" H 16600 10450 50  0001 C CNN
+F 1 "GND" H 16600 10550 50  0000 C CNN
+F 2 "" H 16600 10700 50  0000 C CNN
+F 3 "" H 16600 10700 50  0000 C CNN
+	1    16600 10700
+	1    0    0    -1
+$EndComp
+Wire Wire Line
+	16700 10200 16600 10200
+Wire Wire Line
+	16600 10200 16600 10700
+Wire Wire Line
+	16700 10600 16600 10600
+Connection ~ 16600 10600
+$Comp
+L GND #PWR?
+U 1 1 5AAF6DF2
+P 17100 11200
+F 0 "#PWR?" H 17100 10950 50  0001 C CNN
+F 1 "GND" H 17100 11050 50  0000 C CNN
+F 2 "" H 17100 11200 50  0000 C CNN
+F 3 "" H 17100 11200 50  0000 C CNN
+	1    17100 11200
+	1    0    0    -1
+$EndComp
+Wire Wire Line
+	17100 11200 17100 11100
+Text Label 16550 7900 2    60   ~ 0
+3V3
+Text Label 17100 9600 2    60   ~ 0
+3V3
+NoConn ~ 16700 10500
+NoConn ~ 16700 10400
+NoConn ~ 17500 10400
+NoConn ~ 17500 10500
+NoConn ~ 17500 10600
+NoConn ~ 17500 10700
+Wire Wire Line
+	16600 10000 16700 10000
+Text Label 16600 10100 2    60   ~ 0
+UB_RX0TX1
+Wire Wire Line
+	16700 10100 16600 10100
+Text Label 16050 8300 2    60   ~ 0
+LB_HP_RX
+Text Label 16050 8400 2    60   ~ 0
+LB_HP_TX
+Text Label 16050 8500 2    60   ~ 0
+UB_HP_TX
+NoConn ~ 17500 10300
+Wire Wire Line
+	17500 10200 17600 10200
+Wire Wire Line
+	17500 10100 17600 10100
+Wire Wire Line
+	17500 10000 17600 10000
+Text Label 17600 10000 0    60   ~ 0
+V1
+Text Label 17600 10100 0    60   ~ 0
+V2
+Text Label 17600 10200 0    60   ~ 0
+V3
+Text Label 17150 8600 0    60   ~ 0
+V1
+Text Label 17150 8700 0    60   ~ 0
+V2
+Text Label 17150 8800 0    60   ~ 0
+V3
+Wire Wire Line
+	17150 8600 17050 8600
+Wire Wire Line
+	17050 8700 17150 8700
+Wire Wire Line
+	17150 8800 17050 8800
+Text Notes 17550 9750 0    60   ~ 0
+Draw the truth table!\nNote that the state of one band affects\nthe other...
 $EndSCHEMATC

Commit message: Added truth table for antenna feed selection
Other:
- note added: "1"
- note added: "Antenna feed select truth table"
- note added: "J1"
- note added: "J2"
- note added: "J3"
- note added: "LB_RX0TX1"
- note added: "NC"
- note added: "UB_RX0TX1"
- note removed: "Draw the truth table!\nNote that the state of one band affects\nthe other..."

Commit message: Added UB PA components
Parts:
- removed C? (x2): 39pF, SFUSat:C_0402, symbol C
- removed C?: 7.5pF, SFUSat:C_0402, symbol C
- removed C?: 15pF, SFUSat:C_0402, symbol C
- removed C?: 10pF, SFUSat:C_0402, symbol C
- removed C?: 12pF, SFUSat:C_0402, symbol C
- removed C?: 0.5pF, SFUSat:C_0402, symbol C
- removed C?: 5.6pF, SFUSat:C_0402, symbol C
- removed C?: 27pF, SFUSat:C_0402, symbol C
- removed L?: 2.7nH, SFUSat:L_0402, symbol L
- removed L? (x3): 0R0, SFUSat:L_0603, symbol L
- removed L?: 5.6nH, SFUSat:L_0402, symbol L
- removed L?: 1.5nH, SFUSat:L_0603, symbol L
- added C?: 15pF, SFUSat-cap:C_0402, symbol C_15p0_5%_50V_NP0_HIQ_0402
- added C? (x2): 39pF, SFUSat-cap:C_0402, symbol C_39p0_5%_50V_NP0_0402
- added C?: 12pF, SFUSat-cap:C_0402, symbol C_12p0_5%_50V_NP0_HIQ_0402
- added C?: 7.5pF, SFUSat-cap:C_0402, symbol C_7p5_0.1pF_50V_NP0_0402
- added C?: 10pF, SFUSat-cap:C_0402, symbol C_10p0_5%_50V_NP0_HIQ_0402
- added C?: 27pF, SFUSat-cap:C_0402, symbol C_27p0_5%_50V_NP0_HIQ_0402
- added C?: 5.6pF, SFUSat-cap:C_0402, symbol C_5p6_0.25pF_50V_NP0_HIQ_0402
- added C?: 0.5pF, SFUSat-cap:C_0402, symbol C_500f0_0.25pF_50V_NP0_HIQ_0402
- added L? (x2): 220R, SFUSat-ind:L_0603, symbol FB_220R0_2A_0603
- added L?: 2.7nH, SFUSat-ind:L_0402, symbol L_2n7_5%_640mA_0402
- added L?: 5.6nH, SFUSat-ind:L_1606, symbol L_5n6_5%_1600mA_1606
- added L?: DNP, SFUSat-ind:L_0603, symbol FB_220R0_2A_0603
- added L?: 1.5nH, SFUSat-ind:L_0603, symbol L_1n5_0.3nH_500mA_0603
- L?: footprint SFUSat:L_0402 -> SFUSat-ind:L_1606
Connections:
- wire segments 172 -> 174
Other:
- note removed: "Copy eval board BOM"
- moved on the sheet: C?, J?

Commit message: Fixed rescue-lib components and CONN_02X05
Parts:
- J1: symbol PC104-8BIT-RESCUE-SFUSat-Radio -> PC104-8BIT
Connections:
- wire segments 174 -> 173
Other:
- note removed: "Need another SPDT switch, bu this one needs to handle 2W"
Changed lines of the file:
@@
 $Descr A2 23386 16535
 encoding utf-8
-Sheet 1 15
+Sheet 1 14
 Title "Digital Transciever Unit with RF Calibration Source"
 Date ""
@@
 $EndComp
 $Comp
-L PC104-8BIT-RESCUE-SFUSat-Radio J1
+L PC104-8BIT J1
 U 1 1 59239648
 P 1750 2500
@@
 F4 "IN" I L 10375 7550 60
 F5 "OUT" I R 11325 7550 60
-$EndSheet
-$Sheet
-S 18250 5925 600  375
-U 5A589287
-F0 "Diplexer" 60
-F1 "Diplexer.sch" 60
-F2 "LB" I L 18250 6025 60
-F3 "UB" I L 18250 6200 60
-F4 "Mixed" I R 18850 6100 60
 $EndSheet
 $Comp
@@
 Text Label 12050 6075 0    60   ~ 0
 LB_HP_RX
-Text Notes 13975 6700 0    60   ~ 0
-Need another SPDT switch, bu this one needs to handle 2W
 Text Notes 5325 5600 0    118  ~ 0
 435Mhz Lower Band (LB)
@@
 	10300 7350 10375 7350
 Wire Wire Line
-	18850 6100 19025 6100
-Wire Wire Line
 	5275 6675 5375 6675
