File: SFUSat-Radio.sch (KiCad schematic (older format))
At the start: 71 parts, among them J1 PC104-8BIT, J2 PC104PTH, J3 PC104PTH, J4 PC104PTH, J5 PC104PTH, J6 SMA, U101 0433BM15A0001, U111 0915BM15A0001E

Commit message: Numbered PA reference designators
Parts:
- gave numbers to parts that had none: 34
Other:
- note added: "REF 4**"
- note added: "REF 5**"
- note removed: "REF 2**"
- note removed: "REF 3**"
Changed lines of the file:
@@
 $Descr A2 23386 16535
 encoding utf-8
-Sheet 1 14
+Sheet 1 12
 Title "Digital Transciever Unit with RF Calibration Source"
 Date ""
@@
 $EndComp
 $Comp
-L C C?
+L C C400
 U 1 1 5AA0EB2B
 P 9425 7550
-F 0 "C?" V 9300 7550 50  0000 C BNN
+F 0 "C400" V 9300 7550 50  0000 C BNN
 F 1 "100pF" V 9550 7550 50  0000 C TNN
 F 2 "SFUSat:C_0402" H 9463 7400 50  0001 C CNN
@@
 $EndComp
 $Comp
-L C C?
+L C C401
 U 1 1 5AA0EB35
 P 10075 7550
-F 0 "C?" V 9950 7550 50  0000 C BNN
+F 0 "C401" V 9950 7550 50  0000 C BNN
 F 1 "22pF" V 10200 7550 50  0000 C TNN
 F 2 "SFUSat:C_0402" H 10113 7400 50  0001 C CNN
@@
 $EndComp
 $Comp
-L L L?
+L L L400
 U 1 1 5AA0EB3F
 P 9775 7850
-F 0 "L?" H 9825 7925 50  0000 L BNN
-F 1 "8.2nH" H 9825 7775 50  0000 L TNN
+F 0 "L400" V 9775 7850 50  0000 C BNN
+F 1 "8.2nH" V 9800 7850 50  0000 C TNN
 F 2 "SFUSat:L_0402" H 9775 7850 50  0001 C CNN
 F 3 "" H 9775 7850 50  0000 C CNN
@@
 $EndComp
 $Comp
-L C C?
+L C C402
 U 1 1 5AA1228A
 P 11450 7800
-F 0 "C?" H 11475 7900 50  0000 L CNN
+F 0 "C402" H 11475 7900 50  0000 L CNN
 F 1 "DNP" H 11475 7700 50  0000 L CNN
 F 2 "SFUSat:C_0402" H 11488 7650 50  0001 C CNN
@@
 $EndComp
 $Comp
-L C C?
+L C C403
 U 1 1 5AA12294
 P 11700 7800
-F 0 "C?" H 11725 7900 50  0000 L CNN
+F 0 "C403" H 11725 7900 50  0000 L CNN
 F 1 "10pF" H 11725 7700 50  0000 L CNN
 F 2 "SFUSat:C_0402" H 11738 7650 50  0001 C CNN
@@
 $EndComp
 $Comp
-L C C?
+L C C404
 U 1 1 5AA1229E
 P 11950 7800
-F 0 "C?" H 11975 7900 50  0000 L CNN
+F 0 "C404" H 11975 7900 50  0000 L CNN
 F 1 "27pF" H 11975 7700 50  0000 L CNN
 F 2 "SFUSat:C_0402" H 11988 7650 50  0001 C CNN
@@
 $EndComp
 $Comp
-L C C?
+L C C407
 U 1 1 5AA122A8
 P 12750 7800
-F 0 "C?" H 12775 7900 50  0000 L CNN
+F 0 "C407" H 12775 7900 50  0000 L CNN
 F 1 "1.2pF" H 12775 7700 50  0000 L CNN
 F 2 "SFUSat:C_0402" H 12788 7650 50  0001 C CNN
@@
 3V6
 $Comp
-L L L?
+L L L402
 U 1 1 5AA122ED
 P 12050 6725
-F 0 "L?" V 12000 6725 50  0000 C CNN
+F 0 "L402" V 12000 6725 50  0000 C CNN
 F 1 "0R0" V 12125 6725 50  0000 C CNN
 F 2 "SFUSat:L_0603" H 12050 6725 50  0001 C CNN
@@
 $EndComp
 $Comp
-L L L?
+L L L403
 U 1 1 5AA122F7
 P 12250 6725
-F 0 "L?" V 12200 6725 50  0000 C CNN
+F 0 "L403" V 12200 6725 50  0000 C CNN
 F 1 "0R0" V 12325 6725 50  0000 C CNN
 F 2 "SFUSat:L_0603" H 12250 6725 50  0001 C CNN
@@
 $EndComp
 $Comp
-L C C?
+L C C406
 U 1 1 5AA12301
 P 12500 7800
-F 0 "C?" H 12525 7900 50  0000 L CNN
+F 0 "C406" H 12525 7900 50  0000 L CNN
 F 1 "10pF" H 12525 7700 50  0000 L CNN
 F 2 "SFUSat:C_0402" H 12538 7650 50  0001 C CNN
@@
 $EndComp
 $Comp
-L C C?
+L C C408
 U 1 1 5AA1230B
 P 13150 7550
-F 0 "C?" V 13025 7550 50  0000 C BNN
+F 0 "C408" V 13025 7550 50  0000 C BNN
 F 1 "100pF" V 13275 7550 50  0000 C TNN
 F 2 "SFUSat:C_0402" H 13188 7400 50  0001 C CNN
@@
 $EndComp
 $Comp
-L C C?
+L C C405
 U 1 1 5AA12315
 P 12300 7050
-F 0 "C?" V 12200 7050 50  0000 C BNN
+F 0 "C405" V 12200 7050 50  0000 C BNN
 F 1 "2.2uF" V 12400 7050 50  0000 C TNN
 F 2 "SFUSat:C_0402" H 12338 6900 50  0001 C CNN
@@
 $EndComp
 $Comp
-L L L?
+L L L404
 U 1 1 5AA1231F
 P 12050 7250
-F 0 "L?" H 12025 7325 50  0000 R BNN
-F 1 "12.55nH" H 12025 7175 50  0000 R TNN
+F 0 "L404" V 12050 7250 50  0000 C BNN
+F 1 "12.55nH" V 12075 7250 50  0000 C TNN
 F 2 "SFUSat-ind:L_1606" H 12050 7250 50  0001 C CNN
 F 3 "" H 12050 7250 50  0000 C CNN
@@
 $EndComp
 $Comp
-L L L?
+L L L401
 U 1 1 5AA12329
 P 11850 6725
-F 0 "L?" V 11800 6725 50  0000 C CNN
+F 0 "L401" V 11800 6725 50  0000 C CNN
 F 1 "0R0" V 11925 6725 50  0000 C CNN
 F 2 "SFUSat:L_0603" H 11850 6725 50  0001 C CNN
@@
 $EndComp
 $Comp
-L L L?
+L L L405
 U 1 1 5AA12333
 P 12300 7550
-F 0 "L?" V 12250 7550 50  0000 C CNN
+F 0 "L405" V 12250 7550 50  0000 C CNN
 F 1 "0R0" V 12375 7550 50  0000 C CNN
 F 2 "SFUSat:L_0603" H 12300 7550 50  0001 C CNN
@@
 Text HLabel 11850 8700 0    60   Input ~ 0
 3V6
-Text Notes 11500 7275 0    60   ~ 0
+Text Notes 11250 7075 0    60   ~ 0
 strange pkg
 Text Notes 11400 9500 0    60   ~ 0
@@
 REF 11*
 Text Notes 10650 6850 0    60   ~ 0
-REF 2**
+REF 4**
 Text Notes 10650 9200 0    60   ~ 0
-REF 3**
+REF 5**
 $Comp
 L SMA J?
@@
 $EndComp
 $Comp
-L SMA J?
+L SMA J500
 U 1 1 5AB823BA
 P 13200 8900
-F 0 "J?" H 13150 8700 60  0000 C CNN
+F 0 "J500" H 13150 8700 60  0000 C CNN
 F 1 "SMA" H 13200 9050 60  0000 C CNN
 F 2 "SFUSat:UFL-R-SMT-1-Coaxial-Connector" H 13400 8950 60  0001 C CNN
@@
 $EndComp
 $Comp
-L SINGLE_0402 U?
+L SINGLE_0402 U500
 U 1 1 5AB823C0
 P 13150 9450
-F 0 "U?" V 13150 9375 60  0000 R CNN
+F 0 "U500" V 13150 9375 60  0000 R CNN
 F 1 "SINGLE_0402" H 13150 9350 60  0001 C TNN
 F 2 "SFUSat:SINGLE_0402" H 13150 9450 60  0001 C CNN
@@
 $EndComp
 $Comp
-L SMA J?
+L SMA J400
 U 1 1 5AB82F29
 P 13200 6725
-F 0 "J?" H 13150 6525 60  0000 C CNN
+F 0 "J400" H 13150 6525 60  0000 C CNN
 F 1 "SMA" H 13200 6875 60  0000 C CNN
 F 2 "SFUSat:UFL-R-SMT-1-Coaxial-Connector" H 13400 6775 60  0001 C CNN
@@
 $EndComp
 $Comp
-L SINGLE_0402 U?
+L SINGLE_0402 U400
 U 1 1 5AB82F2F
 P 13150 7275
-F 0 "U?" V 13150 7200 60  0000 R CNN
+F 0 "U400" V 13150 7200 60  0000 R CNN
 F 1 "SINGLE_0402" H 13150 7175 60  0001 C TNN
 F 2 "SFUSat:SINGLE_0402" H 13150 7275 60  0001 C CNN
@@
 Antenna feed select truth table
 $Comp
-L C_15p0_5%_50V_NP0_HIQ_0402 C?
+L C_15p0_5%_50V_NP0_HIQ_0402 C502
 U 1 1 5AB37D89
 P 11450 10000
-F 0 "C?" H 11450 10050 50  0000 L BNN
+F 0 "C502" H 11450 10050 50  0000 L BNN
 F 1 "15pF" H 11450 9950 50  0000 L TNN
 F 2 "SFUSat-cap:C_0402" H 11450 10000 50  0001 C CNN
@@
 	11450 9850 11450 9750
 $Comp
-L C_12p0_5%_50V_NP0_HIQ_0402 C?
+L C_12p0_5%_50V_NP0_HIQ_0402 C503
 U 1 1 5AB4C042
 P 11700 10000
-F 0 "C?" H 11700 10050 50  0000 L BNN
+F 0 "C503" H 11700 10050 50  0000 L BNN
 F 1 "12pF" H 11700 9950 50  0000 L TNN
 F 2 "SFUSat-cap:C_0402" H 11700 10000 50  0001 C CNN
@@
 $EndComp
 $Comp
-L C_10p0_5%_50V_NP0_HIQ_0402 C?
+L C_10p0_5%_50V_NP0_HIQ_0402 C504
 U 1 1 5AB4CD77
 P 11950 10000
-F 0 "C?" H 11950 10050 50  0000 L BNN
+F 0 "C504" H 11950 10050 50  0000 L BNN
 F 1 "10pF" H 11950 9950 50  0000 L TNN
 F 2 "SFUSat-cap:C_0402" H 11950 10000 50  0001 C CNN
@@
 $EndComp
 $Comp
-L C_27p0_5%_50V_NP0_HIQ_0402 C?
+L C_27p0_5%_50V_NP0_HIQ_0402 C505
 U 1 1 5AB53C7D
 P 12300 9250
-F 0 "C?" V 12200 9250 50  0000 C BNN
+F 0 "C505" V 12200 9250 50  0000 C BNN
 F 1 "27pF" V 12400 9250 50  0000 C TNN
 F 2 "SFUSat-cap:C_0402" H 12300 9250 50  0001 C CNN
@@
 	12050 9250 12150 9250
 $Comp
-L L_1n5_0.3nH_500mA_0603 L?
+L L_1n5_0.3nH_500mA_0603 L505
 U 1 1 5AB5746D
 P 12300 9750
-F 0 "L?" H 12300 9800 50  0000 C BNN
+F 0 "L505" H 12300 9800 50  0000 C BNN
 F 1 "1.5nH" H 12300 9700 50  0000 C TNN
 F 2 "SFUSat-ind:L_0603" H 12300 9750 50  0001 C CNN
@@
 $EndComp
 $Comp
-L C_5p6_0.25pF_50V_NP0_HIQ_0402 C?
+L C_5p6_0.25pF_50V_NP0_HIQ_0402 C506
 U 1 1 5AB57EB2
 P 12500 10000
-F 0 "C?" H 12500 10050 50  0000 L BNN
+F 0 "C506" H 12500 10050 50  0000 L BNN
 F 1 "5.6pF" H 12500 9950 50  0000 L TNN
 F 2 "SFUSat-cap:C_0402" H 12500 10000 50  0001 C CNN
@@
 $EndComp
 $Comp
-L C_500f0_0.25pF_50V_NP0_HIQ_0402 C?
+L C_500f0_0.25pF_50V_NP0_HIQ_0402 C507
 U 1 1 5AB5816E
 P 12750 10000
-F 0 "C?" H 12750 10050 50  0000 L BNN
+F 0 "C507" H 12750 10050 50  0000 L BNN
 F 1 "0.5pF" H 12750 9950 50  0000 L TNN
 F 2 "SFUSat-cap:C_0402" H 12750 10000 50  0001 C CNN
@@
 $EndComp
 $Comp
-L C_39p0_5%_50V_NP0_0402 C?
+L C_39p0_5%_50V_NP0_0402 C508
 U 1 1 5AB59E70
 P 13150 9750
-F 0 "C?" V 13050 9750 50  0000 C BNN
+F 0 "C508" V 13050 9750 50  0000 C BNN
 F 1 "39pF" V 13250 9750 50  0000 C TNN
 F 2 "SFUSat-cap:C_0402" H 13150 9750 50  0001 C CNN
@@
 $EndComp
 $Comp
-L C_39p0_5%_50V_NP0_0402 C?
+L C_39p0_5%_50V_NP0_0402 C500
 U 1 1 5AB3D56D
 P 9400 9750
-F 0 "C?" V 9300 9750 50  0000 C BNN
+F 0 "C500" V 9300 9750 50  0000 C BNN
 F 1 "39pF" V 9500 9750 50  0000 C TNN
 F 2 "SFUSat-cap:C_0402" H 9400 9750 50  0001 C CNN
@@
 Connection ~ 8100 9750
 $Comp
-L C_7p5_0.1pF_50V_NP0_0402 C?
+L C_7p5_0.1pF_50V_NP0_0402 C501
 U 1 1 5AB4C19D
 P 10100 9750
-F 0 "C?" V 10000 9750 50  0000 C BNN
+F 0 "C501" V 10000 9750 50  0000 C BNN
 F 1 "7.5pF" V 10200 9750 50  0000 C TNN
 F 2 "SFUSat-cap:C_0402" H 10100 9750 50  0001 C CNN
@@
 $EndComp
 $Comp
-L FB_220R0_2A_0603 L?
+L FB_220R0_2A_0603 L502
 U 1 1 5AB3890A
 P 12050 8900
-F 0 "L?" H 12050 8900 50  0000 C TNN
+F 0 "L502" H 12050 8900 50  0000 C TNN
 F 1 "220R" H 12050 8950 50  0000 C BNN
 F 2 "SFUSat-ind:L_0603" H 12050 8900 50  0001 C CNN
@@
 $EndComp
 $Comp
-L FB_220R0_2A_0603 L?
+L FB_220R0_2A_0603 L501
 U 1 1 5AB3A707
 P 11850 8900
-F 0 "L?" H 11850 8900 50  0000 C TNN
+F 0 "L501" H 11850 8900 50  0000 C TNN
 F 1 "220R" H 11850 8950 50  0000 C BNN
 F 2 "SFUSat-ind:L_0603" H 11850 8900 50  0001 C CNN
@@
 $EndComp
 $Comp
-L FB_220R0_2A_0603 L?
+L FB_220R0_2A_0603 L503
 U 1 1 5AB4346C
 P 12250 8900
-F 0 "L?" H 12250 8900 50  0000 C TNN
+F 0 "L503" H 12250 8900 50  0000 C TNN
 F 1 "DNP" H 12250 8950 50  0000 C BNN
 F 2 "SFUSat-ind:L_0603" H 12250 8900 50  0001 C CNN
@@
 	11850 8700 12250 8700
 $Comp
-L L_5n6_5%_1600mA_1606 L?
+L L_5n6_5%_1600mA_1606 L504
 U 1 1 5AB3A5ED
 P 12050 9450
-F 0 "L?" H 12050 9450 50  0000 C TNN
+F 0 "L504" H 12050 9450 50  0000 C TNN
 F 1 "5.6nH" H 12050 9500 50  0000 C BNN
 F 2 "SFUSat-ind:L_1606" H 12050 9450 50  0001 C CNN
@@
 $EndComp
 $Comp
-L L_2n7_5%_640mA_0402 L?
+L L_2n7_5%_640mA_0402 L500
 U 1 1 5AB390BC
 P 9750 10050
-F 0 "L?" H 9750 10050 50  0000 C TNN
+F 0 "L500" H 9750 10050 50  0000 C TNN
 F 1 "2.7nH" H 9750 10100 50  0000 C BNN
 F 2 "SFUSat-ind:L_0402" H 9750 10050 50  0001 C CNN

Commit message: Changed temp sense reference designator prefix
Initally overlapped with PA LB reference designator prefix
Parts:
- renumbered R400 to R600, R401 to R601, R402 to R602, R403 to R603, R404 to R604, R405 to R605, R410 to R610, R411 to R611, R412 to R612, R413 to R613, R414 to R614, R415 to R615
Other:
- note added: "REF 60*"
- note added: "REF 61*"
- note removed: "REF 40*"
- note removed: "REF 41*"
