File: CC1101.sch (KiCad schematic (older format))
At the start: 13 parts, among them U100 CC1101-Q1, X100 NX3225GA

Commit message: Annotated the schematics
Parts:
- gave numbers to parts that had none: 2
Changed lines of the file:
@@
 $Descr A4 11693 8268
 encoding utf-8
-Sheet 10 12
+Sheet 8 12
 Title ""
 Date ""
@@
 P 4500 4500
 AR Path="/5AA44392/592A0E9A" Ref="U100"  Part="1"
-AR Path="/5AA72383/592A0E9A" Ref="U100"  Part="1"
-F 0 "U100" H 4500 4550 60  0000 C BNN
+AR Path="/5AA72383/592A0E9A" Ref="U110"  Part="1"
+F 0 "U110" H 4500 4550 60  0000 C BNN
 F 1 "CC1101-Q1" H 4500 4450 60  0000 C TNN
 F 2 "SFUSat:CC1101-Q1" H 4350 4500 60  0001 C CNN
@@
 $EndComp
 $Comp
-L GND #PWR065
+L GND #PWR86
 U 1 1 592A76F5
 P 4150 5625
-AR Path="/5AA44392/592A76F5" Ref="#PWR065"  Part="1"
-AR Path="/5AA72383/592A76F5" Ref="#PWR065"  Part="1"
-F 0 "#PWR065" H 4150 5375 50  0001 C CNN
+AR Path="/5AA44392/592A76F5" Ref="#PWR86"  Part="1"
+AR Path="/5AA72383/592A76F5" Ref="#PWR97"  Part="1"
+F 0 "#PWR97" H 4150 5375 50  0001 C CNN
 F 1 "GND" H 4150 5475 50  0000 C CNN
 F 2 "" H 4150 5625 50  0000 C CNN
@@
 $EndComp
 $Comp
-L GND #PWR066
+L GND #PWR87
 U 1 1 592A8C09
 P 4750 6050
-AR Path="/5AA44392/592A8C09" Ref="#PWR066"  Part="1"
-AR Path="/5AA72383/592A8C09" Ref="#PWR066"  Part="1"
-F 0 "#PWR066" H 4750 5800 50  0001 C CNN
+AR Path="/5AA44392/592A8C09" Ref="#PWR87"  Part="1"
+AR Path="/5AA72383/592A8C09" Ref="#PWR98"  Part="1"
+F 0 "#PWR98" H 4750 5800 50  0001 C CNN
 F 1 "GND" H 4750 5900 50  0000 C CNN
 F 2 "" H 4750 6050 50  0000 C CNN
@@
 $EndComp
 $Comp
-L GND #PWR067
+L GND #PWR90
 U 1 1 592ACEFE
 P 5950 5175
-AR Path="/5AA44392/592ACEFE" Ref="#PWR067"  Part="1"
-AR Path="/5AA72383/592ACEFE" Ref="#PWR067"  Part="1"
-F 0 "#PWR067" H 5950 4925 50  0001 C CNN
+AR Path="/5AA44392/592ACEFE" Ref="#PWR90"  Part="1"
+AR Path="/5AA72383/592ACEFE" Ref="#PWR101"  Part="1"
+F 0 "#PWR101" H 5950 4925 50  0001 C CNN
 F 1 "GND" H 5950 5025 50  0000 C CNN
 F 2 "" H 5950 5175 50  0000 C CNN
@@
 $EndComp
 $Comp
-L GND #PWR069
+L GND #PWR85
 U 1 1 592AE8E9
 P 3525 2875
-AR Path="/5AA44392/592AE8E9" Ref="#PWR069"  Part="1"
-AR Path="/5AA72383/592AE8E9" Ref="#PWR069"  Part="1"
-F 0 "#PWR069" H 3525 2625 50  0001 C CNN
+AR Path="/5AA44392/592AE8E9" Ref="#PWR85"  Part="1"
+AR Path="/5AA72383/592AE8E9" Ref="#PWR96"  Part="1"
+F 0 "#PWR96" H 3525 2625 50  0001 C CNN
 F 1 "GND" H 3525 2725 50  0000 C CNN
 F 2 "" H 3525 2875 50  0000 C CNN
@@
 $EndComp
 $Comp
-L GND #PWR070
+L GND #PWR81
 U 1 1 592A789E
 P 1400 3850
-AR Path="/5AA44392/592A789E" Ref="#PWR070"  Part="1"
-AR Path="/5AA72383/592A789E" Ref="#PWR070"  Part="1"
-F 0 "#PWR070" H 1400 3600 50  0001 C CNN
+AR Path="/5AA44392/592A789E" Ref="#PWR81"  Part="1"
+AR Path="/5AA72383/592A789E" Ref="#PWR92"  Part="1"
+F 0 "#PWR92" H 1400 3600 50  0001 C CNN
 F 1 "GND" H 1400 3700 50  0000 C CNN
 F 2 "" H 1400 3850 50  0000 C CNN
@@
 $EndComp
 $Comp
-L GND #PWR071
+L GND #PWR82
 U 1 1 592A7939
 P 1400 4450
-AR Path="/5AA44392/592A7939" Ref="#PWR071"  Part="1"
-AR Path="/5AA72383/592A7939" Ref="#PWR071"  Part="1"
-F 0 "#PWR071" H 1400 4200 50  0001 C CNN
+AR Path="/5AA44392/592A7939" Ref="#PWR82"  Part="1"
+AR Path="/5AA72383/592A7939" Ref="#PWR93"  Part="1"
+F 0 "#PWR93" H 1400 4200 50  0001 C CNN
 F 1 "GND" H 1400 4300 50  0000 C CNN
 F 2 "" H 1400 4450 50  0000 C CNN
@@
 $EndComp
 $Comp
-L GND #PWR075
+L GND #PWR83
 U 1 1 592F1736
 P 3525 2000
-AR Path="/5AA44392/592F1736" Ref="#PWR075"  Part="1"
-AR Path="/5AA72383/592F1736" Ref="#PWR075"  Part="1"
-F 0 "#PWR075" H 3525 1750 50  0001 C CNN
+AR Path="/5AA44392/592F1736" Ref="#PWR83"  Part="1"
+AR Path="/5AA72383/592F1736" Ref="#PWR94"  Part="1"
+F 0 "#PWR94" H 3525 1750 50  0001 C CNN
 F 1 "GND" H 3525 1850 50  0000 C CNN
 F 2 "" H 3525 2000 50  0000 C CNN
@@
 $EndComp
 $Comp
-L GND #PWR076
+L GND #PWR84
 U 1 1 592F173C
 P 3525 2425
-AR Path="/5AA44392/592F173C" Ref="#PWR076"  Part="1"
-AR Path="/5AA72383/592F173C" Ref="#PWR076"  Part="1"
-F 0 "#PWR076" H 3525 2175 50  0001 C CNN
+AR Path="/5AA44392/592F173C" Ref="#PWR84"  Part="1"
+AR Path="/5AA72383/592F173C" Ref="#PWR95"  Part="1"
+F 0 "#PWR95" H 3525 2175 50  0001 C CNN
 F 1 "GND" H 3525 2275 50  0000 C CNN
 F 2 "" H 3525 2425 50  0000 C CNN
@@
 $EndComp
 $Comp
-L GND #PWR077
+L GND #PWR89
 U 1 1 592F1E87
 P 5475 3300
-AR Path="/5AA44392/592F1E87" Ref="#PWR077"  Part="1"
-AR Path="/5AA72383/592F1E87" Ref="#PWR077"  Part="1"
-F 0 "#PWR077" H 5475 3050 50  0001 C CNN
+AR Path="/5AA44392/592F1E87" Ref="#PWR89"  Part="1"
+AR Path="/5AA72383/592F1E87" Ref="#PWR100"  Part="1"
+F 0 "#PWR100" H 5475 3050 50  0001 C CNN
 F 1 "GND" H 5475 3150 50  0000 C CNN
 F 2 "" H 5475 3300 50  0000 C CNN
@@
 $EndComp
 $Comp
-L GND #PWR078
+L GND #PWR88
 U 1 1 592F1E8D
 P 5475 2875
-AR Path="/5AA44392/592F1E8D" Ref="#PWR078"  Part="1"
-AR Path="/5AA72383/592F1E8D" Ref="#PWR078"  Part="1"
-F 0 "#PWR078" H 5475 2625 50  0001 C CNN
+AR Path="/5AA44392/592F1E8D" Ref="#PWR88"  Part="1"
+AR Path="/5AA72383/592F1E8D" Ref="#PWR99"  Part="1"
+F 0 "#PWR99" H 5475 2625 50  0001 C CNN
 F 1 "GND" H 5475 2725 50  0000 C CNN
 F 2 "" H 5475 2875 50  0000 C CNN
@@
 OP_3.3
 $Comp
-L GND #PWR?
+L GND #PWR91
 U 1 1 5AAD2BB4
 P 7650 1950
-AR Path="/5AA44392/5AAD2BB4" Ref="#PWR?"  Part="1"
-AR Path="/5AA72383/5AAD2BB4" Ref="#PWR?"  Part="1"
-F 0 "#PWR?" H 7650 1700 50  0001 C CNN
+AR Path="/5AA44392/5AAD2BB4" Ref="#PWR91"  Part="1"
+AR Path="/5AA72383/5AAD2BB4" Ref="#PWR102"  Part="1"
+F 0 "#PWR102" H 7650 1700 50  0001 C CNN
 F 1 "GND" H 7650 1800 50  0000 C CNN
 F 2 "" H 7650 1950 50  0000 C CNN
@@
 VDD_3.3
 $Comp
-L CONN_01X03 J?
+L CONN_01X03 J19
 U 1 1 5ABB51CC
 P 8300 3200
-AR Path="/5AA44392/5ABB51CC" Ref="J?"  Part="1"
-AR Path="/5AA72383/5ABB51CC" Ref="J?"  Part="1"
+AR Path="/5AA44392/5ABB51CC" Ref="J19"  Part="1"
+AR Path="/5AA72383/5ABB51CC" Ref="J20"  Part="1"
 AR Path="/5ABB51CC" Ref="J?"  Part="1"
-F 0 "J?" H 8300 3400 50  0000 C CNN
+F 0 "J20" H 8300 3400 50  0000 C CNN
 F 1 "Conn_01x03" H 8300 3000 50  0000 C CNN
 F 2 "Socket_Strips:Socket_Strip_Straight_1x03_Pitch2.54mm" H 8300 3200 50  0001 C CNN
@@
 If the debugger power supply is used,\n the radio must only be operated through \nthe u.fl debug ports adjasent to the balun.
 $Comp
-L CONN_02X05_SHRD U?
+L CONN_02X05_SHRD U13
 U 1 1 5AB496AE
 P 8250 2150
-AR Path="/5AA72383/5AB496AE" Ref="U?"  Part="1"
-AR Path="/5AA44392/5AB496AE" Ref="U?"  Part="1"
-F 0 "U?" H 8250 2450 50  0000 C BNN
+AR Path="/5AA72383/5AB496AE" Ref="U13"  Part="1"
+AR Path="/5AA44392/5AB496AE" Ref="U12"  Part="1"
+F 0 "U13" H 8250 2450 50  0000 C BNN
 F 1 "CONN_02X05_SHRD" H 8300 1850 50  0000 C TNN
 F 2 "SFUSat:Socket_Strip_Straight_2x05" H 8150 2350 50  0001 C CNN
