File: CC1101.sch (KiCad schematic (older format))
At the start: 13 parts, among them J19 Conn_01x03, U100 CC1101-Q1, U13 CONN_02X05_SHRD, X100 NX3225GA

Commit message: layed out indicator lights
Changed lines of the file:
@@
 $Descr A4 11693 8268
 encoding utf-8
-Sheet 7 15
+Sheet 6 15
 Title ""
 Date ""
@@
 AR Path="/5AA44392/592A0E9A" Ref="U100"  Part="1"
 AR Path="/5AA72383/592A0E9A" Ref="U110"  Part="1"
-F 0 "U100" H 4500 4550 60  0000 C BNN
+F 0 "U110" H 4500 4550 60  0000 C BNN
 F 1 "CC1101-Q1" H 4500 4450 60  0000 C TNN
 F 2 "SFUSat:CC1101-Q1" H 4350 4500 60  0001 C CNN
@@
 $EndComp
 $Comp
-L GND #PWR075
+L GND #PWR81
 U 1 1 592A76F5
 P 4150 5625
-AR Path="/5AA44392/592A76F5" Ref="#PWR075"  Part="1"
-AR Path="/5AA72383/592A76F5" Ref="#PWR086"  Part="1"
-F 0 "#PWR075" H 4150 5375 50  0001 C CNN
+AR Path="/5AA44392/592A76F5" Ref="#PWR81"  Part="1"
+AR Path="/5AA72383/592A76F5" Ref="#PWR92"  Part="1"
+F 0 "#PWR92" H 4150 5375 50  0001 C CNN
 F 1 "GND" H 4150 5475 50  0000 C CNN
 F 2 "" H 4150 5625 50  0000 C CNN
@@
 AR Path="/5AA44392/592A885A" Ref="C106"  Part="1"
 AR Path="/5AA72383/592A885A" Ref="C116"  Part="1"
-F 0 "C106" H 4775 5875 50  0000 L CNN
+F 0 "C116" H 4775 5875 50  0000 L CNN
 F 1 "100nF" H 4775 5675 50  0000 L CNN
 F 2 "SFUSat:C_0402" H 4788 5625 50  0001 C CNN
@@
 $EndComp
 $Comp
-L GND #PWR076
+L GND #PWR82
 U 1 1 592A8C09
 P 4750 6050
-AR Path="/5AA44392/592A8C09" Ref="#PWR076"  Part="1"
-AR Path="/5AA72383/592A8C09" Ref="#PWR087"  Part="1"
-F 0 "#PWR076" H 4750 5800 50  0001 C CNN
+AR Path="/5AA44392/592A8C09" Ref="#PWR82"  Part="1"
+AR Path="/5AA72383/592A8C09" Ref="#PWR93"  Part="1"
+F 0 "#PWR93" H 4750 5800 50  0001 C CNN
 F 1 "GND" H 4750 5900 50  0000 C CNN
 F 2 "" H 4750 6050 50  0000 C CNN
@@
 AR Path="/5AA44392/592ACE93" Ref="R100"  Part="1"
 AR Path="/5AA72383/592ACE93" Ref="R110"  Part="1"
-F 0 "R100" H 6000 4900 50  0000 L CNN
+F 0 "R110" H 6000 4900 50  0000 L CNN
 F 1 "56k" V 5950 4900 50  0000 C CNN
 F 2 "SFUSat:R_0402" V 5880 4900 50  0001 C CNN
@@
 $EndComp
 $Comp
-L GND #PWR077
+L GND #PWR85
 U 1 1 592ACEFE
 P 5950 5175
-AR Path="/5AA44392/592ACEFE" Ref="#PWR077"  Part="1"
-AR Path="/5AA72383/592ACEFE" Ref="#PWR088"  Part="1"
-F 0 "#PWR077" H 5950 4925 50  0001 C CNN
+AR Path="/5AA44392/592ACEFE" Ref="#PWR85"  Part="1"
+AR Path="/5AA72383/592ACEFE" Ref="#PWR96"  Part="1"
+F 0 "#PWR96" H 5950 4925 50  0001 C CNN
 F 1 "GND" H 5950 5025 50  0000 C CNN
 F 2 "" H 5950 5175 50  0000 C CNN
@@
 $EndComp
 $Comp
-L GND #PWR078
+L GND #PWR80
 U 1 1 592AE8E9
 P 3525 2875
-AR Path="/5AA44392/592AE8E9" Ref="#PWR078"  Part="1"
-AR Path="/5AA72383/592AE8E9" Ref="#PWR089"  Part="1"
-F 0 "#PWR078" H 3525 2625 50  0001 C CNN
+AR Path="/5AA44392/592AE8E9" Ref="#PWR80"  Part="1"
+AR Path="/5AA72383/592AE8E9" Ref="#PWR91"  Part="1"
+F 0 "#PWR91" H 3525 2625 50  0001 C CNN
 F 1 "GND" H 3525 2725 50  0000 C CNN
 F 2 "" H 3525 2875 50  0000 C CNN
@@
 AR Path="/5AA44392/592A69DC" Ref="X100"  Part="1"
 AR Path="/5AA72383/592A69DC" Ref="X110"  Part="1"
-F 0 "X100" V 2000 4325 60  0000 L CNN
+F 0 "X110" V 2000 4325 60  0000 L CNN
 F 1 "NX3225GA" H 2000 3950 60  0000 C TNN
 F 2 "SFUSat:NX3225GA" H 2000 4150 60  0001 C CNN
@@
 AR Path="/5AA44392/592A70F9" Ref="C101"  Part="1"
 AR Path="/5AA72383/592A70F9" Ref="C111"  Part="1"
-F 0 "C101" V 1700 3850 50  0000 C CNN
+F 0 "C111" V 1700 3850 50  0000 C CNN
 F 1 "12pF" V 1400 3850 50  0000 C CNN
 F 2 "SFUSat:C_0402" H 1588 3700 50  0001 C CNN
@@
 AR Path="/5AA44392/592A730F" Ref="C102"  Part="1"
 AR Path="/5AA72383/592A730F" Ref="C112"  Part="1"
-F 0 "C102" V 1700 4450 50  0000 C CNN
+F 0 "C112" V 1700 4450 50  0000 C CNN
 F 1 "15pF" V 1400 4450 50  0000 C CNN
 F 2 "SFUSat:C_0402" H 1588 4300 50  0001 C CNN
@@
 $EndComp
 $Comp
-L GND #PWR079
+L GND #PWR76
 U 1 1 592A789E
 P 1400 3850
-AR Path="/5AA44392/592A789E" Ref="#PWR079"  Part="1"
-AR Path="/5AA72383/592A789E" Ref="#PWR090"  Part="1"
-F 0 "#PWR079" H 1400 3600 50  0001 C CNN
+AR Path="/5AA44392/592A789E" Ref="#PWR76"  Part="1"
+AR Path="/5AA72383/592A789E" Ref="#PWR87"  Part="1"
+F 0 "#PWR87" H 1400 3600 50  0001 C CNN
 F 1 "GND" H 1400 3700 50  0000 C CNN
 F 2 "" H 1400 3850 50  0000 C CNN
@@
 $EndComp
 $Comp
-L GND #PWR080
+L GND #PWR77
 U 1 1 592A7939
 P 1400 4450
-AR Path="/5AA44392/592A7939" Ref="#PWR080"  Part="1"
-AR Path="/5AA72383/592A7939" Ref="#PWR091"  Part="1"
-F 0 "#PWR080" H 1400 4200 50  0001 C CNN
+AR Path="/5AA44392/592A7939" Ref="#PWR77"  Part="1"
+AR Path="/5AA72383/592A7939" Ref="#PWR88"  Part="1"
+F 0 "#PWR88" H 1400 4200 50  0001 C CNN
 F 1 "GND" H 1400 4300 50  0000 C CNN
 F 2 "" H 1400 4450 50  0000 C CNN
@@
 AR Path="/5AA44392/592F0537" Ref="C105"  Part="1"
 AR Path="/5AA72383/592F0537" Ref="C115"  Part="1"
-F 0 "C105" V 3825 2875 50  0000 C CNN
+F 0 "C115" V 3825 2875 50  0000 C CNN
 F 1 "100nF" V 3525 2875 50  0000 C CNN
 F 2 "SFUSat:C_0402" H 3713 2725 50  0001 C CNN
@@
 $EndComp
 $Comp
-L GND #PWR081
+L GND #PWR78
 U 1 1 592F1736
 P 3525 2000
-AR Path="/5AA44392/592F1736" Ref="#PWR081"  Part="1"
-AR Path="/5AA72383/592F1736" Ref="#PWR092"  Part="1"
-F 0 "#PWR081" H 3525 1750 50  0001 C CNN
+AR Path="/5AA44392/592F1736" Ref="#PWR78"  Part="1"
+AR Path="/5AA72383/592F1736" Ref="#PWR89"  Part="1"
+F 0 "#PWR89" H 3525 1750 50  0001 C CNN
 F 1 "GND" H 3525 1850 50  0000 C CNN
 F 2 "" H 3525 2000 50  0000 C CNN
@@
 $EndComp
 $Comp
-L GND #PWR082
+L GND #PWR79
 U 1 1 592F173C
 P 3525 2425
-AR Path="/5AA44392/592F173C" Ref="#PWR082"  Part="1"
-AR Path="/5AA72383/592F173C" Ref="#PWR093"  Part="1"
-F 0 "#PWR082" H 3525 2175 50  0001 C CNN
+AR Path="/5AA44392/592F173C" Ref="#PWR79"  Part="1"
+AR Path="/5AA72383/592F173C" Ref="#PWR90"  Part="1"
+F 0 "#PWR90" H 3525 2175 50  0001 C CNN
 F 1 "GND" H 3525 2275 50  0000 C CNN
 F 2 "" H 3525 2425 50  0000 C CNN
@@
 AR Path="/5AA44392/592F1742" Ref="C104"  Part="1"
 AR Path="/5AA72383/592F1742" Ref="C114"  Part="1"
-F 0 "C104" V 3825 2425 50  0000 C CNN
+F 0 "C114" V 3825 2425 50  0000 C CNN
 F 1 "220pF" V 3525 2425 50  0000 C CNN
 F 2 "SFUSat:C_0402" H 3713 2275 50  0001 C CNN
@@
 AR Path="/5AA44392/592F1748" Ref="C103"  Part="1"
 AR Path="/5AA72383/592F1748" Ref="C113"  Part="1"
-F 0 "C103" V 3825 2000 50  0000 C CNN
+F 0 "C113" V 3825 2000 50  0000 C CNN
 F 1 "100nF" V 3525 2000 50  0000 C CNN
 F 2 "SFUSat:C_0402" H 3713 1850 50  0001 C CNN
@@
 $EndComp
 $Comp
-L GND #PWR083
+L GND #PWR84
 U 1 1 592F1E87
 P 5475 3300
-AR Path="/5AA44392/592F1E87" Ref="#PWR083"  Part="1"
-AR Path="/5AA72383/592F1E87" Ref="#PWR094"  Part="1"
-F 0 "#PWR083" H 5475 3050 50  0001 C CNN
+AR Path="/5AA44392/592F1E87" Ref="#PWR84"  Part="1"
+AR Path="/5AA72383/592F1E87" Ref="#PWR95"  Part="1"
+F 0 "#PWR95" H 5475 3050 50  0001 C CNN
 F 1 "GND" H 5475 3150 50  0000 C CNN
 F 2 "" H 5475 3300 50  0000 C CNN
@@
 $EndComp
 $Comp
-L GND #PWR084
+L GND #PWR83
 U 1 1 592F1E8D
 P 5475 2875
-AR Path="/5AA44392/592F1E8D" Ref="#PWR084"  Part="1"
-AR Path="/5AA72383/592F1E8D" Ref="#PWR095"  Part="1"
-F 0 "#PWR084" H 5475 2625 50  0001 C CNN
+AR Path="/5AA44392/592F1E8D" Ref="#PWR83"  Part="1"
+AR Path="/5AA72383/592F1E8D" Ref="#PWR94"  Part="1"
+F 0 "#PWR94" H 5475 2625 50  0001 C CNN
 F 1 "GND" H 5475 2725 50  0000 C CNN
 F 2 "" H 5475 2875 50  0000 C CNN
@@
 AR Path="/5AA44392/592F1E93" Ref="C107"  Part="1"
 AR Path="/5AA72383/592F1E93" Ref="C117"  Part="1"
-F 0 "C107" V 5175 2875 50  0000 C CNN
+F 0 "C117" V 5175 2875 50  0000 C CNN
 F 1 "100nF" V 5475 2875 50  0000 C CNN
 F 2 "SFUSat:C_0402" H 5363 2725 50  0001 C CNN
@@
 AR Path="/5AA44392/592F1E99" Ref="C100"  Part="1"
 AR Path="/5AA72383/592F1E99" Ref="C110"  Part="1"
-F 0 "C100" V 5175 3300 50  0000 C CNN
+F 0 "C110" V 5175 3300 50  0000 C CNN
 F 1 "100nF" V 5475 3300 50  0000 C CNN
 F 2 "SFUSat:C_0402" H 5363 3150 50  0001 C CNN
@@
 OP_3.3
 $Comp
-L GND #PWR085
+L GND #PWR86
 U 1 1 5AAD2BB4
 P 7650 1950
-AR Path="/5AA44392/5AAD2BB4" Ref="#PWR085"  Part="1"
-AR Path="/5AA72383/5AAD2BB4" Ref="#PWR096"  Part="1"
-F 0 "#PWR085" H 7650 1700 50  0001 C CNN
+AR Path="/5AA44392/5AAD2BB4" Ref="#PWR86"  Part="1"
+AR Path="/5AA72383/5AAD2BB4" Ref="#PWR97"  Part="1"
+F 0 "#PWR97" H 7650 1700 50  0001 C CNN
 F 1 "GND" H 7650 1800 50  0000 C CNN
 F 2 "" H 7650 1950 50  0000 C CNN
@@
 AR Path="/5AA72383/5ABB51CC" Ref="J20"  Part="1"
 AR Path="/5ABB51CC" Ref="J?"  Part="1"
-F 0 "J19" H 8300 3400 50  0000 C CNN
+F 0 "J20" H 8300 3400 50  0000 C CNN
 F 1 "Conn_01x03" H 8300 3000 50  0000 C CNN
 F 2 "Socket_Strips:Socket_Strip_Straight_1x03_Pitch2.54mm" H 8300 3200 50  0001 C CNN
@@
 AR Path="/5AA72383/5AB496AE" Ref="U13"  Part="1"
 AR Path="/5AA44392/5AB496AE" Ref="U12"  Part="1"
-F 0 "U12" H 8250 2450 50  0000 C BNN
+F 0 "U13" H 8250 2450 50  0000 C BNN
 F 1 "CONN_02X05_SHRD" H 8300 1850 50  0000 C TNN
 F 2 "SFUSat:Socket_Strip_Straight_2x05" H 8150 2350 50  0001 C CNN
