File: CC1101.sch (KiCad schematic (older format))
At the start: 13 parts, among them J19 Conn_01x03, U100 CC1101-Q1, U13 CONN_02X05_SHRD, X100 NX3225GA

Commit message: Continued power floods
Changed lines of the file:
@@
 AR Path="/5AA44392/592A0E9A" Ref="U100"  Part="1"
 AR Path="/5AA72383/592A0E9A" Ref="U110"  Part="1"
-F 0 "U110" H 4500 4550 60  0000 C BNN
+F 0 "U100" H 4500 4550 60  0000 C BNN
 F 1 "CC1101-Q1" H 4500 4450 60  0000 C TNN
 F 2 "SFUSat:CC1101-Q1" H 4350 4500 60  0001 C CNN
@@
 AR Path="/5AA44392/592A76F5" Ref="#PWR077"  Part="1"
 AR Path="/5AA72383/592A76F5" Ref="#PWR088"  Part="1"
-F 0 "#PWR088" H 4150 5375 50  0001 C CNN
+F 0 "#PWR077" H 4150 5375 50  0001 C CNN
 F 1 "GND" H 4150 5475 50  0000 C CNN
 F 2 "" H 4150 5625 50  0000 C CNN
@@
 AR Path="/5AA44392/592A885A" Ref="C106"  Part="1"
 AR Path="/5AA72383/592A885A" Ref="C116"  Part="1"
-F 0 "C116" H 4775 5875 50  0000 L CNN
+F 0 "C106" H 4775 5875 50  0000 L CNN
 F 1 "100nF" H 4775 5675 50  0000 L CNN
 F 2 "SFUSat:C_0402" H 4788 5625 50  0001 C CNN
@@
 AR Path="/5AA44392/592A8C09" Ref="#PWR078"  Part="1"
 AR Path="/5AA72383/592A8C09" Ref="#PWR089"  Part="1"
-F 0 "#PWR089" H 4750 5800 50  0001 C CNN
+F 0 "#PWR078" H 4750 5800 50  0001 C CNN
 F 1 "GND" H 4750 5900 50  0000 C CNN
 F 2 "" H 4750 6050 50  0000 C CNN
@@
 AR Path="/5AA44392/592ACE93" Ref="R100"  Part="1"
 AR Path="/5AA72383/592ACE93" Ref="R110"  Part="1"
-F 0 "R110" H 6000 4900 50  0000 L CNN
+F 0 "R100" H 6000 4900 50  0000 L CNN
 F 1 "56k" V 5950 4900 50  0000 C CNN
 F 2 "SFUSat:R_0402" V 5880 4900 50  0001 C CNN
@@
 AR Path="/5AA44392/592ACEFE" Ref="#PWR079"  Part="1"
 AR Path="/5AA72383/592ACEFE" Ref="#PWR090"  Part="1"
-F 0 "#PWR090" H 5950 4925 50  0001 C CNN
+F 0 "#PWR079" H 5950 4925 50  0001 C CNN
 F 1 "GND" H 5950 5025 50  0000 C CNN
 F 2 "" H 5950 5175 50  0000 C CNN
@@
 AR Path="/5AA44392/592AE8E9" Ref="#PWR080"  Part="1"
 AR Path="/5AA72383/592AE8E9" Ref="#PWR091"  Part="1"
-F 0 "#PWR091" H 3525 2625 50  0001 C CNN
+F 0 "#PWR080" H 3525 2625 50  0001 C CNN
 F 1 "GND" H 3525 2725 50  0000 C CNN
 F 2 "" H 3525 2875 50  0000 C CNN
@@
 AR Path="/5AA44392/592A69DC" Ref="X100"  Part="1"
 AR Path="/5AA72383/592A69DC" Ref="X110"  Part="1"
-F 0 "X110" V 2000 4325 60  0000 L CNN
+F 0 "X100" V 2000 4325 60  0000 L CNN
 F 1 "NX3225GA" H 2000 3950 60  0000 C TNN
 F 2 "SFUSat:NX3225GA" H 2000 4150 60  0001 C CNN
@@
 AR Path="/5AA44392/592A70F9" Ref="C101"  Part="1"
 AR Path="/5AA72383/592A70F9" Ref="C111"  Part="1"
-F 0 "C111" V 1700 3850 50  0000 C CNN
+F 0 "C101" V 1700 3850 50  0000 C CNN
 F 1 "12pF" V 1400 3850 50  0000 C CNN
 F 2 "SFUSat:C_0402" H 1588 3700 50  0001 C CNN
@@
 AR Path="/5AA44392/592A730F" Ref="C102"  Part="1"
 AR Path="/5AA72383/592A730F" Ref="C112"  Part="1"
-F 0 "C112" V 1700 4450 50  0000 C CNN
+F 0 "C102" V 1700 4450 50  0000 C CNN
 F 1 "15pF" V 1400 4450 50  0000 C CNN
 F 2 "SFUSat:C_0402" H 1588 4300 50  0001 C CNN
@@
 AR Path="/5AA44392/592A789E" Ref="#PWR081"  Part="1"
 AR Path="/5AA72383/592A789E" Ref="#PWR092"  Part="1"
-F 0 "#PWR092" H 1400 3600 50  0001 C CNN
+F 0 "#PWR081" H 1400 3600 50  0001 C CNN
 F 1 "GND" H 1400 3700 50  0000 C CNN
 F 2 "" H 1400 3850 50  0000 C CNN
@@
 AR Path="/5AA44392/592A7939" Ref="#PWR082"  Part="1"
 AR Path="/5AA72383/592A7939" Ref="#PWR093"  Part="1"
-F 0 "#PWR093" H 1400 4200 50  0001 C CNN
+F 0 "#PWR082" H 1400 4200 50  0001 C CNN
 F 1 "GND" H 1400 4300 50  0000 C CNN
 F 2 "" H 1400 4450 50  0000 C CNN
@@
 AR Path="/5AA44392/592F0537" Ref="C105"  Part="1"
 AR Path="/5AA72383/592F0537" Ref="C115"  Part="1"
-F 0 "C115" V 3825 2875 50  0000 C CNN
+F 0 "C105" V 3825 2875 50  0000 C CNN
 F 1 "100nF" V 3525 2875 50  0000 C CNN
 F 2 "SFUSat:C_0402" H 3713 2725 50  0001 C CNN
@@
 AR Path="/5AA44392/592F1736" Ref="#PWR083"  Part="1"
 AR Path="/5AA72383/592F1736" Ref="#PWR094"  Part="1"
-F 0 "#PWR094" H 3525 1750 50  0001 C CNN
+F 0 "#PWR083" H 3525 1750 50  0001 C CNN
 F 1 "GND" H 3525 1850 50  0000 C CNN
 F 2 "" H 3525 2000 50  0000 C CNN
@@
 AR Path="/5AA44392/592F173C" Ref="#PWR084"  Part="1"
 AR Path="/5AA72383/592F173C" Ref="#PWR095"  Part="1"
-F 0 "#PWR095" H 3525 2175 50  0001 C CNN
+F 0 "#PWR084" H 3525 2175 50  0001 C CNN
 F 1 "GND" H 3525 2275 50  0000 C CNN
 F 2 "" H 3525 2425 50  0000 C CNN
@@
 AR Path="/5AA44392/592F1742" Ref="C104"  Part="1"
 AR Path="/5AA72383/592F1742" Ref="C114"  Part="1"
-F 0 "C114" V 3825 2425 50  0000 C CNN
+F 0 "C104" V 3825 2425 50  0000 C CNN
 F 1 "220pF" V 3525 2425 50  0000 C CNN
 F 2 "SFUSat:C_0402" H 3713 2275 50  0001 C CNN
@@
 AR Path="/5AA44392/592F1748" Ref="C103"  Part="1"
 AR Path="/5AA72383/592F1748" Ref="C113"  Part="1"
-F 0 "C113" V 3825 2000 50  0000 C CNN
+F 0 "C103" V 3825 2000 50  0000 C CNN
 F 1 "100nF" V 3525 2000 50  0000 C CNN
 F 2 "SFUSat:C_0402" H 3713 1850 50  0001 C CNN
@@
 AR Path="/5AA44392/592F1E87" Ref="#PWR085"  Part="1"
 AR Path="/5AA72383/592F1E87" Ref="#PWR096"  Part="1"
-F 0 "#PWR096" H 5475 3050 50  0001 C CNN
+F 0 "#PWR085" H 5475 3050 50  0001 C CNN
 F 1 "GND" H 5475 3150 50  0000 C CNN
 F 2 "" H 5475 3300 50  0000 C CNN
@@
 AR Path="/5AA44392/592F1E8D" Ref="#PWR086"  Part="1"
 AR Path="/5AA72383/592F1E8D" Ref="#PWR097"  Part="1"
-F 0 "#PWR097" H 5475 2625 50  0001 C CNN
+F 0 "#PWR086" H 5475 2625 50  0001 C CNN
 F 1 "GND" H 5475 2725 50  0000 C CNN
 F 2 "" H 5475 2875 50  0000 C CNN
@@
 AR Path="/5AA44392/592F1E93" Ref="C107"  Part="1"
 AR Path="/5AA72383/592F1E93" Ref="C117"  Part="1"
-F 0 "C117" V 5175 2875 50  0000 C CNN
+F 0 "C107" V 5175 2875 50  0000 C CNN
 F 1 "100nF" V 5475 2875 50  0000 C CNN
 F 2 "SFUSat:C_0402" H 5363 2725 50  0001 C CNN
@@
 AR Path="/5AA44392/592F1E99" Ref="C100"  Part="1"
 AR Path="/5AA72383/592F1E99" Ref="C110"  Part="1"
-F 0 "C110" V 5175 3300 50  0000 C CNN
+F 0 "C100" V 5175 3300 50  0000 C CNN
 F 1 "100nF" V 5475 3300 50  0000 C CNN
 F 2 "SFUSat:C_0402" H 5363 3150 50  0001 C CNN
@@
 AR Path="/5AA44392/5AAD2BB4" Ref="#PWR087"  Part="1"
 AR Path="/5AA72383/5AAD2BB4" Ref="#PWR098"  Part="1"
-F 0 "#PWR098" H 7650 1700 50  0001 C CNN
+F 0 "#PWR087" H 7650 1700 50  0001 C CNN
 F 1 "GND" H 7650 1800 50  0000 C CNN
 F 2 "" H 7650 1950 50  0000 C CNN
@@
 AR Path="/5AA72383/5ABB51CC" Ref="J20"  Part="1"
 AR Path="/5ABB51CC" Ref="J?"  Part="1"
-F 0 "J20" H 8300 3400 50  0000 C CNN
+F 0 "J19" H 8300 3400 50  0000 C CNN
 F 1 "Conn_01x03" H 8300 3000 50  0000 C CNN
 F 2 "Socket_Strips:Socket_Strip_Straight_1x03_Pitch2.54mm" H 8300 3200 50  0001 C CNN
@@
 AR Path="/5AA72383/5AB496AE" Ref="U13"  Part="1"
 AR Path="/5AA44392/5AB496AE" Ref="U12"  Part="1"
-F 0 "U13" H 8250 2450 50  0000 C BNN
+F 0 "U12" H 8250 2450 50  0000 C BNN
 F 1 "CONN_02X05_SHRD" H 8300 1850 50  0000 C TNN
 F 2 "SFUSat:Socket_Strip_Straight_2x05" H 8150 2350 50  0001 C CNN

Commit message: removed op_3v3, routed SPI
Parts:
- removed J19: Conn_01x03, Socket_Strips:Socket_Strip_Straight_1x03_Pitch2.54mm, symbol CONN_01X03
Connections:
- net labels removed: VDD_3.3
- wire segments 46 -> 43
Other:
- note removed: "If the debugger power supply is used,\n the radio must only be operated through \nthe u.fl debug ports adjasent to the balun."
- note removed: "This sub-circuit can use either power \nprovided by the Debugger or from \nthe onboard regulator. VDD_3.3 is \nthe power rail for this circuit."
Changed lines of the file:
@@
 AR Path="/5AA44392/592A0E9A" Ref="U100"  Part="1"
 AR Path="/5AA72383/592A0E9A" Ref="U110"  Part="1"
-F 0 "U100" H 4500 4550 60  0000 C BNN
+F 0 "U110" H 4500 4550 60  0000 C BNN
 F 1 "CC1101-Q1" H 4500 4450 60  0000 C TNN
 F 2 "SFUSat:CC1101-Q1" H 4350 4500 60  0001 C CNN
@@
 AR Path="/5AA44392/592A76F5" Ref="#PWR077"  Part="1"
 AR Path="/5AA72383/592A76F5" Ref="#PWR088"  Part="1"
-F 0 "#PWR077" H 4150 5375 50  0001 C CNN
+F 0 "#PWR088" H 4150 5375 50  0001 C CNN
 F 1 "GND" H 4150 5475 50  0000 C CNN
 F 2 "" H 4150 5625 50  0000 C CNN
@@
 AR Path="/5AA44392/592A885A" Ref="C106"  Part="1"
 AR Path="/5AA72383/592A885A" Ref="C116"  Part="1"
-F 0 "C106" H 4775 5875 50  0000 L CNN
+F 0 "C116" H 4775 5875 50  0000 L CNN
 F 1 "100nF" H 4775 5675 50  0000 L CNN
 F 2 "SFUSat:C_0402" H 4788 5625 50  0001 C CNN
@@
 AR Path="/5AA44392/592A8C09" Ref="#PWR078"  Part="1"
 AR Path="/5AA72383/592A8C09" Ref="#PWR089"  Part="1"
-F 0 "#PWR078" H 4750 5800 50  0001 C CNN
+F 0 "#PWR089" H 4750 5800 50  0001 C CNN
 F 1 "GND" H 4750 5900 50  0000 C CNN
 F 2 "" H 4750 6050 50  0000 C CNN
@@
 AR Path="/5AA44392/592ACE93" Ref="R100"  Part="1"
 AR Path="/5AA72383/592ACE93" Ref="R110"  Part="1"
-F 0 "R100" H 6000 4900 50  0000 L CNN
+F 0 "R110" H 6000 4900 50  0000 L CNN
 F 1 "56k" V 5950 4900 50  0000 C CNN
 F 2 "SFUSat:R_0402" V 5880 4900 50  0001 C CNN
@@
 AR Path="/5AA44392/592ACEFE" Ref="#PWR079"  Part="1"
 AR Path="/5AA72383/592ACEFE" Ref="#PWR090"  Part="1"
-F 0 "#PWR079" H 5950 4925 50  0001 C CNN
+F 0 "#PWR090" H 5950 4925 50  0001 C CNN
 F 1 "GND" H 5950 5025 50  0000 C CNN
 F 2 "" H 5950 5175 50  0000 C CNN
@@
 AR Path="/5AA44392/592AE8E9" Ref="#PWR080"  Part="1"
 AR Path="/5AA72383/592AE8E9" Ref="#PWR091"  Part="1"
-F 0 "#PWR080" H 3525 2625 50  0001 C CNN
+F 0 "#PWR091" H 3525 2625 50  0001 C CNN
 F 1 "GND" H 3525 2725 50  0000 C CNN
 F 2 "" H 3525 2875 50  0000 C CNN
@@
 AR Path="/5AA44392/592A69DC" Ref="X100"  Part="1"
 AR Path="/5AA72383/592A69DC" Ref="X110"  Part="1"
-F 0 "X100" V 2000 4325 60  0000 L CNN
+F 0 "X110" V 2000 4325 60  0000 L CNN
 F 1 "NX3225GA" H 2000 3950 60  0000 C TNN
 F 2 "SFUSat:NX3225GA" H 2000 4150 60  0001 C CNN
@@
 AR Path="/5AA44392/592A70F9" Ref="C101"  Part="1"
 AR Path="/5AA72383/592A70F9" Ref="C111"  Part="1"
-F 0 "C101" V 1700 3850 50  0000 C CNN
+F 0 "C111" V 1700 3850 50  0000 C CNN
 F 1 "12pF" V 1400 3850 50  0000 C CNN
 F 2 "SFUSat:C_0402" H 1588 3700 50  0001 C CNN
@@
 AR Path="/5AA44392/592A730F" Ref="C102"  Part="1"
 AR Path="/5AA72383/592A730F" Ref="C112"  Part="1"
-F 0 "C102" V 1700 4450 50  0000 C CNN
+F 0 "C112" V 1700 4450 50  0000 C CNN
 F 1 "15pF" V 1400 4450 50  0000 C CNN
 F 2 "SFUSat:C_0402" H 1588 4300 50  0001 C CNN
@@
 AR Path="/5AA44392/592A789E" Ref="#PWR081"  Part="1"
 AR Path="/5AA72383/592A789E" Ref="#PWR092"  Part="1"
-F 0 "#PWR081" H 1400 3600 50  0001 C CNN
+F 0 "#PWR092" H 1400 3600 50  0001 C CNN
 F 1 "GND" H 1400 3700 50  0000 C CNN
 F 2 "" H 1400 3850 50  0000 C CNN
@@
 AR Path="/5AA44392/592A7939" Ref="#PWR082"  Part="1"
 AR Path="/5AA72383/592A7939" Ref="#PWR093"  Part="1"
-F 0 "#PWR082" H 1400 4200 50  0001 C CNN
+F 0 "#PWR093" H 1400 4200 50  0001 C CNN
 F 1 "GND" H 1400 4300 50  0000 C CNN
 F 2 "" H 1400 4450 50  0000 C CNN
@@
 AR Path="/5AA44392/592F0537" Ref="C105"  Part="1"
 AR Path="/5AA72383/592F0537" Ref="C115"  Part="1"
-F 0 "C105" V 3825 2875 50  0000 C CNN
+F 0 "C115" V 3825 2875 50  0000 C CNN
 F 1 "100nF" V 3525 2875 50  0000 C CNN
 F 2 "SFUSat:C_0402" H 3713 2725 50  0001 C CNN
@@
 AR Path="/5AA44392/592F1736" Ref="#PWR083"  Part="1"
 AR Path="/5AA72383/592F1736" Ref="#PWR094"  Part="1"
-F 0 "#PWR083" H 3525 1750 50  0001 C CNN
+F 0 "#PWR094" H 3525 1750 50  0001 C CNN
 F 1 "GND" H 3525 1850 50  0000 C CNN
 F 2 "" H 3525 2000 50  0000 C CNN
@@
 AR Path="/5AA44392/592F173C" Ref="#PWR084"  Part="1"
 AR Path="/5AA72383/592F173C" Ref="#PWR095"  Part="1"
-F 0 "#PWR084" H 3525 2175 50  0001 C CNN
+F 0 "#PWR095" H 3525 2175 50  0001 C CNN
 F 1 "GND" H 3525 2275 50  0000 C CNN
 F 2 "" H 3525 2425 50  0000 C CNN
@@
 AR Path="/5AA44392/592F1742" Ref="C104"  Part="1"
 AR Path="/5AA72383/592F1742" Ref="C114"  Part="1"
-F 0 "C104" V 3825 2425 50  0000 C CNN
+F 0 "C114" V 3825 2425 50  0000 C CNN
 F 1 "220pF" V 3525 2425 50  0000 C CNN
 F 2 "SFUSat:C_0402" H 3713 2275 50  0001 C CNN
@@
 AR Path="/5AA44392/592F1748" Ref="C103"  Part="1"
 AR Path="/5AA72383/592F1748" Ref="C113"  Part="1"
-F 0 "C103" V 3825 2000 50  0000 C CNN
+F 0 "C113" V 3825 2000 50  0000 C CNN
 F 1 "100nF" V 3525 2000 50  0000 C CNN
 F 2 "SFUSat:C_0402" H 3713 1850 50  0001 C CNN
@@
 AR Path="/5AA44392/592F1E87" Ref="#PWR085"  Part="1"
 AR Path="/5AA72383/592F1E87" Ref="#PWR096"  Part="1"
-F 0 "#PWR085" H 5475 3050 50  0001 C CNN
+F 0 "#PWR096" H 5475 3050 50  0001 C CNN
 F 1 "GND" H 5475 3150 50  0000 C CNN
 F 2 "" H 5475 3300 50  0000 C CNN
@@
 AR Path="/5AA44392/592F1E8D" Ref="#PWR086"  Part="1"
 AR Path="/5AA72383/592F1E8D" Ref="#PWR097"  Part="1"
-F 0 "#PWR086" H 5475 2625 50  0001 C CNN
+F 0 "#PWR097" H 5475 2625 50  0001 C CNN
 F 1 "GND" H 5475 2725 50  0000 C CNN
 F 2 "" H 5475 2875 50  0000 C CNN
@@
 AR Path="/5AA44392/592F1E93" Ref="C107"  Part="1"
 AR Path="/5AA72383/592F1E93" Ref="C117"  Part="1"
-F 0 "C107" V 5175 2875 50  0000 C CNN
+F 0 "C117" V 5175 2875 50  0000 C CNN
 F 1 "100nF" V 5475 2875 50  0000 C CNN
 F 2 "SFUSat:C_0402" H 5363 2725 50  0001 C CNN
@@
 AR Path="/5AA44392/592F1E99" Ref="C100"  Part="1"
 AR Path="/5AA72383/592F1E99" Ref="C110"  Part="1"
-F 0 "C100" V 5175 3300 50  0000 C CNN
+F 0 "C110" V 5175 3300 50  0000 C CNN
 F 1 "100nF" V 5475 3300 50  0000 C CNN
 F 2 "SFUSat:C_0402" H 5363 3150 50  0001 C CNN
@@
 Wire Wire Line
 	5850 4350 6000 4350
-Text Label 8850 1950 2    60   ~ 0
-VDD_3.3
 Text Label 8850 2350 2    60   ~ 0
 MISO
@@
 AR Path="/5AA44392/5AAD2BB4" Ref="#PWR087"  Part="1"
 AR Path="/5AA72383/5AAD2BB4" Ref="#PWR098"  Part="1"
-F 0 "#PWR087" H 7650 1700 50  0001 C CNN
+F 0 "#PWR098" H 7650 1700 50  0001 C CNN
 F 1 "GND" H 7650 1800 50  0000 C CNN
 F 2 "" H 7650 1950 50  0000 C CNN
@@
 Wire Wire Line
 	8050 2350 7650 2350
-Text Label 8600 3100 0    60   ~ 0
-OP_3.3
-Text Label 8600 3200 0    60   ~ 0
-VDD_3.3
-$Comp
-L CONN_01X03 J19
-U 1 1 5ABB51CC
-P 8300 3200
-AR Path="/5AA44392/5ABB51CC" Ref="J19"  Part="1"
-AR Path="/5AA72383/5ABB51CC" Ref="J20"  Part="1"
-AR Path="/5ABB51CC" Ref="J?"  Part="1"
-F 0 "J19" H 8300 3400 50  0000 C CNN
-F 1 "Conn_01x03" H 8300 3000 50  0000 C CNN
-F 2 "Socket_Strips:Socket_Strip_Straight_1x03_Pitch2.54mm" H 8300 3200 50  0001 C CNN
-F 3 "" H 8300 3200 50  0001 C CNN
-	1    8300 3200
-	-1   0    0    1
-$EndComp
-Text HLabel 8600 3300 2    60   Input ~ 0
-3V3
-Wire Wire Line
-	8500 3100 8600 3100
-Wire Wire Line
-	8500 3200 8600 3200
-Wire Wire Line
-	8500 3300 8600 3300
 Text Notes 8925 1925 0    60   ~ 0
 Required Power for Debugger operation
@@
 Text Label 3100 5000 2    60   ~ 0
 GPIO0
-Text Label 4450 1650 0    60   ~ 0
-VDD_3.3
-Text Notes 9075 3325 0    60   ~ 0
-This sub-circuit can use either power \nprovided by the Debugger or from \nthe onboard regulator. VDD_3.3 is \nthe power rail for this circuit.
-Text Notes 8025 3750 0    60   ~ 0
-If the debugger power supply is used,\n the radio must only be operated through \nthe u.fl debug ports adjasent to the balun.
 $Comp
 L CONN_02X05_SHRD U13
@@
 AR Path="/5AA72383/5AB496AE" Ref="U13"  Part="1"
 AR Path="/5AA44392/5AB496AE" Ref="U12"  Part="1"
-F 0 "U12" H 8250 2450 50  0000 C BNN
+F 0 "U13" H 8250 2450 50  0000 C BNN
 F 1 "CONN_02X05_SHRD" H 8300 1850 50  0000 C TNN
 F 2 "SFUSat:Socket_Strip_Straight_2x05" H 8150 2350 50  0001 C CNN
@@
 	1    0    0    -1
 $EndComp
+Text HLabel 4450 1650 2    60   Input ~ 0
+3V3
+Text HLabel 8850 1950 2    60   Input ~ 0
+3V3
 $EndSCHEMATC

Commit message: modified proposed pot schematic
Changed lines of the file:
@@
 AR Path="/5AA44392/592A0E9A" Ref="U100"  Part="1"
 AR Path="/5AA72383/592A0E9A" Ref="U110"  Part="1"
-F 0 "U110" H 4500 4550 60  0000 C BNN
+F 0 "U100" H 4500 4550 60  0000 C BNN
 F 1 "CC1101-Q1" H 4500 4450 60  0000 C TNN
 F 2 "SFUSat:CC1101-Q1" H 4350 4500 60  0001 C CNN
@@
 AR Path="/5AA44392/592A76F5" Ref="#PWR077"  Part="1"
 AR Path="/5AA72383/592A76F5" Ref="#PWR088"  Part="1"
-F 0 "#PWR088" H 4150 5375 50  0001 C CNN
+F 0 "#PWR077" H 4150 5375 50  0001 C CNN
 F 1 "GND" H 4150 5475 50  0000 C CNN
 F 2 "" H 4150 5625 50  0000 C CNN
@@
 AR Path="/5AA44392/592A885A" Ref="C106"  Part="1"
 AR Path="/5AA72383/592A885A" Ref="C116"  Part="1"
-F 0 "C116" H 4775 5875 50  0000 L CNN
+F 0 "C106" H 4775 5875 50  0000 L CNN
 F 1 "100nF" H 4775 5675 50  0000 L CNN
 F 2 "SFUSat:C_0402" H 4788 5625 50  0001 C CNN
@@
 AR Path="/5AA44392/592A8C09" Ref="#PWR078"  Part="1"
 AR Path="/5AA72383/592A8C09" Ref="#PWR089"  Part="1"
-F 0 "#PWR089" H 4750 5800 50  0001 C CNN
+F 0 "#PWR078" H 4750 5800 50  0001 C CNN
 F 1 "GND" H 4750 5900 50  0000 C CNN
 F 2 "" H 4750 6050 50  0000 C CNN
@@
 AR Path="/5AA44392/592ACE93" Ref="R100"  Part="1"
 AR Path="/5AA72383/592ACE93" Ref="R110"  Part="1"
-F 0 "R110" H 6000 4900 50  0000 L CNN
+F 0 "R100" H 6000 4900 50  0000 L CNN
 F 1 "56k" V 5950 4900 50  0000 C CNN
 F 2 "SFUSat:R_0402" V 5880 4900 50  0001 C CNN
@@
 AR Path="/5AA44392/592ACEFE" Ref="#PWR079"  Part="1"
 AR Path="/5AA72383/592ACEFE" Ref="#PWR090"  Part="1"
-F 0 "#PWR090" H 5950 4925 50  0001 C CNN
+F 0 "#PWR079" H 5950 4925 50  0001 C CNN
 F 1 "GND" H 5950 5025 50  0000 C CNN
 F 2 "" H 5950 5175 50  0000 C CNN
@@
 AR Path="/5AA44392/592AE8E9" Ref="#PWR080"  Part="1"
 AR Path="/5AA72383/592AE8E9" Ref="#PWR091"  Part="1"
-F 0 "#PWR091" H 3525 2625 50  0001 C CNN
+F 0 "#PWR080" H 3525 2625 50  0001 C CNN
 F 1 "GND" H 3525 2725 50  0000 C CNN
 F 2 "" H 3525 2875 50  0000 C CNN
@@
 AR Path="/5AA44392/592A69DC" Ref="X100"  Part="1"
 AR Path="/5AA72383/592A69DC" Ref="X110"  Part="1"
-F 0 "X110" V 2000 4325 60  0000 L CNN
+F 0 "X100" V 2000 4325 60  0000 L CNN
 F 1 "NX3225GA" H 2000 3950 60  0000 C TNN
 F 2 "SFUSat:NX3225GA" H 2000 4150 60  0001 C CNN
@@
 AR Path="/5AA44392/592A70F9" Ref="C101"  Part="1"
 AR Path="/5AA72383/592A70F9" Ref="C111"  Part="1"
-F 0 "C111" V 1700 3850 50  0000 C CNN
+F 0 "C101" V 1700 3850 50  0000 C CNN
 F 1 "12pF" V 1400 3850 50  0000 C CNN
 F 2 "SFUSat:C_0402" H 1588 3700 50  0001 C CNN
@@
 AR Path="/5AA44392/592A730F" Ref="C102"  Part="1"
 AR Path="/5AA72383/592A730F" Ref="C112"  Part="1"
-F 0 "C112" V 1700 4450 50  0000 C CNN
+F 0 "C102" V 1700 4450 50  0000 C CNN
 F 1 "15pF" V 1400 4450 50  0000 C CNN
 F 2 "SFUSat:C_0402" H 1588 4300 50  0001 C CNN
@@
 AR Path="/5AA44392/592A789E" Ref="#PWR081"  Part="1"
 AR Path="/5AA72383/592A789E" Ref="#PWR092"  Part="1"
-F 0 "#PWR092" H 1400 3600 50  0001 C CNN
+F 0 "#PWR081" H 1400 3600 50  0001 C CNN
 F 1 "GND" H 1400 3700 50  0000 C CNN
 F 2 "" H 1400 3850 50  0000 C CNN
@@
 AR Path="/5AA44392/592A7939" Ref="#PWR082"  Part="1"
 AR Path="/5AA72383/592A7939" Ref="#PWR093"  Part="1"
-F 0 "#PWR093" H 1400 4200 50  0001 C CNN
+F 0 "#PWR082" H 1400 4200 50  0001 C CNN
 F 1 "GND" H 1400 4300 50  0000 C CNN
 F 2 "" H 1400 4450 50  0000 C CNN
@@
 AR Path="/5AA44392/592F0537" Ref="C105"  Part="1"
 AR Path="/5AA72383/592F0537" Ref="C115"  Part="1"
-F 0 "C115" V 3825 2875 50  0000 C CNN
+F 0 "C105" V 3825 2875 50  0000 C CNN
 F 1 "100nF" V 3525 2875 50  0000 C CNN
 F 2 "SFUSat:C_0402" H 3713 2725 50  0001 C CNN
@@
 AR Path="/5AA44392/592F1736" Ref="#PWR083"  Part="1"
 AR Path="/5AA72383/592F1736" Ref="#PWR094"  Part="1"
-F 0 "#PWR094" H 3525 1750 50  0001 C CNN
+F 0 "#PWR083" H 3525 1750 50  0001 C CNN
 F 1 "GND" H 3525 1850 50  0000 C CNN
 F 2 "" H 3525 2000 50  0000 C CNN
@@
 AR Path="/5AA44392/592F173C" Ref="#PWR084"  Part="1"
 AR Path="/5AA72383/592F173C" Ref="#PWR095"  Part="1"
-F 0 "#PWR095" H 3525 2175 50  0001 C CNN
+F 0 "#PWR084" H 3525 2175 50  0001 C CNN
 F 1 "GND" H 3525 2275 50  0000 C CNN
 F 2 "" H 3525 2425 50  0000 C CNN
@@
 AR Path="/5AA44392/592F1742" Ref="C104"  Part="1"
 AR Path="/5AA72383/592F1742" Ref="C114"  Part="1"
-F 0 "C114" V 3825 2425 50  0000 C CNN
+F 0 "C104" V 3825 2425 50  0000 C CNN
 F 1 "220pF" V 3525 2425 50  0000 C CNN
 F 2 "SFUSat:C_0402" H 3713 2275 50  0001 C CNN
@@
 AR Path="/5AA44392/592F1748" Ref="C103"  Part="1"
 AR Path="/5AA72383/592F1748" Ref="C113"  Part="1"
-F 0 "C113" V 3825 2000 50  0000 C CNN
+F 0 "C103" V 3825 2000 50  0000 C CNN
 F 1 "100nF" V 3525 2000 50  0000 C CNN
 F 2 "SFUSat:C_0402" H 3713 1850 50  0001 C CNN
@@
 AR Path="/5AA44392/592F1E87" Ref="#PWR085"  Part="1"
 AR Path="/5AA72383/592F1E87" Ref="#PWR096"  Part="1"
-F 0 "#PWR096" H 5475 3050 50  0001 C CNN
+F 0 "#PWR085" H 5475 3050 50  0001 C CNN
 F 1 "GND" H 5475 3150 50  0000 C CNN
 F 2 "" H 5475 3300 50  0000 C CNN
@@
 AR Path="/5AA44392/592F1E8D" Ref="#PWR086"  Part="1"
 AR Path="/5AA72383/592F1E8D" Ref="#PWR097"  Part="1"
-F 0 "#PWR097" H 5475 2625 50  0001 C CNN
+F 0 "#PWR086" H 5475 2625 50  0001 C CNN
 F 1 "GND" H 5475 2725 50  0000 C CNN
 F 2 "" H 5475 2875 50  0000 C CNN
@@
 AR Path="/5AA44392/592F1E93" Ref="C107"  Part="1"
 AR Path="/5AA72383/592F1E93" Ref="C117"  Part="1"
-F 0 "C117" V 5175 2875 50  0000 C CNN
+F 0 "C107" V 5175 2875 50  0000 C CNN
 F 1 "100nF" V 5475 2875 50  0000 C CNN
 F 2 "SFUSat:C_0402" H 5363 2725 50  0001 C CNN
@@
 AR Path="/5AA44392/592F1E99" Ref="C100"  Part="1"
 AR Path="/5AA72383/592F1E99" Ref="C110"  Part="1"
-F 0 "C110" V 5175 3300 50  0000 C CNN
+F 0 "C100" V 5175 3300 50  0000 C CNN
 F 1 "100nF" V 5475 3300 50  0000 C CNN
 F 2 "SFUSat:C_0402" H 5363 3150 50  0001 C CNN
@@
 AR Path="/5AA44392/5AAD2BB4" Ref="#PWR087"  Part="1"
 AR Path="/5AA72383/5AAD2BB4" Ref="#PWR098"  Part="1"
-F 0 "#PWR098" H 7650 1700 50  0001 C CNN
+F 0 "#PWR087" H 7650 1700 50  0001 C CNN
 F 1 "GND" H 7650 1800 50  0000 C CNN
 F 2 "" H 7650 1950 50  0000 C CNN
@@
 AR Path="/5AA72383/5AB496AE" Ref="U13"  Part="1"
 AR Path="/5AA44392/5AB496AE" Ref="U12"  Part="1"
-F 0 "U13" H 8250 2450 50  0000 C BNN
+F 0 "U12" H 8250 2450 50  0000 C BNN
 F 1 "CONN_02X05_SHRD" H 8300 1850 50  0000 C TNN
 F 2 "SFUSat:Socket_Strip_Straight_2x05" H 8150 2350 50  0001 C CNN
