File: RF_SPDT.sch (KiCad schematic (older format))
At the start: 11 parts

Commit message: layed out upper band and lower band schematic. Need to add a 2W rated SPDT switch to connect the RX and TX stages together before the diplexer
Parts:
- removed J?: SMA, SFUSat:UFL-R-SMT-1-Coaxial-Connector, symbol SMA
- removed U?: SINGLE_0402, SFUSat:SINGLE_0402, symbol SINGLE_0402
Changed lines of the file:
@@
 $Descr A4 11693 8268
 encoding utf-8
-Sheet 8 9
+Sheet 7 9
 Title ""
 Date ""
@@
 $Comp
 L SMA J?
-U 1 1 5AA2DAC6
-P 4625 3150
-F 0 "J?" H 4575 2950 60  0000 C CNN
-F 1 "SMA" H 4625 3300 60  0000 C CNN
-F 2 "SFUSat:UFL-R-SMT-1-Coaxial-Connector" H 4825 3200 60  0001 C CNN
-F 3 "" H 4825 3200 60  0000 C CNN
-F 4 "H9161-ND" H 4625 3150 60  0001 C CNN "Digikey"
-	1    4625 3150
-	0    -1   -1   0
-$EndComp
-$Comp
-L SMA J?
 U 1 1 5AA2DACE
 P 7200 2900
@@
 $EndComp
 $Comp
-L SINGLE_0402 U?
-U 1 1 5AA2DADD
-P 4575 3700
-F 0 "U?" V 4575 3625 60  0000 R CNN
-F 1 "SINGLE_0402" H 4575 3600 60  0001 C TNN
-F 2 "SFUSat:SINGLE_0402" H 4575 3700 60  0001 C CNN
-F 3 "" H 4575 3700 60  0001 C CNN
-	1    4575 3700
-	0    1    1    0
-$EndComp
-$Comp
-L GND #PWR?
-U 1 1 5AA2DAE4
-P 4725 3450
-F 0 "#PWR?" H 4725 3200 50  0001 C CNN
-F 1 "GND" H 4725 3300 50  0000 C CNN
-F 2 "" H 4725 3450 50  0000 C CNN
-F 3 "" H 4725 3450 50  0000 C CNN
-	1    4725 3450
-	1    0    0    -1
-$EndComp
-$Comp

Commit message: Annotated the schematics
Parts:
- gave numbers to parts that had none: 9
Changed lines of the file:
@@
 3V3
 $Comp
-L C C?
+L C C12
 U 1 1 5AA2DA8E
 P 4575 4000
-F 0 "C?" V 4725 4000 50  0000 C CNN
+F 0 "C12" V 4725 4000 50  0000 C CNN
 F 1 "47pF" V 4425 4000 50  0000 C CNN
 F 2 "SFUSat:C_0402" H 4613 3850 50  0001 C CNN
@@
 $EndComp
 $Comp
-L C C?
+L C C14
 U 1 1 5AA2DA95
 P 7150 3750
-F 0 "C?" V 7000 3750 50  0000 C CNN
+F 0 "C14" V 7000 3750 50  0000 C CNN
 F 1 "47pF" V 7300 3750 50  0000 C CNN
 F 2 "SFUSat:C_0402" H 7188 3600 50  0001 C CNN
@@
 $EndComp
 $Comp
-L C C?
+L C C15
 U 1 1 5AA2DA9C
 P 7150 4250
-F 0 "C?" V 7000 4250 50  0000 C CNN
+F 0 "C15" V 7000 4250 50  0000 C CNN
 F 1 "47pF" V 7300 4250 50  0000 C CNN
 F 2 "SFUSat:C_0402" H 7188 4100 50  0001 C CNN
@@
 B2
 $Comp
-L GND #PWR?
+L GND #PWR77
 U 1 1 5AA2DAAA
 P 5900 4725
-F 0 "#PWR?" H 5900 4475 50  0001 C CNN
+F 0 "#PWR77" H 5900 4475 50  0001 C CNN
 F 1 "GND" H 5900 4575 50  0000 C CNN
 F 2 "" H 5900 4725 50  0000 C CNN
@@
 $EndComp
 $Comp
-L SKY13372-467LF U?
+L SKY13372-467LF U7
 U 1 1 5AA2DAB0
 P 5850 4000
-F 0 "U?" H 5850 3975 60  0000 C TNN
+F 0 "U7" H 5850 3975 60  0000 C TNN
 F 1 "SKY13372-467LF" H 5850 4025 60  0000 C BNN
 F 2 "SFUSat:QFN-16_650P" H 5650 4200 60  0001 C CNN
@@
 $EndComp
 $Comp
-L C C?
+L C C13
 U 1 1 5AA2DAB8
 P 6175 3225
-F 0 "C?" H 6200 3325 50  0000 L CNN
+F 0 "C13" H 6200 3325 50  0000 L CNN
 F 1 "47nF" H 6200 3125 50  0000 L CNN
 F 2 "SFUSat:C_0402" H 6213 3075 50  0001 C CNN
@@
 $EndComp
 $Comp
-L GND #PWR?
+L GND #PWR78
 U 1 1 5AA2DABF
 P 6175 3425
-F 0 "#PWR?" H 6175 3175 50  0001 C CNN
+F 0 "#PWR78" H 6175 3175 50  0001 C CNN
 F 1 "GND" H 6175 3275 50  0000 C CNN
 F 2 "" H 6175 3425 50  0000 C CNN
@@
 $EndComp
 $Comp
-L SMA J?
+L SMA J18
 U 1 1 5AA2DACE
 P 7200 2900
-F 0 "J?" H 7150 2700 60  0000 C CNN
+F 0 "J18" H 7150 2700 60  0000 C CNN
 F 1 "SMA" H 7200 3050 60  0000 C CNN
 F 2 "SFUSat:UFL-R-SMT-1-Coaxial-Connector" H 7400 2950 60  0001 C CNN
@@
 $EndComp
 $Comp
-L SMA J?
+L SMA J17
 U 1 1 5AA2DAD6
 P 7100 5100
-F 0 "J?" H 7050 4900 60  0000 C CNN
+F 0 "J17" H 7050 4900 60  0000 C CNN
 F 1 "SMA" H 7100 5250 60  0000 C CNN
 F 2 "SFUSat:UFL-R-SMT-1-Coaxial-Connector" H 7300 5150 60  0001 C CNN
@@
 $EndComp
 $Comp
-L SINGLE_0402 U?
+L SINGLE_0402 U8
 U 1 1 5AA2DAEA
 P 7150 3450
-F 0 "U?" V 7150 3375 60  0000 R CNN
+F 0 "U8" V 7150 3375 60  0000 R CNN
 F 1 "SINGLE_0402" H 7150 3350 60  0001 C TNN
 F 2 "SFUSat:SINGLE_0402" H 7150 3450 60  0001 C CNN
@@
 $EndComp
 $Comp
-L GND #PWR?
+L GND #PWR80
 U 1 1 5AA2DAF1
 P 7300 3200
-F 0 "#PWR?" H 7300 2950 50  0001 C CNN
+F 0 "#PWR80" H 7300 2950 50  0001 C CNN
 F 1 "GND" H 7300 3050 50  0000 C CNN
 F 2 "" H 7300 3200 50  0000 C CNN
@@
 $EndComp
 $Comp
-L GND #PWR?
+L GND #PWR79
 U 1 1 5AA2DAF7
 P 7000 4800
-F 0 "#PWR?" H 7000 4550 50  0001 C CNN
+F 0 "#PWR79" H 7000 4550 50  0001 C CNN
 F 1 "GND" H 7000 4650 50  0000 C CNN
 F 2 "" H 7000 4800 50  0000 C CNN
@@
 $EndComp
 $Comp
-L SINGLE_0402 U?
+L SINGLE_0402 U11
 U 1 1 5AA2DAFD
 P 7150 4550
-F 0 "U?" V 7150 4475 60  0000 R CNN
+F 0 "U11" V 7150 4475 60  0000 R CNN
 F 1 "SINGLE_0402" H 7150 4450 60  0001 C TNN
 F 2 "SFUSat:SINGLE_0402" H 7150 4550 60  0001 C CNN
