File: TEMP_SENSE.sch (KiCad schematic (older format))
At the start: 2 parts, among them U400 STLM75

Commit message: Changed temp sense reference designator prefix
Initally overlapped with PA LB reference designator prefix
Parts:
- renumbered C400 to C600, U400 to U600
Changed lines of the file:
@@
 $Descr A4 11693 8268
 encoding utf-8
-Sheet 15 12
+Sheet 12 12
 Title "Board Surface Temperature Sensor"
 Date ""
@@
 $EndDescr
 $Comp
-L STLM75 U400
+L STLM75 U600
 U 1 1 5AC2622D
 P 5950 3825
-AR Path="/5AC235B1/5AC2622D" Ref="U400"  Part="1"
-AR Path="/5AD08722/5AC2622D" Ref="U410"  Part="1"
-F 0 "U410" H 5950 3975 60  0000 C CNN
+AR Path="/5AC235B1/5AC2622D" Ref="U600"  Part="1"
+AR Path="/5AD08722/5AC2622D" Ref="U610"  Part="1"
+F 0 "U610" H 5950 3975 60  0000 C CNN
 F 1 "STLM75" H 5950 3525 60  0000 C CNN
 F 2 "" H 5900 3825 60  0001 C CNN
@@
 	6500 4025 6450 4025
 $Comp
-L C C400
+L C C600
 U 1 1 5AD2851F
 P 6975 3800
-AR Path="/5AC235B1/5AD2851F" Ref="C400"  Part="1"
-AR Path="/5AD08722/5AD2851F" Ref="C410"  Part="1"
-F 0 "C410" H 7000 3900 50  0000 L CNN
+AR Path="/5AC235B1/5AD2851F" Ref="C600"  Part="1"
+AR Path="/5AD08722/5AD2851F" Ref="C610"  Part="1"
+F 0 "C610" H 7000 3900 50  0000 L CNN
 F 1 "DNP" H 7000 3700 50  0000 L CNN
 F 2 "SFUSat-cap:C_0402" H 7013 3650 50  0001 C CNN
