File: TEMP_SENSE.sch (KiCad schematic (older format))
At the start: 2 parts, among them U600 STLM75

Commit message: power schematic complete
Parts:
- U600: footprint (none) -> SFUSat:TSSOP-8-3x3mm-SOT505-1
Changed lines of the file:
@@
 LIBS:SFUSat-ind
 LIBS:SFUSat-res
+LIBS:SFUSat-power
 LIBS:SFUSat-Radio-cache
 EELAYER 25 0
@@
 $Descr A4 11693 8268
 encoding utf-8
-Sheet 12 12
+Sheet 11 15
 Title "Board Surface Temperature Sensor"
 Date ""
@@
 F 0 "U610" H 5950 3975 60  0000 C CNN
 F 1 "STLM75" H 5950 3525 60  0000 C CNN
-F 2 "" H 5900 3825 60  0001 C CNN
+F 2 "SFUSat:TSSOP-8-3x3mm-SOT505-1" H 5900 3825 60  0001 C CNN
 F 3 "" H 5900 3825 60  0001 C CNN
 	1    5950 3825
@@
 SCL
 $Comp
-L GND #PWR0122
+L GND #PWR090
 U 1 1 5AC262E6
 P 5425 4075
-AR Path="/5AC235B1/5AC262E6" Ref="#PWR0122"  Part="1"
-AR Path="/5AD08722/5AC262E6" Ref="#PWR0128"  Part="1"
-F 0 "#PWR0128" H 5425 3825 50  0001 C CNN
+AR Path="/5AC235B1/5AC262E6" Ref="#PWR090"  Part="1"
+AR Path="/5AD08722/5AC262E6" Ref="#PWR096"  Part="1"
+F 0 "#PWR096" H 5425 3825 50  0001 C CNN
 F 1 "GND" H 5425 3925 50  0000 C CNN
 F 2 "" H 5425 4075 50  0001 C CNN
@@
 $EndComp
 $Comp
-L GND #PWR0123
+L GND #PWR091
 U 1 1 5AD28594
 P 6975 3950
-AR Path="/5AC235B1/5AD28594" Ref="#PWR0123"  Part="1"
-AR Path="/5AD08722/5AD28594" Ref="#PWR0129"  Part="1"
-F 0 "#PWR0129" H 6975 3700 50  0001 C CNN
+AR Path="/5AC235B1/5AD28594" Ref="#PWR091"  Part="1"
+AR Path="/5AD08722/5AD28594" Ref="#PWR097"  Part="1"
+F 0 "#PWR097" H 6975 3700 50  0001 C CNN
 F 1 "GND" H 6975 3800 50  0000 C CNN
 F 2 "" H 6975 3950 50  0001 C CNN

Commit message: Continued routing
Changed lines of the file:
@@
 AR Path="/5AC235B1/5AC2622D" Ref="U600"  Part="1"
 AR Path="/5AD08722/5AC2622D" Ref="U610"  Part="1"
-F 0 "U610" H 5950 3975 60  0000 C CNN
+F 0 "U600" H 5950 3975 60  0000 C CNN
 F 1 "STLM75" H 5950 3525 60  0000 C CNN
 F 2 "SFUSat:TSSOP-8-3x3mm-SOT505-1" H 5900 3825 60  0001 C CNN
@@
 SCL
 $Comp
-L GND #PWR95
+L GND #PWR095
 U 1 1 5AC262E6
 P 5425 4075
-AR Path="/5AC235B1/5AC262E6" Ref="#PWR95"  Part="1"
-AR Path="/5AD08722/5AC262E6" Ref="#PWR101"  Part="1"
-F 0 "#PWR101" H 5425 3825 50  0001 C CNN
+AR Path="/5AC235B1/5AC262E6" Ref="#PWR095"  Part="1"
+AR Path="/5AD08722/5AC262E6" Ref="#PWR0101"  Part="1"
+F 0 "#PWR0101" H 5425 3825 50  0001 C CNN
 F 1 "GND" H 5425 3925 50  0000 C CNN
 F 2 "" H 5425 4075 50  0001 C CNN
@@
 AR Path="/5AC235B1/5AD2851F" Ref="C600"  Part="1"
 AR Path="/5AD08722/5AD2851F" Ref="C610"  Part="1"
-F 0 "C610" H 7000 3900 50  0000 L CNN
+F 0 "C600" H 7000 3900 50  0000 L CNN
 F 1 "DNP" H 7000 3700 50  0000 L CNN
 F 2 "SFUSat-cap:C_0402" H 7013 3650 50  0001 C CNN
@@
 $EndComp
 $Comp
-L GND #PWR96
+L GND #PWR096
 U 1 1 5AD28594
 P 6975 3950
-AR Path="/5AC235B1/5AD28594" Ref="#PWR96"  Part="1"
-AR Path="/5AD08722/5AD28594" Ref="#PWR102"  Part="1"
-F 0 "#PWR102" H 6975 3700 50  0001 C CNN
+AR Path="/5AC235B1/5AD28594" Ref="#PWR096"  Part="1"
+AR Path="/5AD08722/5AD28594" Ref="#PWR0102"  Part="1"
+F 0 "#PWR0102" H 6975 3700 50  0001 C CNN
 F 1 "GND" H 6975 3800 50  0000 C CNN
 F 2 "" H 6975 3950 50  0001 C CNN

Commit message: layed out planes around regulator. The default clearance for poly was set to 1.27 mm but PCBway requires a minimum track spacing of 0.1524mm
Changed lines of the file:
@@
 AR Path="/5AC235B1/5AC2622D" Ref="U600"  Part="1"
 AR Path="/5AD08722/5AC2622D" Ref="U610"  Part="1"
-F 0 "U600" H 5950 3975 60  0000 C CNN
+F 0 "U610" H 5950 3975 60  0000 C CNN
 F 1 "STLM75" H 5950 3525 60  0000 C CNN
 F 2 "SFUSat:TSSOP-8-3x3mm-SOT505-1" H 5900 3825 60  0001 C CNN
@@
 AR Path="/5AC235B1/5AD2851F" Ref="C600"  Part="1"
 AR Path="/5AD08722/5AD2851F" Ref="C610"  Part="1"
-F 0 "C600" H 7000 3900 50  0000 L CNN
+F 0 "C610" H 7000 3900 50  0000 L CNN
 F 1 "DNP" H 7000 3700 50  0000 L CNN
 F 2 "SFUSat-cap:C_0402" H 7013 3650 50  0001 C CNN

Commit message: layed out temp sensor
Changed lines of the file:
@@
 AR Path="/5AC235B1/5AC2622D" Ref="U600"  Part="1"
 AR Path="/5AD08722/5AC2622D" Ref="U610"  Part="1"
-F 0 "U610" H 5950 3975 60  0000 C CNN
+F 0 "U600" H 5950 3975 60  0000 C CNN
 F 1 "STLM75" H 5950 3525 60  0000 C CNN
 F 2 "SFUSat:TSSOP-8-3x3mm-SOT505-1" H 5900 3825 60  0001 C CNN
@@
 AR Path="/5AC235B1/5AC262E6" Ref="#PWR097"  Part="1"
 AR Path="/5AD08722/5AC262E6" Ref="#PWR0103"  Part="1"
-F 0 "#PWR0103" H 5425 3825 50  0001 C CNN
+F 0 "#PWR097" H 5425 3825 50  0001 C CNN
 F 1 "GND" H 5425 3925 50  0000 C CNN
 F 2 "" H 5425 4075 50  0001 C CNN
@@
 AR Path="/5AC235B1/5AD2851F" Ref="C600"  Part="1"
 AR Path="/5AD08722/5AD2851F" Ref="C610"  Part="1"
-F 0 "C610" H 7000 3900 50  0000 L CNN
+F 0 "C600" H 7000 3900 50  0000 L CNN
 F 1 "DNP" H 7000 3700 50  0000 L CNN
 F 2 "SFUSat-cap:C_0402" H 7013 3650 50  0001 C CNN
@@
 AR Path="/5AC235B1/5AD28594" Ref="#PWR098"  Part="1"
 AR Path="/5AD08722/5AD28594" Ref="#PWR0104"  Part="1"
-F 0 "#PWR0104" H 6975 3700 50  0001 C CNN
+F 0 "#PWR098" H 6975 3700 50  0001 C CNN
 F 1 "GND" H 6975 3800 50  0000 C CNN
 F 2 "" H 6975 3950 50  0001 C CNN
