File: TEMP_SENSE.sch (KiCad schematic (older format))
At the start: 2 parts, among them U600 STLM75

Commit message: layed out indicator lights
Changed lines of the file:
@@
 AR Path="/5AC235B1/5AC2622D" Ref="U600"  Part="1"
 AR Path="/5AD08722/5AC2622D" Ref="U610"  Part="1"
-F 0 "U600" H 5950 3975 60  0000 C CNN
+F 0 "U610" H 5950 3975 60  0000 C CNN
 F 1 "STLM75" H 5950 3525 60  0000 C CNN
 F 2 "SFUSat:TSSOP-8-3x3mm-SOT505-1" H 5900 3825 60  0001 C CNN
@@
 SCL
 $Comp
-L GND #PWR097
+L GND #PWR98
 U 1 1 5AC262E6
 P 5425 4075
-AR Path="/5AC235B1/5AC262E6" Ref="#PWR097"  Part="1"
-AR Path="/5AD08722/5AC262E6" Ref="#PWR0103"  Part="1"
-F 0 "#PWR097" H 5425 3825 50  0001 C CNN
+AR Path="/5AC235B1/5AC262E6" Ref="#PWR98"  Part="1"
+AR Path="/5AD08722/5AC262E6" Ref="#PWR104"  Part="1"
+F 0 "#PWR104" H 5425 3825 50  0001 C CNN
 F 1 "GND" H 5425 3925 50  0000 C CNN
 F 2 "" H 5425 4075 50  0001 C CNN
@@
 AR Path="/5AC235B1/5AD2851F" Ref="C600"  Part="1"
 AR Path="/5AD08722/5AD2851F" Ref="C610"  Part="1"
-F 0 "C600" H 7000 3900 50  0000 L CNN
+F 0 "C610" H 7000 3900 50  0000 L CNN
 F 1 "DNP" H 7000 3700 50  0000 L CNN
 F 2 "SFUSat-cap:C_0402" H 7013 3650 50  0001 C CNN
@@
 $EndComp
 $Comp
-L GND #PWR098
+L GND #PWR99
 U 1 1 5AD28594
 P 6975 3950
-AR Path="/5AC235B1/5AD28594" Ref="#PWR098"  Part="1"
-AR Path="/5AD08722/5AD28594" Ref="#PWR0104"  Part="1"
-F 0 "#PWR098" H 6975 3700 50  0001 C CNN
+AR Path="/5AC235B1/5AD28594" Ref="#PWR99"  Part="1"
+AR Path="/5AD08722/5AD28594" Ref="#PWR105"  Part="1"
+F 0 "#PWR105" H 6975 3700 50  0001 C CNN
 F 1 "GND" H 6975 3800 50  0000 C CNN
 F 2 "" H 6975 3950 50  0001 C CNN

Commit message: modified proposed pot schematic
Changed lines of the file:
@@
 $Descr A4 11693 8268
 encoding utf-8
-Sheet 11 15
+Sheet 8 15
 Title "Board Surface Temperature Sensor"
 Date ""
@@
 AR Path="/5AC235B1/5AC2622D" Ref="U600"  Part="1"
 AR Path="/5AD08722/5AC2622D" Ref="U610"  Part="1"
-F 0 "U610" H 5950 3975 60  0000 C CNN
+F 0 "U600" H 5950 3975 60  0000 C CNN
 F 1 "STLM75" H 5950 3525 60  0000 C CNN
 F 2 "SFUSat:TSSOP-8-3x3mm-SOT505-1" H 5900 3825 60  0001 C CNN
@@
 AR Path="/5AC235B1/5AC262E6" Ref="#PWR099"  Part="1"
 AR Path="/5AD08722/5AC262E6" Ref="#PWR0105"  Part="1"
-F 0 "#PWR0105" H 5425 3825 50  0001 C CNN
+F 0 "#PWR099" H 5425 3825 50  0001 C CNN
 F 1 "GND" H 5425 3925 50  0000 C CNN
 F 2 "" H 5425 4075 50  0001 C CNN
@@
 AR Path="/5AC235B1/5AD2851F" Ref="C600"  Part="1"
 AR Path="/5AD08722/5AD2851F" Ref="C610"  Part="1"
-F 0 "C610" H 7000 3900 50  0000 L CNN
+F 0 "C600" H 7000 3900 50  0000 L CNN
 F 1 "DNP" H 7000 3700 50  0000 L CNN
 F 2 "SFUSat-cap:C_0402" H 7013 3650 50  0001 C CNN
@@
 AR Path="/5AC235B1/5AD28594" Ref="#PWR0100"  Part="1"
 AR Path="/5AD08722/5AD28594" Ref="#PWR0106"  Part="1"
-F 0 "#PWR0106" H 6975 3700 50  0001 C CNN
+F 0 "#PWR0100" H 6975 3700 50  0001 C CNN
 F 1 "GND" H 6975 3800 50  0000 C CNN
 F 2 "" H 6975 3950 50  0001 C CNN

Commit message: Changed 'DNP' to 'DNF' for new BOM tool
Parts:
- C600: value DNP -> DNF
Changed lines of the file:
@@
 AR Path="/5AC235B1/5AC262E6" Ref="#PWR099"  Part="1"
 AR Path="/5AD08722/5AC262E6" Ref="#PWR0105"  Part="1"
-F 0 "#PWR0105" H 5425 3825 50  0001 C CNN
+F 0 "#PWR099" H 5425 3825 50  0001 C CNN
 F 1 "GND" H 5425 3925 50  0000 C CNN
 F 2 "" H 5425 4075 50  0001 C CNN
@@
 AR Path="/5AD08722/5AD2851F" Ref="C610"  Part="1"
 F 0 "C600" H 7000 3900 50  0000 L CNN
-F 1 "DNP" H 7000 3700 50  0000 L CNN
+F 1 "DNF" H 7000 3700 50  0000 L CNN
 F 2 "SFUSat-cap:C_0402" H 7013 3650 50  0001 C CNN
 F 3 "" H 6975 3800 50  0001 C CNN
@@
 AR Path="/5AC235B1/5AD28594" Ref="#PWR0100"  Part="1"
 AR Path="/5AD08722/5AD28594" Ref="#PWR0106"  Part="1"
-F 0 "#PWR0106" H 6975 3700 50  0001 C CNN
+F 0 "#PWR0100" H 6975 3700 50  0001 C CNN
 F 1 "GND" H 6975 3800 50  0000 C CNN
 F 2 "" H 6975 3950 50  0001 C CNN

Commit message: Closes #58
Changed lines of the file:
@@
 AR Path="/5AC235B1/5AC2622D" Ref="U600"  Part="1"
 AR Path="/5AD08722/5AC2622D" Ref="U610"  Part="1"
-F 0 "U600" H 5950 3975 60  0000 C CNN
+F 0 "U610" H 5950 3975 60  0000 C CNN
 F 1 "STLM75" H 5950 3525 60  0000 C CNN
 F 2 "SFUSat:TSSOP-8-3x3mm-SOT505-1" H 5900 3825 60  0001 C CNN
@@
 AR Path="/5AC235B1/5AC262E6" Ref="#PWR099"  Part="1"
 AR Path="/5AD08722/5AC262E6" Ref="#PWR0105"  Part="1"
-F 0 "#PWR099" H 5425 3825 50  0001 C CNN
+F 0 "#PWR0105" H 5425 3825 50  0001 C CNN
 F 1 "GND" H 5425 3925 50  0000 C CNN
 F 2 "" H 5425 4075 50  0001 C CNN
@@
 AR Path="/5AC235B1/5AD2851F" Ref="C600"  Part="1"
 AR Path="/5AD08722/5AD2851F" Ref="C610"  Part="1"
-F 0 "C600" H 7000 3900 50  0000 L CNN
+F 0 "C610" H 7000 3900 50  0000 L CNN
 F 1 "DNF" H 7000 3700 50  0000 L CNN
 F 2 "SFUSat-cap:C_0402" H 7013 3650 50  0001 C CNN
@@
 AR Path="/5AC235B1/5AD28594" Ref="#PWR0100"  Part="1"
 AR Path="/5AD08722/5AD28594" Ref="#PWR0106"  Part="1"
-F 0 "#PWR0100" H 6975 3700 50  0001 C CNN
+F 0 "#PWR0106" H 6975 3700 50  0001 C CNN
 F 1 "GND" H 6975 3800 50  0000 C CNN
 F 2 "" H 6975 3950 50  0001 C CNN
