File: Reg_3V6.sch (KiCad schematic (older format))
At the start: 22 parts, among them U4 LMS3635AQRNLRQ1

Commit message: layed out power system
Parts:
- U4: Digikey (none) -> 296-47482-1-ND; Mouser (none) -> 595-LMS3635AQRNLTQ1
Connections:
- wire segments 66 -> 70
Changed lines of the file:
@@
 	1    0    0    -1
 $EndComp
-Wire Wire Line
-	2950 3125 2950 3175
-Wire Wire Line
-	2650 3125 2650 3175
-Wire Wire Line
-	2350 3125 2350 3175
 $Comp
 L GND #PWR0101
@@
 	1    0    0    -1
 $EndComp
-Wire Wire Line
-	6575 3475 6575 3525
-Wire Wire Line
-	5725 1700 7175 1700
-Connection ~ 7125 1700
-Wire Wire Line
-	7475 1700 9950 1700
-Wire Wire Line
-	7975 1700 7975 1750
-Wire Wire Line
-	7575 1750 7575 1700
-Connection ~ 7575 1700
-Wire Wire Line
-	7975 2050 7975 2150
-Wire Wire Line
-	7275 2100 7975 2100
-Connection ~ 7975 2100
-Wire Wire Line
-	7575 2050 7575 2100
-Connection ~ 7575 2100
 $Comp
 L GND #PWR0102
@@
 	1    0    0    -1
 $EndComp
-Wire Wire Line
-	8225 3700 8225 3800
-Wire Wire Line
-	8225 4100 8225 4150
 $Comp
 L GND #PWR0103
@@
 	1    0    0    -1
 $EndComp
-Wire Wire Line
-	7975 2450 7975 2500
 $Comp
 L C_47u0_10%_6.3V_X5R_1206 C26
@@
 	1    0    0    -1
 $EndComp
-Wire Wire Line
-	8575 2050 8575 2100
 $Comp
 L C_47u0_10%_6.3V_X5R_1206 C27
@@
 	1    0    0    -1
 $EndComp
-Wire Wire Line
-	8875 2050 8875 2100
 $Comp
 L C_47u0_10%_6.3V_X5R_1206 C28
@@
 	1    0    0    -1
 $EndComp
-Wire Wire Line
-	9175 2050 9175 2100
 $Comp
 L C_47u0_10%_6.3V_X5R_1206 C29
@@
 	1    0    0    -1
 $EndComp
-Wire Wire Line
-	9475 2050 9475 2100
-Wire Wire Line
-	9475 1700 9475 1750
-Connection ~ 7975 1700
-Wire Wire Line
-	9175 1750 9175 1700
-Connection ~ 9175 1700
-Wire Wire Line
-	8875 1750 8875 1700
-Connection ~ 8875 1700
-Wire Wire Line
-	8575 1750 8575 1700
-Connection ~ 8575 1700
-Wire Wire Line
-	8225 1700 8225 3400
-Connection ~ 8225 1700
 $Comp
 L C_10u0_10%_16V_X5R_1210 C1
@@
 	1    0    0    -1
 $EndComp
-Wire Wire Line
-	2050 3125 2050 3175
 $Comp
 L C_10u0_10%_16V_X5R_1210 C20
@@
 	1    0    0    -1
 $EndComp
-Wire Wire Line
-	4150 3125 4150 3175
-Wire Wire Line
-	3850 3125 3850 3175
-Wire Wire Line
-	3550 3125 3550 3175
 $Comp
 L C_10u0_10%_16V_X5R_1210 C18
@@
 	1    0    0    -1
 $EndComp
-Wire Wire Line
-	3250 3125 3250 3175
-Wire Wire Line
-	1925 2775 4875 2775
-Wire Wire Line
-	2050 2825 2050 2775
-Connection ~ 2050 2775
-Wire Wire Line
-	2350 2825 2350 2775
-Connection ~ 2350 2775
-Wire Wire Line
-	2650 2825 2650 2775
-Connection ~ 2650 2775
-Wire Wire Line
-	2950 2825 2950 2775
-Connection ~ 2950 2775
-Wire Wire Line
-	3250 2825 3250 2775
-Connection ~ 3250 2775
-Wire Wire Line
-	3550 2825 3550 2775
-Connection ~ 3550 2775
-Wire Wire Line
-	3850 2825 3850 2775
-Connection ~ 3850 2775
-Wire Wire Line
-	4150 2825 4150 2775
-Connection ~ 4150 2775
 $Comp
 L C_47u0_10%_6.3V_X5R_1206 C30
@@
 	1    0    0    -1
 $EndComp
-Wire Wire Line
-	9775 2050 9775 2100
-Wire Wire Line
-	9775 1700 9775 1750
-Connection ~ 9475 1700
-Connection ~ 9775 1700
 Text HLabel 5325 3650 3    60   Input ~ 0
 EN_3V6
@@
 F 2 "SFUSat:LMS3635AQRNLTQ1" H 5675 2575 60  0001 C CNN
 F 3 "" H 5675 2575 60  0001 C CNN
+F 4 "296-47482-1-ND" H 5675 2725 60  0001 C CNN "Digikey"
+F 5 "595-LMS3635AQRNLTQ1" H 5675 2725 60  0001 C CNN "Mouser"
 	1    5675 2725
 	1    0    0    -1
 $EndComp
-Wire Wire Line
-	6475 3125 6575 3125
-Wire Wire Line
-	6575 3125 6575 3175
-Wire Wire Line
-	4875 2625 4725 2625
-Wire Wire Line
-	4725 2625 4725 2775
-Connection ~ 4725 2775
-Wire Wire Line
-	4725 2700 6525 2700
-Wire Wire Line
-	6525 2700 6525 2625
-Wire Wire Line
-	6525 2625 6475 2625
-Connection ~ 4725 2700
-Wire Wire Line
-	5325 3525 5325 3650
 $Comp
 L GND #PWR0114
@@
 	1    0    0    -1
 $EndComp
-Wire Wire Line
-	4875 2975 4750 2975
-Wire Wire Line
-	4750 2975 4750 3100
 $Comp
 L GND #PWR0115
@@
 $EndComp
 NoConn ~ 5475 3525
-Wire Wire Line
-	6475 2375 6575 2375
-Wire Wire Line
-	6475 2275 6525 2275
-Wire Wire Line
-	6525 2275 6525 2475
-Connection ~ 6525 2375
-Wire Wire Line
-	6525 2475 6475 2475
-Wire Wire Line
-	5625 3525 5625 3600
-Wire Wire Line
-	6475 2975 6650 2975
-Wire Wire Line
-	7125 2975 6950 2975
-Wire Wire Line
-	7125 2975 7125 1700
-Wire Wire Line
-	7275 2100 7275 3850
-Wire Wire Line
-	7275 3850 5775 3850
-Wire Wire Line
-	5775 3850 5775 3525
-Wire Wire Line
-	5725 1700 5725 1875
-Wire Wire Line
-	5925 3525 5925 3775
-Wire Wire Line
-	5925 3775 8225 3775
-Connection ~ 8225 3775
 $Comp
 L GND #PWR0117
@@
 	0    -1   -1   0
 $EndComp
-Wire Wire Line
-	6475 2825 6550 2825
 $Comp
 L GND #PWR0118
@@
 	-1   0    0    1
 $EndComp
+$Comp
+L GND #PWR0120
+U 1 1 5AD173E7
+P 4725 2375
+F 0 "#PWR0120" H 4725 2125 50  0001 C CNN
+F 1 "GND" H 4725 2225 50  0000 C CNN
+F 2 "" H 4725 2375 50  0001 C CNN
+F 3 "" H 4725 2375 50  0001 C CNN
+	1    4725 2375
+	0    1    1    0
+$EndComp
+Wire Wire Line
+	2950 3125 2950 3175
+Wire Wire Line
+	2650 3125 2650 3175
+Wire Wire Line
+	2350 3125 2350 3175
+Wire Wire Line
+	6575 3475 6575 3525
+Wire Wire Line
+	5725 1700 7175 1700
+Connection ~ 7125 1700
+Wire Wire Line
+	7475 1700 9950 1700
+Wire Wire Line
+	7975 1700 7975 1750
+Wire Wire Line
+	7575 1750 7575 1700
+Connection ~ 7575 1700
+Wire Wire Line
+	7975 2050 7975 2150
+Wire Wire Line
+	7275 2100 7975 2100
+Connection ~ 7975 2100
+Wire Wire Line
+	7575 2050 7575 2100
+Connection ~ 7575 2100
+Wire Wire Line
+	8225 3700 8225 3800
+Wire Wire Line
+	8225 4100 8225 4150
+Wire Wire Line
+	7975 2450 7975 2500
+Wire Wire Line
+	8575 2050 8575 2100
+Wire Wire Line
+	8875 2050 8875 2100
+Wire Wire Line
+	9175 2050 9175 2100
+Wire Wire Line
+	9475 2050 9475 2100
+Wire Wire Line
+	9475 1700 9475 1750
+Connection ~ 7975 1700
+Wire Wire Line
+	9175 1750 9175 1700
+Connection ~ 9175 1700
+Wire Wire Line
+	8875 1750 8875 1700
+Connection ~ 8875 1700
+Wire Wire Line
+	8575 1750 8575 1700
+Connection ~ 8575 1700
+Wire Wire Line
+	8225 1700 8225 3400
+Connection ~ 8225 1700
+Wire Wire Line
+	2050 3125 2050 3175
+Wire Wire Line
+	4150 3125 4150 3175
+Wire Wire Line
+	3850 3125 3850 3175
+Wire Wire Line
+	3550 3125 3550 3175
+Wire Wire Line
+	3250 3125 3250 3175
+Wire Wire Line
+	1925 2775 4875 2775
+Wire Wire Line
+	2050 2825 2050 2775
+Connection ~ 2050 2775
+Wire Wire Line
+	2350 2825 2350 2775
+Connection ~ 2350 2775
+Wire Wire Line
+	2650 2825 2650 2775
+Connection ~ 2650 2775
+Wire Wire Line
+	2950 2825 2950 2775
+Connection ~ 2950 2775
+Wire Wire Line
+	3250 2825 3250 2775
+Connection ~ 3250 2775
+Wire Wire Line
+	3550 2825 3550 2775
+Connection ~ 3550 2775
+Wire Wire Line
+	3850 2825 3850 2775
+Connection ~ 3850 2775
+Wire Wire Line
+	4150 2825 4150 2775
+Connection ~ 4150 2775
+Wire Wire Line
+	9775 2050 9775 2100
+Wire Wire Line
+	9775 1700 9775 1750
+Connection ~ 9475 1700
+Connection ~ 9775 1700
+Wire Wire Line
+	6475 3125 6575 3125
+Wire Wire Line
+	6575 3125 6575 3175
+Wire Wire Line
+	4875 2625 4725 2625
+Wire Wire Line
+	4725 2625 4725 2775
+Connection ~ 4725 2775
+Wire Wire Line
+	4725 2700 6525 2700
+Wire Wire Line
+	6525 2700 6525 2625
+Wire Wire Line
+	6525 2625 6475 2625
+Connection ~ 4725 2700
+Wire Wire Line
+	5325 3525 5325 3650
+Wire Wire Line
+	4875 2975 4750 2975
+Wire Wire Line
+	4750 2975 4750 3100
+Wire Wire Line
+	6475 2375 6575 2375
+Wire Wire Line
+	6475 2275 6525 2275
+Wire Wire Line
+	6525 2275 6525 2475
+Connection ~ 6525 2375
+Wire Wire Line
+	6525 2475 6475 2475
+Wire Wire Line
+	5625 3525 5625 3600
+Wire Wire Line
+	6475 2975 6650 2975
+Wire Wire Line
+	7125 2975 6950 2975
+Wire Wire Line
+	7125 2975 7125 1700
+Wire Wire Line
+	7275 2100 7275 3850
+Wire Wire Line
+	7275 3850 5775 3850
+Wire Wire Line
+	5775 3850 5775 3525
+Wire Wire Line
+	5725 1700 5725 1875
+Wire Wire Line
+	5925 3525 5925 3775
+Wire Wire Line
+	5925 3775 8225 3775
+Connection ~ 8225 3775
+Wire Wire Line
+	6475 2825 6550 2825
 Wire Wire Line
 	5875 1825 5875 1875
 Wire Wire Line
 	5525 1825 5525 1875
+Wire Wire Line
+	4875 2275 4800 2275
+Wire Wire Line
+	4800 2275 4800 2475
+Wire Wire Line
+	4800 2475 4875 2475
+Wire Wire Line
+	4725 2375 4875 2375
+Connection ~ 4800 2375
 $EndSCHEMATC

Commit message: Closes 45
Connections:
- wire segments 70 -> 68

Commit message: layed out planes around regulator. The default clearance for poly was set to 1.27 mm but PCBway requires a minimum track spacing of 0.1524mm
Connections:
- net labels added: BIAS, BOOST, FB, SW
Changed lines of the file:
@@
 Wire Wire Line
 	4700 2650 4700 2800
+Text Label 7250 2425 0    60   ~ 0
+FB
+Text Label 7450 3800 0    60   ~ 0
+BIAS
+Text Label 6475 1725 0    60   ~ 0
+SW
+Text Label 6500 3000 0    60   ~ 0
+BOOST
 $EndSCHEMATC
