File: Reg_3V1.sch (KiCad schematic (older format))
At the start: 6 parts, among them J26 TEST_1P, U9 TLV702

Commit message: layed out power system
Parts:
- removed D1: PESD5Zx, SFUSat:PESD57zx, symbol PESD5Zx
Connections:
- wire segments 9 -> 8
Other:
- note removed: "Do we need this diode?"
Changed lines of the file:
@@
 $Descr A4 11693 8268
 encoding utf-8
-Sheet 14 15
+Sheet 13 15
 Title ""
 Date ""
@@
 $EndComp
 $Comp
-L GND #PWR0120
+L GND #PWR0121
 U 1 1 5AC11B00
 P 5500 4225
-F 0 "#PWR0120" H 5500 3975 50  0001 C CNN
+F 0 "#PWR0121" H 5500 3975 50  0001 C CNN
 F 1 "GND" H 5500 4075 50  0000 C CNN
 F 2 "" H 5500 4225 50  0001 C CNN
@@
 $EndComp
 $Comp
-L GND #PWR0121
+L GND #PWR0122
 U 1 1 5AC11B1A
 P 4775 3875
-F 0 "#PWR0121" H 4775 3625 50  0001 C CNN
+F 0 "#PWR0122" H 4775 3625 50  0001 C CNN
 F 1 "GND" H 4775 3725 50  0000 C CNN
 F 2 "" H 4775 3875 50  0001 C CNN
@@
 $EndComp
 $Comp
-L GND #PWR0122
+L GND #PWR0123
 U 1 1 5AC11B20
 P 6250 3875
-F 0 "#PWR0122" H 6250 3625 50  0001 C CNN
+F 0 "#PWR0123" H 6250 3625 50  0001 C CNN
 F 1 "GND" H 6250 3725 50  0000 C CNN
 F 2 "" H 6250 3875 50  0001 C CNN
@@
 3V6
 $Comp
-L PESD5Zx D1
-U 1 1 5AC11B36
-P 6625 3825
-F 0 "D1" H 6725 3625 60  0000 C CNN
-F 1 "PESD5Zx" V 6850 3825 60  0000 C CNN
-F 2 "SFUSat:PESD57zx" H 6625 3825 60  0001 C CNN
-F 3 "" H 6625 3825 60  0001 C CNN
-F 4 "PESD5Z3.3,115" H 6625 3825 60  0001 C CNN "Part Number"
-F 5 "1727-5814-1-ND" H 6625 3825 60  0001 C CNN "Digi-Key"
-F 6 "771-PESD5Z33115" H 6625 3825 60  0001 C CNN "Mouser"
-	1    6625 3825
-	1    0    0    -1
-$EndComp
-$Comp
-L GND #PWR0123
-U 1 1 5AC11B3D
-P 6625 4175
-F 0 "#PWR0123" H 6625 3925 50  0001 C CNN
-F 1 "GND" H 6625 4025 50  0000 C CNN
-F 2 "" H 6625 4175 50  0001 C CNN
-F 3 "" H 6625 4175 50  0001 C CNN
-	1    6625 4175
-	1    0    0    -1
-$EndComp
-$Comp
 L TEST_1P J26
 U 1 1 5AC11B43
@@
 Wire Wire Line
 	6250 3450 6250 3525
-Connection ~ 6625 3525
-Wire Wire Line
-	6625 4175 6625 4125
 Wire Wire Line
 	5025 3725 5025 3475
@@
 Wire Wire Line
 	5500 4225 5500 4175
-Text Notes 6300 4200 0    60   ~ 0
-Do we need this diode?
 $EndSCHEMATC

Commit message: Continued routing
Parts:
- removed J26: TEST_1P, SFUSat:Measurement_Point_Round-SMD-Pad_Big, symbol TEST_1P
- added J26: TP_TH_150, SFUSat:TP_TH_150, symbol TP_TH_150
Connections:
- net labels removed: 3V6
- wire segments 8 -> 9
Changed lines of the file:
@@
 $EndComp
 $Comp
-L GND #PWR127
+L GND #PWR0126
 U 1 1 5AC11B00
 P 5500 4225
-F 0 "#PWR127" H 5500 3975 50  0001 C CNN
+F 0 "#PWR0126" H 5500 3975 50  0001 C CNN
 F 1 "GND" H 5500 4075 50  0000 C CNN
 F 2 "" H 5500 4225 50  0001 C CNN
@@
 $EndComp
 $Comp
-L GND #PWR126
+L GND #PWR0127
 U 1 1 5AC11B1A
 P 4775 3875
-F 0 "#PWR126" H 4775 3625 50  0001 C CNN
+F 0 "#PWR0127" H 4775 3625 50  0001 C CNN
 F 1 "GND" H 4775 3725 50  0000 C CNN
 F 2 "" H 4775 3875 50  0001 C CNN
@@
 $EndComp
 $Comp
-L GND #PWR128
+L GND #PWR0128
 U 1 1 5AC11B20
 P 6250 3875
-F 0 "#PWR128" H 6250 3625 50  0001 C CNN
+F 0 "#PWR0128" H 6250 3625 50  0001 C CNN
 F 1 "GND" H 6250 3725 50  0000 C CNN
 F 2 "" H 6250 3875 50  0001 C CNN
@@
 	1    0    0    -1
 $EndComp
-Text HLabel 5025 3175 1    60   Input ~ 0
-3V6
-$Comp
-L TEST_1P J26
-U 1 1 5AC11B43
-P 6250 3450
-F 0 "J26" H 6250 3720 50  0000 C CNN
-F 1 "TEST_1P" H 6250 3650 50  0000 C CNN
-F 2 "SFUSat:Measurement_Point_Round-SMD-Pad_Big" H 6450 3450 50  0001 C CNN
-F 3 "" H 6450 3450 50  0001 C CNN
-	1    6250 3450
-	1    0    0    -1
-$EndComp
 Wire Wire Line
 	6250 3450 6250 3525
@@
 Wire Wire Line
 	5500 4225 5500 4175
+$Comp
+L TP_TH_150 J26
+U 1 1 5ADA9957
+P 6250 3450
+F 0 "J26" H 6250 3720 50  0000 C CNN
+F 1 "TP_TH_150" H 6250 3650 50  0000 C CNN
+F 2 "SFUSat:TP_TH_150" H 6250 3450 50  0001 C CNN
+F 3 "" H 6450 3450 50  0000 C CNN
+	1    6250 3450
+	1    0    0    -1
+$EndComp
+Wire Wire Line
+	5025 3175 5025 3100
+Text HLabel 5025 3100 1    60   Input ~ 0
+3V6IN
 $EndSCHEMATC

Commit message: layed out planes around regulator. The default clearance for poly was set to 1.27 mm but PCBway requires a minimum track spacing of 0.1524mm
Parts:
- removed J26: TP_TH_150, SFUSat:TP_TH_150, symbol TP_TH_150
Connections:
- wire segments 9 -> 8
Changed lines of the file:
@@
 $EndComp
-Wire Wire Line
-	6250 3450 6250 3525
 Wire Wire Line
 	5025 3725 5025 3475
@@
 Wire Wire Line
 	5500 4225 5500 4175
-$Comp
-L TP_TH_150 J26
-U 1 1 5ADA9957
-P 6250 3450
-F 0 "J26" H 6250 3720 50  0000 C CNN
-F 1 "TP_TH_150" H 6250 3650 50  0000 C CNN
-F 2 "SFUSat:TP_TH_150" H 6250 3450 50  0001 C CNN
-F 3 "" H 6450 3450 50  0000 C CNN
-	1    6250 3450
-	1    0    0    -1
-$EndComp
 Wire Wire Line
 	5025 3175 5025 3100
