File: indicator.sch (KiCad schematic (older format))
At the start: 7 parts, among them J23 TP_TH_150, J24 TP_TH_150, U420 2N7002DW

Commit message: modified proposed pot schematic
Changed lines of the file:
@@
 $Descr A4 11693 8268
 encoding utf-8
-Sheet 10 15
+Sheet 9 15
 Title ""
 Date ""
@@
 AR Path="/5AC903D9/5AC92C0F" Ref="U420"  Part="1"
 AR Path="/5AC9A534/5AC92C0F" Ref="U14"  Part="1"
-F 0 "U14" H 5725 3625 60  0000 C CNN
+F 0 "U420" H 5725 3625 60  0000 C CNN
 F 1 "2N7002DW" H 5525 4125 60  0000 C CNN
 F 2 "SFUSat:SOT-363" H 5525 3875 60  0001 C CNN
@@
 AR Path="/5AC903D9/5AC92C16" Ref="D420"  Part="1"
 AR Path="/5AC9A534/5AC92C16" Ref="D2"  Part="1"
-F 0 "D2" H 6125 3625 50  0000 C CNN
+F 0 "D420" H 6125 3625 50  0000 C CNN
 F 1 "GREEN" H 6125 3425 50  0000 C CNN
 F 2 "SFUSat:LED_0603" H 6125 3525 50  0001 C CNN
@@
 AR Path="/5AC903D9/5AC92C1D" Ref="R420"  Part="1"
 AR Path="/5AC9A534/5AC92C1D" Ref="R8"  Part="1"
-F 0 "R8" V 6205 3175 50  0000 C CNN
+F 0 "R420" V 6205 3175 50  0000 C CNN
 F 1 "287" V 6125 3175 50  0000 C CNN
 F 2 "SFUSat:R_0402" V 6055 3175 50  0001 C CNN
@@
 AR Path="/5AC903D9/5AC92C24" Ref="R421"  Part="1"
 AR Path="/5AC9A534/5AC92C24" Ref="R14"  Part="1"
-F 0 "R14" V 6505 3175 50  0000 C CNN
+F 0 "R421" V 6505 3175 50  0000 C CNN
 F 1 "287" V 6425 3175 50  0000 C CNN
 F 2 "SFUSat:R_0402" V 6355 3175 50  0001 C CNN
@@
 AR Path="/5AC903D9/5AC92C2B" Ref="D421"  Part="1"
 AR Path="/5AC9A534/5AC92C2B" Ref="D4"  Part="1"
-F 0 "D4" H 6425 3625 50  0000 C CNN
+F 0 "D421" H 6425 3625 50  0000 C CNN
 F 1 "GREEN" H 6425 3425 50  0000 C CNN
 F 2 "SFUSat:LED_0603" H 6425 3525 50  0001 C CNN
@@
 AR Path="/5AC903D9/5AC92C32" Ref="#PWR0101"  Part="1"
 AR Path="/5AC9A534/5AC92C32" Ref="#PWR0103"  Part="1"
-F 0 "#PWR0103" H 5975 3575 50  0001 C CNN
+F 0 "#PWR0101" H 5975 3575 50  0001 C CNN
 F 1 "GND" H 5975 3675 50  0000 C CNN
 F 2 "" H 5975 3825 50  0000 C CNN
@@
 AR Path="/5AC903D9/5AC92C38" Ref="#PWR0102"  Part="1"
 AR Path="/5AC9A534/5AC92C38" Ref="#PWR0104"  Part="1"
-F 0 "#PWR0104" H 5975 3775 50  0001 C CNN
+F 0 "#PWR0102" H 5975 3775 50  0001 C CNN
 F 1 "GND" H 5975 3875 50  0000 C CNN
 F 2 "" H 5975 4025 50  0000 C CNN
@@
 AR Path="/5AC9A534/5AD94712" Ref="J24"  Part="1"
 AR Path="/5AC903D9/5AD94712" Ref="J22"  Part="1"
-F 0 "J24" H 5025 4320 50  0000 C CNN
+F 0 "J22" H 5025 4320 50  0000 C CNN
 F 1 "TP_TH_150" H 5025 4250 50  0000 C CNN
 F 2 "SFUSat:TP_TH_150" H 5025 4050 50  0001 C CNN
@@
 AR Path="/5AC9A534/5AD94797" Ref="J23"  Part="1"
 AR Path="/5AC903D9/5AD94797" Ref="J21"  Part="1"
-F 0 "J23" H 5025 3970 50  0000 C CNN
+F 0 "J21" H 5025 3970 50  0000 C CNN
 F 1 "TP_TH_150" H 5025 3900 50  0000 C CNN
 F 2 "SFUSat:TP_TH_150" H 5025 3700 50  0001 C CNN

Commit message: final cleanup and check
Changed lines of the file:
@@
 $Descr A4 11693 8268
 encoding utf-8
-Sheet 9 15
+Sheet 10 15
 Title ""
 Date ""
@@
 AR Path="/5AC903D9/5AC92C0F" Ref="U420"  Part="1"
 AR Path="/5AC9A534/5AC92C0F" Ref="U14"  Part="1"
-F 0 "U420" H 5725 3625 60  0000 C CNN
+F 0 "U14" H 5725 3625 60  0000 C CNN
 F 1 "2N7002DW" H 5525 4125 60  0000 C CNN
 F 2 "SFUSat:SOT-363" H 5525 3875 60  0001 C CNN
@@
 AR Path="/5AC903D9/5AC92C16" Ref="D420"  Part="1"
 AR Path="/5AC9A534/5AC92C16" Ref="D2"  Part="1"
-F 0 "D420" H 6125 3625 50  0000 C CNN
+F 0 "D2" H 6125 3625 50  0000 C CNN
 F 1 "GREEN" H 6125 3425 50  0000 C CNN
 F 2 "SFUSat:LED_0603" H 6125 3525 50  0001 C CNN
@@
 AR Path="/5AC903D9/5AC92C1D" Ref="R420"  Part="1"
 AR Path="/5AC9A534/5AC92C1D" Ref="R8"  Part="1"
-F 0 "R420" V 6205 3175 50  0000 C CNN
+F 0 "R8" V 6205 3175 50  0000 C CNN
 F 1 "287" V 6125 3175 50  0000 C CNN
 F 2 "SFUSat:R_0402" V 6055 3175 50  0001 C CNN
@@
 AR Path="/5AC903D9/5AC92C24" Ref="R421"  Part="1"
 AR Path="/5AC9A534/5AC92C24" Ref="R14"  Part="1"
-F 0 "R421" V 6505 3175 50  0000 C CNN
+F 0 "R14" V 6505 3175 50  0000 C CNN
 F 1 "287" V 6425 3175 50  0000 C CNN
 F 2 "SFUSat:R_0402" V 6355 3175 50  0001 C CNN
@@
 AR Path="/5AC903D9/5AC92C2B" Ref="D421"  Part="1"
 AR Path="/5AC9A534/5AC92C2B" Ref="D4"  Part="1"
-F 0 "D421" H 6425 3625 50  0000 C CNN
+F 0 "D4" H 6425 3625 50  0000 C CNN
 F 1 "GREEN" H 6425 3425 50  0000 C CNN
 F 2 "SFUSat:LED_0603" H 6425 3525 50  0001 C CNN
@@
 AR Path="/5AC9A534/5AD94712" Ref="J24"  Part="1"
 AR Path="/5AC903D9/5AD94712" Ref="J22"  Part="1"
-F 0 "J22" H 5025 4320 50  0000 C CNN
+F 0 "J24" H 5025 4320 50  0000 C CNN
 F 1 "TP_TH_150" H 5025 4250 50  0000 C CNN
 F 2 "SFUSat:TP_TH_150" H 5025 4050 50  0001 C CNN
@@
 AR Path="/5AC9A534/5AD94797" Ref="J23"  Part="1"
 AR Path="/5AC903D9/5AD94797" Ref="J21"  Part="1"
-F 0 "J21" H 5025 3970 50  0000 C CNN
+F 0 "J23" H 5025 3970 50  0000 C CNN
 F 1 "TP_TH_150" H 5025 3900 50  0000 C CNN
 F 2 "SFUSat:TP_TH_150" H 5025 3700 50  0001 C CNN
