File: Reg_5V0.sch (KiCad schematic (older format))
At the start: 11 parts, among them U15 TPS62175DQCR, U16 TPS71750DSER

Commit message: layed out power system
Connections:
- wire segments 40 -> 42
Changed lines of the file:
@@
 $EndComp
 $Comp
-L GND #PWR0128
+L GND #PWR0129
 U 1 1 5AC130F2
 P 4200 4325
-F 0 "#PWR0128" H 4200 4075 50  0001 C CNN
+F 0 "#PWR0129" H 4200 4075 50  0001 C CNN
 F 1 "GND" H 4200 4175 50  0000 C CNN
 F 2 "" H 4200 4325 50  0001 C CNN
@@
 Connection ~ 3650 3550
 $Comp
-L GND #PWR0129
+L GND #PWR0130
 U 1 1 5AC13104
 P 3350 4000
-F 0 "#PWR0129" H 3350 3750 50  0001 C CNN
+F 0 "#PWR0130" H 3350 3750 50  0001 C CNN
 F 1 "GND" H 3350 3850 50  0000 C CNN
 F 2 "" H 3350 4000 50  0001 C CNN
@@
 $EndComp
 $Comp
-L GND #PWR0130
+L GND #PWR0131
 U 1 1 5AC1310A
 P 5775 4050
-F 0 "#PWR0130" H 5775 3800 50  0001 C CNN
+F 0 "#PWR0131" H 5775 3800 50  0001 C CNN
 F 1 "GND" H 5775 3900 50  0000 C CNN
 F 2 "" H 5775 4050 50  0001 C CNN
@@
 	5775 3950 5775 4050
 $Comp
-L GND #PWR0131
+L GND #PWR0132
 U 1 1 5AC13126
 P 5500 4300
-F 0 "#PWR0131" H 5500 4050 50  0001 C CNN
+F 0 "#PWR0132" H 5500 4050 50  0001 C CNN
 F 1 "GND" H 5500 4150 50  0000 C CNN
 F 2 "" H 5500 4300 50  0001 C CNN
@@
 $EndComp
 $Comp
-L GND #PWR0132
+L GND #PWR0133
 U 1 1 5AC131B1
 P 6225 4000
-F 0 "#PWR0132" H 6225 3750 50  0001 C CNN
+F 0 "#PWR0133" H 6225 3750 50  0001 C CNN
 F 1 "GND" H 6225 3850 50  0000 C CNN
 F 2 "" H 6225 4000 50  0001 C CNN
@@
 $EndComp
 $Comp
-L GND #PWR0133
+L GND #PWR0134
 U 1 1 5AC131B7
 P 7475 4150
-F 0 "#PWR0133" H 7475 3900 50  0001 C CNN
+F 0 "#PWR0134" H 7475 3900 50  0001 C CNN
 F 1 "GND" H 7475 4000 50  0000 C CNN
 F 2 "" H 7475 4150 50  0001 C CNN
@@
 $EndComp
 $Comp
-L GND #PWR0134
+L GND #PWR0135
 U 1 1 5AC131BD
 P 7725 3975
-F 0 "#PWR0134" H 7725 3725 50  0001 C CNN
+F 0 "#PWR0135" H 7725 3725 50  0001 C CNN
 F 1 "GND" H 7725 3825 50  0000 C CNN
 F 2 "" H 7725 3975 50  0001 C CNN
@@
 $EndComp
 $Comp
-L GND #PWR0135
+L GND #PWR0136
 U 1 1 5AC131C3
 P 6550 3800
-F 0 "#PWR0135" H 6550 3550 50  0001 C CNN
+F 0 "#PWR0136" H 6550 3550 50  0001 C CNN
 F 1 "GND" H 6550 3650 50  0000 C CNN
 F 2 "" H 6550 3800 50  0001 C CNN
@@
 5V0
 Connection ~ 7725 3550
+Wire Wire Line
+	7400 3750 7400 4125
+Wire Wire Line
+	7400 4125 7475 4125
+Connection ~ 7475 4125
 $EndSCHEMATC
